File: PCB/ISO_PSU.sch (KiCad schematic (older format))
At the start: 11 parts, among them Q1 Q_NPN_CBE, U2 MGJ2

Commit message: Schematics & footprints completed
Ready for PCBnew
Parts:
- C5, C6, C7, C8, C9: footprint (none) -> Capacitors_SMD:C_0805_HandSoldering
- D1: value D_Zener -> MMSZ5251B; footprint (none) -> Diodes_SMD:D_SOD-123
- FL1: footprint (none) -> ENNOID:ACM4520
- Q1: footprint (none) -> TO_SOT_Packages_SMD:SOT-89-3_Handsoldering
- R1, R2: footprint (none) -> Resistors_SMD:R_0805_HandSoldering
- U2: footprint Converters_DCDC_ACDC:DCDC-Conv_muRata_MGJ2 -> ENNOID:DCDC-Conv_muRata_MGJ2
Connections:
- wire segments 40 -> 41
Changed lines of the file:
@@
 $Descr A4 11693 8268
 encoding utf-8
-Sheet 5 6
+Sheet 2 7
 Title ""
 Date ""
@@
 AR Path="/5A300795/5A300C2E" Ref="FL1"  Part="1"
 AR Path="/5A331F4C/5A300C2E" Ref="FL2"  Part="1"
-F 0 "FL2" H 3850 2787 50  0000 C CNN
+F 0 "FL1" H 3850 2787 50  0000 C CNN
 F 1 "ACM4520-142-2P-T000" H 3850 2787 50  0001 C CNN
-F 2 "" V 3850 2640 50  0000 C CNN
+F 2 "ENNOID:ACM4520" V 3850 2640 50  0001 C CNN
 F 3 "" H 3850 2793 50  0001 C CNN
 	1    3850 2600
@@
 AR Path="/5A300795/5A301108" Ref="C6"  Part="1"
 AR Path="/5A331F4C/5A301108" Ref="C11"  Part="1"
-F 0 "C11" H 5015 2600 50  0000 L CNN
+F 0 "C6" H 5015 2600 50  0000 L CNN
 F 1 "1u" H 5015 2555 50  0000 L CNN
-F 2 "" H 4938 2450 50  0001 C CNN
+F 2 "Capacitors_SMD:C_0805_HandSoldering" H 4938 2450 50  0001 C CNN
 F 3 "" H 4900 2600 50  0001 C CNN
 	1    4900 2600
@@
 AR Path="/5A300795/5A301151" Ref="C5"  Part="1"
 AR Path="/5A331F4C/5A301151" Ref="C10"  Part="1"
-F 0 "C10" H 4515 2600 50  0000 L CNN
+F 0 "C5" H 4515 2600 50  0000 L CNN
 F 1 "100n" H 4515 2555 50  0000 L CNN
-F 2 "" H 4438 2450 50  0001 C CNN
+F 2 "Capacitors_SMD:C_0805_HandSoldering" H 4438 2450 50  0001 C CNN
 F 3 "" H 4400 2600 50  0001 C CNN
 	1    4400 2600
@@
 AR Path="/5A300795/5A3089F3" Ref="U2"  Part="1"
 AR Path="/5A331F4C/5A3089F3" Ref="U3"  Part="1"
-F 0 "U3" H 5700 3067 50  0000 C CNN
+F 0 "U2" H 5700 3067 50  0000 C CNN
 F 1 "MGJ2" H 5700 2976 50  0000 C CNN
-F 2 "Converters_DCDC_ACDC:DCDC-Conv_muRata_MGJ2" H 5700 2250 50  0001 C CIN
+F 2 "ENNOID:DCDC-Conv_muRata_MGJ2" H 5700 2250 50  0001 C CIN
 F 3 "https://power.murata.com/data/power/ncl/kdc_mgj2.pdf" H 5700 2600 50  0001 C CNN
 	1    5700 2600
@@
 AR Path="/5A300795/5A308BE5" Ref="C7"  Part="1"
 AR Path="/5A331F4C/5A308BE5" Ref="C12"  Part="1"
-F 0 "C12" H 6815 2350 50  0000 L CNN
+F 0 "C7" H 6815 2350 50  0000 L CNN
 F 1 "1u" H 6815 2305 50  0000 L CNN
-F 2 "" H 6738 2200 50  0001 C CNN
+F 2 "Capacitors_SMD:C_0805_HandSoldering" H 6738 2200 50  0001 C CNN
 F 3 "" H 6700 2350 50  0001 C CNN
 	1    6700 2350
@@
 AR Path="/5A300795/5A308C45" Ref="C8"  Part="1"
 AR Path="/5A331F4C/5A308C45" Ref="C13"  Part="1"
-F 0 "C13" H 6815 2850 50  0000 L CNN
+F 0 "C8" H 6815 2850 50  0000 L CNN
 F 1 "1u" H 6815 2805 50  0000 L CNN
-F 2 "" H 6738 2700 50  0001 C CNN
+F 2 "Capacitors_SMD:C_0805_HandSoldering" H 6738 2700 50  0001 C CNN
 F 3 "" H 6700 2850 50  0001 C CNN
 	1    6700 2850
@@
 	3500 2500 3650 2500
 Wire Wire Line
-	3650 2700 3500 2700
+	3650 2700 3600 2700
 Wire Wire Line
 	4050 2500 4250 2500
@@
 AR Path="/5A300795/5A30AA71" Ref="R1"  Part="1"
 AR Path="/5A331F4C/5A30AA71" Ref="R3"  Part="1"
-F 0 "R3" H 7530 2354 50  0000 R CNN
+F 0 "R1" H 7530 2354 50  0000 R CNN
 F 1 "10k" H 7530 2445 50  0000 R CNN
-F 2 "" V 7530 2400 50  0001 C CNN
+F 2 "Resistors_SMD:R_0805_HandSoldering" V 7530 2400 50  0001 C CNN
 F 3 "" H 7600 2400 50  0001 C CNN
 	1    7600 2400
@@
 AR Path="/5A300795/5A30AEBF" Ref="R2"  Part="1"
 AR Path="/5A331F4C/5A30AEBF" Ref="R4"  Part="1"
-F 0 "R4" V 8257 2600 50  0000 C CNN
+F 0 "R2" V 8257 2600 50  0000 C CNN
 F 1 "0" V 8166 2600 50  0000 C CNN
-F 2 "" V 7980 2600 50  0001 C CNN
+F 2 "Resistors_SMD:R_0805_HandSoldering" V 7980 2600 50  0001 C CNN
 F 3 "" H 8050 2600 50  0001 C CNN
 	1    8050 2600
@@
 AR Path="/5A300795/5A30AF37" Ref="C9"  Part="1"
 AR Path="/5A331F4C/5A30AF37" Ref="C14"  Part="1"
-F 0 "C14" H 8365 2950 50  0000 L CNN
+F 0 "C9" H 8365 2950 50  0000 L CNN
 F 1 "1u" H 8365 2905 50  0000 L CNN
-F 2 "" H 8288 2800 50  0001 C CNN
+F 2 "Capacitors_SMD:C_0805_HandSoldering" H 8288 2800 50  0001 C CNN
 F 3 "" H 8250 2950 50  0001 C CNN
 	1    8250 2950
@@
 AR Path="/5A300795/5A30B06B" Ref="Q1"  Part="1"
 AR Path="/5A331F4C/5A30B06B" Ref="Q2"  Part="1"
-F 0 "Q2" H 8691 2600 50  0000 L CNN
+F 0 "Q1" H 8691 2600 50  0000 L CNN
 F 1 "Q_NPN_CBE" H 8691 2555 50  0001 L CNN
-F 2 "" H 8700 2700 50  0001 C CNN
+F 2 "TO_SOT_Packages_SMD:SOT-89-3_Handsoldering" H 8700 2700 50  0001 C CNN
 F 3 "" H 8500 2600 50  0001 C CNN
 	1    8500 2600
@@
 AR Path="/5A300795/5A310D6B" Ref="D1"  Part="1"
 AR Path="/5A331F4C/5A310D6B" Ref="D2"  Part="1"
-F 0 "D2" V 7554 2929 50  0000 L CNN
-F 1 "D_Zener" V 7645 2929 50  0000 L CNN
-F 2 "" H 7600 2850 50  0001 C CNN
+F 0 "D1" V 7554 2929 50  0000 L CNN
+F 1 "MMSZ5251B" V 7645 2929 50  0000 L CNN
+F 2 "Diodes_SMD:D_SOD-123" H 7600 2850 50  0001 C CNN
 F 3 "https://en.wikipedia.org/wiki/Zener_diode" H 7600 2850 50  0001 C CNN
 	1    7600 2850
@@
 Wire Wire Line
 	7600 3100 8250 3100
+$Comp
+L power:GND #PWR036
+U 1 1 5A57221A
+P 3600 2700
+AR Path="/5A300795/5A57221A" Ref="#PWR036"  Part="1"
+AR Path="/5A331F4C/5A57221A" Ref="#PWR037"  Part="1"
+F 0 "#PWR037" H 3600 2450 50  0001 C CNN
+F 1 "GND" H 3605 2527 50  0000 C CNN
+F 2 "" H 3600 2700 50  0001 C CNN
+F 3 "" H 3600 2700 50  0001 C CNN
+	1    3600 2700
+	1    0    0    -1
+$EndComp
+Connection ~ 3600 2700
+Wire Wire Line
+	3600 2700 3500 2700
 $EndSCHEMATC

Commit message: PCB half-done
Parts:
- removed Q1: Q_NPN_CBE, TO_SOT_Packages_SMD:SOT-89-3_Handsoldering, symbol device:Q_NPN_CBE
- added Q1: Q_NPN_BCE, TO_SOT_Packages_SMD:SOT-89-3_Handsoldering, symbol device:Q_NPN_BCE
Connections:
- net labels added: +24V
Changed lines of the file:
@@
 $Descr A4 11693 8268
 encoding utf-8
-Sheet 2 7
+Sheet 4 7
 Title ""
 Date ""
@@
 AR Path="/5A300795/5A300C2E" Ref="FL1"  Part="1"
 AR Path="/5A331F4C/5A300C2E" Ref="FL2"  Part="1"
-F 0 "FL1" H 3850 2787 50  0000 C CNN
+F 0 "FL2" H 3850 2787 50  0000 C CNN
 F 1 "ACM4520-142-2P-T000" H 3850 2787 50  0001 C CNN
 F 2 "ENNOID:ACM4520" V 3850 2640 50  0001 C CNN
@@
 AR Path="/5A300795/5A301108" Ref="C6"  Part="1"
 AR Path="/5A331F4C/5A301108" Ref="C11"  Part="1"
-F 0 "C6" H 5015 2600 50  0000 L CNN
+F 0 "C11" H 5015 2600 50  0000 L CNN
 F 1 "1u" H 5015 2555 50  0000 L CNN
 F 2 "Capacitors_SMD:C_0805_HandSoldering" H 4938 2450 50  0001 C CNN
@@
 AR Path="/5A300795/5A301151" Ref="C5"  Part="1"
 AR Path="/5A331F4C/5A301151" Ref="C10"  Part="1"
-F 0 "C5" H 4515 2600 50  0000 L CNN
+F 0 "C10" H 4515 2600 50  0000 L CNN
 F 1 "100n" H 4515 2555 50  0000 L CNN
 F 2 "Capacitors_SMD:C_0805_HandSoldering" H 4438 2450 50  0001 C CNN
@@
 AR Path="/5A300795/5A3089F3" Ref="U2"  Part="1"
 AR Path="/5A331F4C/5A3089F3" Ref="U3"  Part="1"
-F 0 "U2" H 5700 3067 50  0000 C CNN
+F 0 "U3" H 5700 3067 50  0000 C CNN
 F 1 "MGJ2" H 5700 2976 50  0000 C CNN
 F 2 "ENNOID:DCDC-Conv_muRata_MGJ2" H 5700 2250 50  0001 C CIN
@@
 AR Path="/5A300795/5A308BE5" Ref="C7"  Part="1"
 AR Path="/5A331F4C/5A308BE5" Ref="C12"  Part="1"
-F 0 "C7" H 6815 2350 50  0000 L CNN
+F 0 "C12" H 6815 2350 50  0000 L CNN
 F 1 "1u" H 6815 2305 50  0000 L CNN
 F 2 "Capacitors_SMD:C_0805_HandSoldering" H 6738 2200 50  0001 C CNN
@@
 AR Path="/5A300795/5A308C45" Ref="C8"  Part="1"
 AR Path="/5A331F4C/5A308C45" Ref="C13"  Part="1"
-F 0 "C8" H 6815 2850 50  0000 L CNN
+F 0 "C13" H 6815 2850 50  0000 L CNN
 F 1 "1u" H 6815 2805 50  0000 L CNN
 F 2 "Capacitors_SMD:C_0805_HandSoldering" H 6738 2700 50  0001 C CNN
@@
 AR Path="/5A300795/5A30AA71" Ref="R1"  Part="1"
 AR Path="/5A331F4C/5A30AA71" Ref="R3"  Part="1"
-F 0 "R1" H 7530 2354 50  0000 R CNN
+F 0 "R3" H 7530 2354 50  0000 R CNN
 F 1 "10k" H 7530 2445 50  0000 R CNN
 F 2 "Resistors_SMD:R_0805_HandSoldering" V 7530 2400 50  0001 C CNN
@@
 AR Path="/5A300795/5A30AEBF" Ref="R2"  Part="1"
 AR Path="/5A331F4C/5A30AEBF" Ref="R4"  Part="1"
-F 0 "R2" V 8257 2600 50  0000 C CNN
+F 0 "R4" V 8257 2600 50  0000 C CNN
 F 1 "0" V 8166 2600 50  0000 C CNN
 F 2 "Resistors_SMD:R_0805_HandSoldering" V 7980 2600 50  0001 C CNN
@@
 AR Path="/5A300795/5A30AF37" Ref="C9"  Part="1"
 AR Path="/5A331F4C/5A30AF37" Ref="C14"  Part="1"
-F 0 "C9" H 8365 2950 50  0000 L CNN
+F 0 "C14" H 8365 2950 50  0000 L CNN
 F 1 "1u" H 8365 2905 50  0000 L CNN
 F 2 "Capacitors_SMD:C_0805_HandSoldering" H 8288 2800 50  0001 C CNN
@@
 	1    0    0    -1
 $EndComp
-$Comp
-L device:Q_NPN_CBE Q1
-U 1 1 5A30B06B
-P 8500 2600
-AR Path="/5A300795/5A30B06B" Ref="Q1"  Part="1"
-AR Path="/5A331F4C/5A30B06B" Ref="Q2"  Part="1"
-F 0 "Q1" H 8691 2600 50  0000 L CNN
-F 1 "Q_NPN_CBE" H 8691 2555 50  0001 L CNN
-F 2 "TO_SOT_Packages_SMD:SOT-89-3_Handsoldering" H 8700 2700 50  0001 C CNN
-F 3 "" H 8500 2600 50  0001 C CNN
-	1    8500 2600
-	1    0    0    -1
-$EndComp
 Wire Wire Line
 	8200 2600 8300 2600
@@
 Wire Wire Line
 	8600 3150 8600 2800
-Connection ~ 8600 2800
 Text HLabel 6950 2600 2    60   Output ~ 0
 PHASE
@@
 AR Path="/5A300795/5A310D6B" Ref="D1"  Part="1"
 AR Path="/5A331F4C/5A310D6B" Ref="D2"  Part="1"
-F 0 "D1" V 7554 2929 50  0000 L CNN
+F 0 "D2" V 7554 2929 50  0000 L CNN
 F 1 "MMSZ5251B" V 7645 2929 50  0000 L CNN
 F 2 "Diodes_SMD:D_SOD-123" H 7600 2850 50  0001 C CNN
@@
 Wire Wire Line
 	3600 2700 3500 2700
+$Comp
+L power:+24V #PWR011
+U 1 1 5A415966
+P 3600 2500
+AR Path="/5A331F4C/5A415966" Ref="#PWR011"  Part="1"
+AR Path="/5A300795/5A415966" Ref="#PWR010"  Part="1"
+F 0 "#PWR011" H 3600 2350 50  0001 C CNN
+F 1 "+24V" H 3615 2673 50  0000 C CNN
+F 2 "" H 3600 2500 50  0001 C CNN
+F 3 "" H 3600 2500 50  0001 C CNN
+	1    3600 2500
+	1    0    0    -1
+$EndComp
+$Comp
+L device:Q_NPN_BCE Q1
+U 1 1 5A34237B
+P 8500 2600
+AR Path="/5A331F4C/5A34237B" Ref="Q1"  Part="1"
+AR Path="/5A300795/5A34237B" Ref="Q2"  Part="1"
+F 0 "Q1" H 8691 2646 50  0000 L CNN
+F 1 "Q_NPN_BCE" H 8691 2555 50  0000 L CNN
+F 2 "TO_SOT_Packages_SMD:SOT-89-3_Handsoldering" H 8700 2700 50  0001 C CNN
+F 3 "" H 8500 2600 50  0001 C CNN
+	1    8500 2600
+	1    0    0    -1
+$EndComp
+Connection ~ 8600 2800
 $EndSCHEMATC

Commit message: PCB completed with readme update
Parts:
- removed FL1: ACM4520-142-2P-T000, ENNOID:ACM4520, symbol device:EMI_Filter_LL
- added FL2: ACM4520, ENNOID:ACM4520, symbol ENNOID:ACM4520
Connections:
- wire segments 41 -> 42
Changed lines of the file:
@@
 Comment4 ""
 $EndDescr
-$Comp
-L device:EMI_Filter_LL FL1
-U 1 1 5A300C2E
-P 3850 2600
-AR Path="/5A300795/5A300C2E" Ref="FL1"  Part="1"
-AR Path="/5A331F4C/5A300C2E" Ref="FL2"  Part="1"
-F 0 "FL2" H 3850 2787 50  0000 C CNN
-F 1 "ACM4520-142-2P-T000" H 3850 2787 50  0001 C CNN
-F 2 "ENNOID:ACM4520" V 3850 2640 50  0001 C CNN
-F 3 "" H 3850 2793 50  0001 C CNN
-	1    3850 2600
-	1    0    0    -1
-$EndComp
 Text HLabel 3500 2500 0    60   Input ~ 0
 VCC_IN
@@
 Wire Wire Line
 	4400 2750 4900 2750
-Wire Wire Line
-	3500 2500 3650 2500
 Wire Wire Line
 	3650 2700 3600 2700
@@
 $EndComp
 Connection ~ 8600 2800
+$Comp
+L ENNOID:ACM4520 FL2
+U 1 1 5A376789
+P 3850 2600
+AR Path="/5A331F4C/5A376789" Ref="FL2"  Part="1"
+AR Path="/5A300795/5A376789" Ref="FL1"  Part="1"
+F 0 "FL2" H 3850 2878 50  0000 C CNN
+F 1 "ACM4520" H 3850 2787 50  0000 C CNN
+F 2 "ENNOID:ACM4520" H 3850 2787 50  0001 C CNN
+F 3 "" V 3850 2640 50  0000 C CNN
+	1    3850 2600
+	1    0    0    -1
+$EndComp
+Wire Wire Line
+	3650 2500 3600 2500
+Wire Wire Line
+	3600 2500 3500 2500
+Connection ~ 3600 2500
 $EndSCHEMATC
