File: PCB/GD.sch (KiCad schematic (older format))
At the start: 28 parts, among them Q3 BSS138, U4 1ED020I12-F2, U5 IXD-609

Commit message: .gitignore for kicad
Parts:
- added D?: D_Zener, symbol device:D_Zener
Connections:
- wire segments 115 -> 116

Commit message: Schematics & footprints completed
Ready for PCBnew
Parts:
- removed D?: D_Zener, symbol device:D_Zener
- added D10: D, Diodes_SMD:D_SMA_Handsoldering, symbol device:D
- C15, C16, C17, C18, C19, C22, C23, C25: footprint (none) -> Capacitors_SMD:C_0805_HandSoldering
- C21: footprint (none) -> Capacitors_SMD:C_1206_HandSoldering
- C31: value 4.7u -> 100n; footprint (none) -> Capacitors_SMD:C_0805_HandSoldering
- C35: footprint (none) -> Resistors_SMD:R_1210_HandSoldering
- D3, D5: footprint (none) -> Diodes_SMD:D_SOD-123
- D4: footprint (none) -> Diodes_THT:D_DO-41_SOD81_P12.70mm_Horizontal
- Q3: value BSS138 -> 2N7002K-7
- R10, R15, R5, R6, R7, R8, R9: footprint (none) -> Resistors_SMD:R_0805_HandSoldering
- R11, R12, R13, R14: footprint (none) -> Resistors_SMD:R_MELF_MMB-0207
- U4: footprint Housings_PG-DSO -15-16 Infineon -> Housings_SOIC:SOIC-16W_7.5x10.3mm_Pitch1.27mm
Changed lines of the file:
@@
 $Descr A4 11693 8268
 encoding utf-8
-Sheet 3 6
+Sheet 5 7
 Title ""
 Date ""
@@
 AR Path="/5A33279F/5A30E40F" Ref="#PWR09"  Part="1"
 AR Path="/5A340028/5A30E40F" Ref="#PWR016"  Part="1"
-F 0 "#PWR09" H 1700 2300 50  0001 C CNN
+F 0 "#PWR016" H 1700 2300 50  0001 C CNN
 F 1 "+5V" H 1715 2623 50  0000 C CNN
 F 2 "" H 1700 2450 50  0001 C CNN
@@
 AR Path="/5A340028/5A30F6FF" Ref="#PWR014"  Part="1"
 AR Path="/5A33279F/5A30F6FF" Ref="#PWR07"  Part="1"
-F 0 "#PWR07" H 1350 4900 50  0001 C CNN
+F 0 "#PWR014" H 1350 4900 50  0001 C CNN
 F 1 "GND" H 1355 4977 50  0000 C CNN
 F 2 "" H 1350 5150 50  0001 C CNN
@@
 F 0 "U4" H 3700 3867 50  0000 C CNN
 F 1 "1ED020I12-F2" H 3700 3776 50  0000 C CNN
-F 2 "Housings_PG-DSO -15-16 Infineon" H 3700 2700 50  0001 C CIN
+F 2 "Housings_SOIC:SOIC-16W_7.5x10.3mm_Pitch1.27mm" H 3700 2700 50  0001 C CIN
 F 3 "https://www.infineon.com/dgdl/Datasheet_1ED020I12-F2_V2_final.pdf?folderId=db3a30432b16d655012b33fafdac11e2&fileId=db3a304330f68606013122ce5f3649cb" H 3700 3600 50  0001 C CNN
 	1    3700 3200
@@
 AR Path="/5A33279F/5A3110EF" Ref="#PWR013"  Part="1"
 AR Path="/5A340028/5A3110EF" Ref="#PWR020"  Part="1"
-F 0 "#PWR013" H 3200 3750 50  0001 C CNN
+F 0 "#PWR020" H 3200 3750 50  0001 C CNN
 F 1 "GND" H 3205 3827 50  0000 C CNN
 F 2 "" H 3200 4000 50  0001 C CNN
@@
 F 0 "C16" H 2965 3796 50  0000 L CNN
 F 1 "100n" H 2965 3705 50  0000 L CNN
-F 2 "" H 2888 3600 50  0001 C CNN
+F 2 "Capacitors_SMD:C_0805_HandSoldering" H 2888 3600 50  0001 C CNN
 F 3 "" H 2850 3750 50  0001 C CNN
 	1    2850 3750
@@
 AR Path="/5A33279F/5A3112E7" Ref="#PWR012"  Part="1"
 AR Path="/5A340028/5A3112E7" Ref="#PWR019"  Part="1"
-F 0 "#PWR012" H 2850 3750 50  0001 C CNN
+F 0 "#PWR019" H 2850 3750 50  0001 C CNN
 F 1 "GND" H 2855 3827 50  0000 C CNN
 F 2 "" H 2850 4000 50  0001 C CNN
@@
 F 0 "R9" H 2420 2896 50  0000 L CNN
 F 1 "10k" H 2420 2805 50  0000 L CNN
-F 2 "" V 2280 2850 50  0001 C CNN
+F 2 "Resistors_SMD:R_0805_HandSoldering" V 2280 2850 50  0001 C CNN
 F 3 "" H 2350 2850 50  0001 C CNN
 	1    2350 2850
@@
 F 0 "R7" H 2120 2896 50  0000 L CNN
 F 1 "10k" H 2120 2805 50  0000 L CNN
-F 2 "" V 1980 2850 50  0001 C CNN
+F 2 "Resistors_SMD:R_0805_HandSoldering" V 1980 2850 50  0001 C CNN
 F 3 "" H 2050 2850 50  0001 C CNN
 	1    2050 2850
@@
 F 0 "R6" V 943 3400 50  0000 C CNN
 F 1 "1k" V 1034 3400 50  0000 C CNN
-F 2 "" V 1080 3400 50  0001 C CNN
+F 2 "Resistors_SMD:R_0805_HandSoldering" V 1080 3400 50  0001 C CNN
 F 3 "" H 1150 3400 50  0001 C CNN
 	1    1150 3400
@@
 F 0 "R8" H 2030 3704 50  0000 R CNN
 F 1 "1k" H 2030 3795 50  0000 R CNN
-F 2 "" V 2030 3750 50  0001 C CNN
+F 2 "Resistors_SMD:R_0805_HandSoldering" V 2030 3750 50  0001 C CNN
 F 3 "" H 2100 3750 50  0001 C CNN
 	1    2100 3750
@@
 F 0 "C15" H 2515 3796 50  0000 L CNN
 F 1 "100n" H 2515 3705 50  0000 L CNN
-F 2 "" H 2438 3600 50  0001 C CNN
+F 2 "Capacitors_SMD:C_0805_HandSoldering" H 2438 3600 50  0001 C CNN
 F 3 "" H 2400 3750 50  0001 C CNN
 	1    2400 3750
@@
 AR Path="/5A33279F/5A3155E3" Ref="#PWR011"  Part="1"
 AR Path="/5A340028/5A3155E3" Ref="#PWR018"  Part="1"
-F 0 "#PWR011" H 2400 3750 50  0001 C CNN
+F 0 "#PWR018" H 2400 3750 50  0001 C CNN
 F 1 "GND" H 2405 3827 50  0000 C CNN
 F 2 "" H 2400 4000 50  0001 C CNN
@@
 AR Path="/5A33279F/5A3155FC" Ref="#PWR010"  Part="1"
 AR Path="/5A340028/5A3155FC" Ref="#PWR017"  Part="1"
-F 0 "#PWR010" H 2100 3750 50  0001 C CNN
+F 0 "#PWR017" H 2100 3750 50  0001 C CNN
 F 1 "GND" H 2105 3827 50  0000 C CNN
 F 2 "" H 2100 4000 50  0001 C CNN
@@
 F 0 "R5" V 893 3750 50  0000 C CNN
 F 1 "1k" V 984 3750 50  0000 C CNN
-F 2 "" V 1030 3750 50  0001 C CNN
+F 2 "Resistors_SMD:R_0805_HandSoldering" V 1030 3750 50  0001 C CNN
 F 3 "" H 1100 3750 50  0001 C CNN
 	1    1100 3750
 	0    1    1    0
 $EndComp
-Wire Wire Line
-	900  3750 950  3750
 $Comp
 L power:GND #PWR08
@@
 AR Path="/5A33279F/5A3180B4" Ref="#PWR08"  Part="1"
 AR Path="/5A340028/5A3180B4" Ref="#PWR015"  Part="1"
-F 0 "#PWR08" H 1600 3750 50  0001 C CNN
+F 0 "#PWR015" H 1600 3750 50  0001 C CNN
 F 1 "GND" H 1605 3827 50  0000 C CNN
 F 2 "" H 1600 4000 50  0001 C CNN
@@
 AR Path="/5A340028/5A318143" Ref="Q4"  Part="1"
 F 0 "Q3" H 1705 3796 50  0000 L CNN
-F 1 "BSS138" H 1705 3705 50  0000 L CNN
+F 1 "2N7002K-7" H 1705 3705 50  0000 L CNN
 F 2 "TO_SOT_Packages_SMD:SOT-23" H 1700 3675 50  0001 L CIN
-F 3 "https://www.fairchildsemi.com/datasheets/BS/BSS138.pdf" H 1500 3750 50  0001 L CNN
+F 3 "" H 1500 3750 50  0001 L CNN
 	1    1500 3750
 	1    0    0    -1
@@
 F 0 "C17" H 4615 2696 50  0000 L CNN
 F 1 "100n" H 4615 2605 50  0000 L CNN
-F 2 "" H 4538 2500 50  0001 C CNN
+F 2 "Capacitors_SMD:C_0805_HandSoldering" H 4538 2500 50  0001 C CNN
 F 3 "" H 4500 2650 50  0001 C CNN
 	1    4500 2650
@@
 F 0 "C18" H 4615 3846 50  0000 L CNN
 F 1 "100n" H 4615 3755 50  0000 L CNN
-F 2 "" H 4538 3650 50  0001 C CNN
+F 2 "Capacitors_SMD:C_0805_HandSoldering" H 4538 3650 50  0001 C CNN
 F 3 "" H 4500 3800 50  0001 C CNN
 	1    4500 3800
@@
 F 0 "R10" V 5743 2900 50  0000 C CNN
 F 1 "10k" V 5834 2900 50  0000 C CNN
-F 2 "" V 5880 2900 50  0001 C CNN
+F 2 "Resistors_SMD:R_0805_HandSoldering" V 5880 2900 50  0001 C CNN
 F 3 "" H 5950 2900 50  0001 C CNN
 	1    5950 2900
@@
 F 0 "C19" H 5715 3696 50  0000 L CNN
 F 1 "DNP" H 5715 3605 50  0000 L CNN
-F 2 "" H 5638 3500 50  0001 C CNN
+F 2 "Capacitors_SMD:C_0805_HandSoldering" H 5638 3500 50  0001 C CNN
 F 3 "" H 5600 3650 50  0001 C CNN
 	1    5600 3650
@@
 F 0 "D3" V 5054 3729 50  0000 L CNN
 F 1 "D_Zener" V 5145 3729 50  0000 L CNN
-F 2 "" H 5100 3650 50  0001 C CNN
+F 2 "Diodes_SMD:D_SOD-123" H 5100 3650 50  0001 C CNN
 F 3 "https://en.wikipedia.org/wiki/Zener_diode" H 5100 3650 50  0001 C CNN
 	1    5100 3650
@@
 F 0 "D5" H 6750 3116 50  0000 C CNN
 F 1 "D_Zener" H 6750 3025 50  0000 C CNN
-F 2 "" H 6750 2900 50  0001 C CNN
+F 2 "Diodes_SMD:D_SOD-123" H 6750 2900 50  0001 C CNN
 F 3 "https://en.wikipedia.org/wiki/Zener_diode" H 6750 2900 50  0001 C CNN
 	1    6750 2900
@@
 F 0 "D4" H 6350 2684 50  0000 C CNN
 F 1 "D" H 6350 2775 50  0000 C CNN
-F 2 "" H 6350 2900 50  0001 C CNN
+F 2 "Diodes_THT:D_DO-41_SOD81_P12.70mm_Horizontal" H 6350 2900 50  0001 C CNN
 F 3 "" H 6350 2900 50  0001 C CNN
 	1    6350 2900
@@
 F 0 "C21" H 8815 3796 50  0000 L CNN
 F 1 "4.7u" H 8815 3705 50  0000 L CNN
-F 2 "" H 8738 3600 50  0001 C CNN
+F 2 "Capacitors_SMD:C_1206_HandSoldering" H 8738 3600 50  0001 C CNN
 F 3 "" H 8700 3750 50  0001 C CNN
 	1    8700 3750
@@
 AR Path="/5A33279F/5A35FF7D" Ref="C20"  Part="1"
 F 0 "C20" H 7215 3796 50  0000 L CNN
-F 1 "4.7u" H 7215 3705 50  0000 L CNN
-F 2 "" H 7138 3600 50  0001 C CNN
+F 1 "100n" H 7215 3705 50  0000 L CNN
+F 2 "Capacitors_SMD:C_0805_HandSoldering" H 7138 3600 50  0001 C CNN
 F 3 "" H 7100 3750 50  0001 C CNN
 	1    7100 3750
@@
 F 0 "R11" V 9357 1800 50  0000 C CNN
 F 1 "DND" V 9266 1800 50  0000 C CNN
-F 2 "" V 9080 1800 50  0001 C CNN
+F 2 "Resistors_SMD:R_MELF_MMB-0207" V 9080 1800 50  0001 C CNN
 F 3 "" H 9150 1800 50  0001 C CNN
 	1    9150 1800
@@
 F 0 "R12" V 9357 2150 50  0000 C CNN
 F 1 "DND" V 9266 2150 50  0000 C CNN
-F 2 "" V 9080 2150 50  0001 C CNN
+F 2 "Resistors_SMD:R_MELF_MMB-0207" V 9080 2150 50  0001 C CNN
 F 3 "" H 9150 2150 50  0001 C CNN
 	1    9150 2150
@@
 F 0 "R13" V 9357 2900 50  0000 C CNN
 F 1 "20" V 9266 2900 50  0000 C CNN
-F 2 "" V 9080 2900 50  0001 C CNN
+F 2 "Resistors_SMD:R_MELF_MMB-0207" V 9080 2900 50  0001 C CNN
 F 3 "" H 9150 2900 50  0001 C CNN
 	1    9150 2900
@@
 F 0 "R14" V 9357 3200 50  0000 C CNN
 F 1 "20" V 9266 3200 50  0000 C CNN
-F 2 "" V 9080 3200 50  0001 C CNN
+F 2 "Resistors_SMD:R_MELF_MMB-0207" V 9080 3200 50  0001 C CNN
 F 3 "" H 9150 3200 50  0001 C CNN
 	1    9150 3200
@@
 F 0 "R15" H 10270 3396 50  0000 L CNN
 F 1 "47k" H 10270 3305 50  0000 L CNN
-F 2 "" V 10130 3350 50  0001 C CNN
+F 2 "Resistors_SMD:R_0805_HandSoldering" V 10130 3350 50  0001 C CNN
 F 3 "" H 10200 3350 50  0001 C CNN
 	1    10200 3350
@@
 F 0 "C25" H 10765 3396 50  0000 L CNN
 F 1 "DNP" H 10765 3305 50  0000 L CNN
-F 2 "" H 10688 3200 50  0001 C CNN
+F 2 "Capacitors_SMD:C_0805_HandSoldering" H 10688 3200 50  0001 C CNN
 F 3 "" H 10650 3350 50  0001 C CNN
 	1    10650 3350
@@
 F 0 "C22" V 9598 3500 50  0000 C CNN
 F 1 "10n" V 9689 3500 50  0000 C CNN
-F 2 "" H 9888 3350 50  0001 C CNN
+F 2 "Capacitors_SMD:C_0805_HandSoldering" H 9888 3350 50  0001 C CNN
 F 3 "" H 9850 3500 50  0001 C CNN
 	1    9850 3500
@@
 F 0 "C23" V 9598 3950 50  0000 C CNN
 F 1 "100n" V 9689 3950 50  0000 C CNN
-F 2 "" H 9888 3800 50  0001 C CNN
+F 2 "Capacitors_SMD:C_0805_HandSoldering" H 9888 3800 50  0001 C CNN
 F 3 "" H 9850 3950 50  0001 C CNN
 	1    9850 3950
@@
 F 0 "C24" V 9598 4350 50  0000 C CNN
 F 1 "10u" V 9689 4350 50  0000 C CNN
-F 2 "" H 9888 4200 50  0001 C CNN
+F 2 "Resistors_SMD:R_1210_HandSoldering" H 9888 4200 50  0001 C CNN
 F 3 "" H 9850 4350 50  0001 C CNN
 	1    9850 4350
@@
 Wire Wire Line
 	8900 3200 9000 3200
-$Comp
-L device:D_Zener D?
-U 1 1 5A38B834
-P 8900 2700
-F 0 "D?" H 8900 2916 50  0000 C CNN
-F 1 "D_Zener" H 8900 2825 50  0000 C CNN
-F 2 "" H 8900 2700 50  0001 C CNN
-F 3 "https://en.wikipedia.org/wiki/Zener_diode" H 8900 2700 50  0001 C CNN
-	1    8900 2700
-	0    1    1    0
-$EndComp
-Wire Wire Line
-	8900 2850 8900 2900
+Wire Wire Line
+	8900 2650 8900 2900
 Connection ~ 8900 2900
 Wire Wire Line
@@
 Connection ~ 8900 2150
 Wire Wire Line
-	8900 2150 8900 2550
+	8900 2150 8900 2350
+$Comp
+L device:D D10
+U 1 1 5A3ACFE6
+P 8900 2500
+AR Path="/5A33279F/5A3ACFE6" Ref="D10"  Part="1"
+AR Path="/5A340028/5A3ACFE6" Ref="D11"  Part="1"
+F 0 "D10" H 8900 2284 50  0000 C CNN
+F 1 "D" H 8900 2375 50  0000 C CNN
+F 2 "Diodes_SMD:D_SMA_Handsoldering" H 8900 2500 50  0001 C CNN
+F 3 "" H 8900 2500 50  0001 C CNN
+	1    8900 2500
+	0    -1   -1   0
+$EndComp
+Wire Wire Line
+	900  3750 950  3750
 $EndSCHEMATC

Commit message: PCB half-done
Parts:
- added R45: DNP, Resistors_SMD:R_0805_HandSoldering, symbol device:R
Connections:
- wire segments 116 -> 127

Commit message: Minor changes
Connections:
- wire segments 127 -> 128
Changed lines of the file:
@@
 $Descr A4 11693 8268
 encoding utf-8
-Sheet 3 7
+Sheet 5 7
 Title ""
 Date ""
@@
 	8500 3300 8700 3300
 Connection ~ 8500 3300
-Connection ~ 8700 3300
-Wire Wire Line
-	8700 3300 8700 3600
 $Comp
 L device:R R15
@@
 	1600 4000 2100 4000
 Connection ~ 2100 4000
+Wire Wire Line
+	8550 3200 8550 3600
+Wire Wire Line
+	8550 3600 8700 3600
+Connection ~ 8550 3200
 $EndSCHEMATC
