File: PCB/GD.sch (KiCad schematic (older format))
At the start: 30 parts, among them Q3 2N7002K-7, U4 1ED020I12-F2, U5 IXD-609

Commit message: Small updates
Parts:
- R8: value 1k -> 47k
Changed lines of the file:
@@
 AR Path="/5A33279F/5A30E40F" Ref="#PWR09"  Part="1"
 AR Path="/5A340028/5A30E40F" Ref="#PWR016"  Part="1"
-F 0 "#PWR09" H 1700 2300 50  0001 C CNN
+F 0 "#PWR016" H 1700 2300 50  0001 C CNN
 F 1 "+5V" H 1715 2623 50  0000 C CNN
 F 2 "" H 1700 2450 50  0001 C CNN
@@
 AR Path="/5A340028/5A30F6FF" Ref="#PWR014"  Part="1"
 AR Path="/5A33279F/5A30F6FF" Ref="#PWR07"  Part="1"
-F 0 "#PWR07" H 1350 4900 50  0001 C CNN
+F 0 "#PWR014" H 1350 4900 50  0001 C CNN
 F 1 "GND" H 1355 4977 50  0000 C CNN
 F 2 "" H 1350 5150 50  0001 C CNN
@@
 AR Path="/5A33279F/5A311090" Ref="U4"  Part="1"
 AR Path="/5A340028/5A311090" Ref="U6"  Part="1"
-F 0 "U4" H 3700 3867 50  0000 C CNN
+F 0 "U6" H 3700 3867 50  0000 C CNN
 F 1 "1ED020I12-F2" H 3700 3776 50  0000 C CNN
 F 2 "Housings_SOIC:SOIC-16W_7.5x10.3mm_Pitch1.27mm" H 3700 2700 50  0001 C CIN
@@
 AR Path="/5A33279F/5A3111D8" Ref="C16"  Part="1"
 AR Path="/5A340028/5A3111D8" Ref="C27"  Part="1"
-F 0 "C16" H 2965 3796 50  0000 L CNN
+F 0 "C27" H 2965 3796 50  0000 L CNN
 F 1 "100n" H 2965 3705 50  0000 L CNN
 F 2 "Capacitors_SMD:C_0805_HandSoldering" H 2888 3600 50  0001 C CNN
@@
 AR Path="/5A33279F/5A311468" Ref="R9"  Part="1"
 AR Path="/5A340028/5A311468" Ref="R20"  Part="1"
-F 0 "R9" H 2420 2896 50  0000 L CNN
+F 0 "R20" H 2420 2896 50  0000 L CNN
 F 1 "10k" H 2420 2805 50  0000 L CNN
 F 2 "Resistors_SMD:R_0805_HandSoldering" V 2280 2850 50  0001 C CNN
@@
 AR Path="/5A33279F/5A311627" Ref="R7"  Part="1"
 AR Path="/5A340028/5A311627" Ref="R18"  Part="1"
-F 0 "R7" H 2120 2896 50  0000 L CNN
+F 0 "R18" H 2120 2896 50  0000 L CNN
 F 1 "10k" H 2120 2805 50  0000 L CNN
 F 2 "Resistors_SMD:R_0805_HandSoldering" V 1980 2850 50  0001 C CNN
@@
 AR Path="/5A33279F/5A31375C" Ref="R6"  Part="1"
 AR Path="/5A340028/5A31375C" Ref="R17"  Part="1"
-F 0 "R6" V 943 3400 50  0000 C CNN
+F 0 "R17" V 943 3400 50  0000 C CNN
 F 1 "1k" V 1034 3400 50  0000 C CNN
 F 2 "Resistors_SMD:R_0805_HandSoldering" V 1080 3400 50  0001 C CNN
@@
 AR Path="/5A33279F/5A314867" Ref="R8"  Part="1"
 AR Path="/5A340028/5A314867" Ref="R19"  Part="1"
-F 0 "R8" H 2030 3704 50  0000 R CNN
-F 1 "1k" H 2030 3795 50  0000 R CNN
+F 0 "R19" H 2030 3704 50  0000 R CNN
+F 1 "47k" H 2030 3795 50  0000 R CNN
 F 2 "Resistors_SMD:R_0805_HandSoldering" V 2030 3750 50  0001 C CNN
 F 3 "" H 2100 3750 50  0001 C CNN
@@
 AR Path="/5A33279F/5A3148BE" Ref="C15"  Part="1"
 AR Path="/5A340028/5A3148BE" Ref="C26"  Part="1"
-F 0 "C15" H 2515 3796 50  0000 L CNN
+F 0 "C26" H 2515 3796 50  0000 L CNN
 F 1 "100n" H 2515 3705 50  0000 L CNN
 F 2 "Capacitors_SMD:C_0805_HandSoldering" H 2438 3600 50  0001 C CNN
@@
 AR Path="/5A33279F/5A316921" Ref="R5"  Part="1"
 AR Path="/5A340028/5A316921" Ref="R16"  Part="1"
-F 0 "R5" V 893 3750 50  0000 C CNN
+F 0 "R16" V 893 3750 50  0000 C CNN
 F 1 "1k" V 984 3750 50  0000 C CNN
 F 2 "Resistors_SMD:R_0805_HandSoldering" V 1030 3750 50  0001 C CNN
@@
 AR Path="/5A33279F/5A3180B4" Ref="#PWR08"  Part="1"
 AR Path="/5A340028/5A3180B4" Ref="#PWR015"  Part="1"
-F 0 "#PWR08" H 1600 3750 50  0001 C CNN
+F 0 "#PWR015" H 1600 3750 50  0001 C CNN
 F 1 "GND" H 1605 3827 50  0000 C CNN
 F 2 "" H 1600 4000 50  0001 C CNN
@@
 AR Path="/5A33279F/5A318143" Ref="Q3"  Part="1"
 AR Path="/5A340028/5A318143" Ref="Q4"  Part="1"
-F 0 "Q3" H 1705 3796 50  0000 L CNN
+F 0 "Q4" H 1705 3796 50  0000 L CNN
 F 1 "2N7002K-7" H 1705 3705 50  0000 L CNN
 F 2 "TO_SOT_Packages_SMD:SOT-23" H 1700 3675 50  0001 L CIN
@@
 AR Path="/5A33279F/5A31BF02" Ref="C17"  Part="1"
 AR Path="/5A340028/5A31BF02" Ref="C28"  Part="1"
-F 0 "C17" H 4915 2696 50  0000 L CNN
+F 0 "C28" H 4915 2696 50  0000 L CNN
 F 1 "100n" H 4915 2605 50  0000 L CNN
 F 2 "Capacitors_SMD:C_0805_HandSoldering" H 4838 2500 50  0001 C CNN
@@
 AR Path="/5A33279F/5A31BF58" Ref="C18"  Part="1"
 AR Path="/5A340028/5A31BF58" Ref="C29"  Part="1"
-F 0 "C18" H 4915 3846 50  0000 L CNN
+F 0 "C29" H 4915 3846 50  0000 L CNN
 F 1 "100n" H 4915 3755 50  0000 L CNN
 F 2 "Capacitors_SMD:C_0805_HandSoldering" H 4838 3650 50  0001 C CNN
@@
 AR Path="/5A33279F/5A324B24" Ref="R10"  Part="1"
 AR Path="/5A340028/5A324B24" Ref="R21"  Part="1"
-F 0 "R10" V 5843 2900 50  0000 C CNN
+F 0 "R21" V 5843 2900 50  0000 C CNN
 F 1 "10k" V 5934 2900 50  0000 C CNN
 F 2 "Resistors_SMD:R_0805_HandSoldering" V 5980 2900 50  0001 C CNN
@@
 AR Path="/5A33279F/5A324960" Ref="C19"  Part="1"
 AR Path="/5A340028/5A324960" Ref="C30"  Part="1"
-F 0 "C19" H 5965 3696 50  0000 L CNN
+F 0 "C30" H 5965 3696 50  0000 L CNN
 F 1 "DNP" H 5965 3605 50  0000 L CNN
 F 2 "Capacitors_SMD:C_0805_HandSoldering" H 5888 3500 50  0001 C CNN
@@
 AR Path="/5A33279F/5A32EFBE" Ref="D3"  Part="1"
 AR Path="/5A340028/5A32EFBE" Ref="D6"  Part="1"
-F 0 "D3" V 5254 3729 50  0000 L CNN
+F 0 "D6" V 5254 3729 50  0000 L CNN
 F 1 "D_Zener" V 5345 3729 50  0000 L CNN
 F 2 "Diodes_SMD:D_SOD-123" H 5300 3650 50  0001 C CNN
@@
 AR Path="/5A33279F/5A331B2A" Ref="D5"  Part="1"
 AR Path="/5A340028/5A331B2A" Ref="D8"  Part="1"
-F 0 "D5" H 6750 3116 50  0000 C CNN
+F 0 "D8" H 6750 3116 50  0000 C CNN
 F 1 "D_Zener" H 6750 3025 50  0000 C CNN
 F 2 "Diodes_SMD:D_SOD-123" H 6750 2900 50  0001 C CNN
@@
 AR Path="/5A33279F/5A331C03" Ref="D4"  Part="1"
 AR Path="/5A340028/5A331C03" Ref="D7"  Part="1"
-F 0 "D4" H 6400 2684 50  0000 C CNN
+F 0 "D7" H 6400 2684 50  0000 C CNN
 F 1 "D" H 6400 2775 50  0000 C CNN
 F 2 "Diodes_THT:D_DO-41_SOD81_P12.70mm_Horizontal" H 6400 2900 50  0001 C CNN
@@
 AR Path="/5A33279F/5A3491F7" Ref="U5"  Part="1"
 AR Path="/5A340028/5A3491F7" Ref="U7"  Part="1"
-F 0 "U5" H 7950 3867 50  0000 C CNN
+F 0 "U7" H 7950 3867 50  0000 C CNN
 F 1 "IXD-609" H 7950 3776 50  0000 C CNN
 F 2 "Housings_SOIC:SOIC-8_3.9x4.9mm_Pitch1.27mm" H 7950 3050 50  0001 C CIN
@@
 AR Path="/5A33279F/5A35FE12" Ref="C21"  Part="1"
 AR Path="/5A340028/5A35FE12" Ref="C32"  Part="1"
-F 0 "C21" H 8815 3796 50  0000 L CNN
+F 0 "C32" H 8815 3796 50  0000 L CNN
 F 1 "4.7u" H 8815 3705 50  0000 L CNN
 F 2 "Capacitors_SMD:C_1206_HandSoldering" H 8738 3600 50  0001 C CNN
@@
 AR Path="/5A340028/5A35FF7D" Ref="C31"  Part="1"
 AR Path="/5A33279F/5A35FF7D" Ref="C20"  Part="1"
-F 0 "C20" H 7215 3796 50  0000 L CNN
+F 0 "C31" H 7215 3796 50  0000 L CNN
 F 1 "100n" H 7215 3705 50  0000 L CNN
 F 2 "Capacitors_SMD:C_0805_HandSoldering" H 7138 3600 50  0001 C CNN
@@
 AR Path="/5A33279F/5A367F6F" Ref="R11"  Part="1"
 AR Path="/5A340028/5A367F6F" Ref="R22"  Part="1"
-F 0 "R11" V 9357 1800 50  0000 C CNN
+F 0 "R22" V 9357 1800 50  0000 C CNN
 F 1 "DND" V 9266 1800 50  0000 C CNN
 F 2 "Resistors_SMD:R_MELF_MMB-0207" V 9080 1800 50  0001 C CNN
@@
 AR Path="/5A33279F/5A3681D4" Ref="R12"  Part="1"
 AR Path="/5A340028/5A3681D4" Ref="R23"  Part="1"
-F 0 "R12" V 9357 2150 50  0000 C CNN
+F 0 "R23" V 9357 2150 50  0000 C CNN
 F 1 "DND" V 9266 2150 50  0000 C CNN
 F 2 "Resistors_SMD:R_MELF_MMB-0207" V 9080 2150 50  0001 C CNN
@@
 AR Path="/5A33279F/5A368218" Ref="R13"  Part="1"
 AR Path="/5A340028/5A368218" Ref="R24"  Part="1"
-F 0 "R13" V 9357 2900 50  0000 C CNN
+F 0 "R24" V 9357 2900 50  0000 C CNN
 F 1 "20" V 9266 2900 50  0000 C CNN
 F 2 "Resistors_SMD:R_MELF_MMB-0207" V 9080 2900 50  0001 C CNN
@@
 AR Path="/5A33279F/5A3682D4" Ref="R14"  Part="1"
 AR Path="/5A340028/5A3682D4" Ref="R25"  Part="1"
-F 0 "R14" V 9357 3200 50  0000 C CNN
+F 0 "R25" V 9357 3200 50  0000 C CNN
 F 1 "20" V 9266 3200 50  0000 C CNN
 F 2 "Resistors_SMD:R_MELF_MMB-0207" V 9080 3200 50  0001 C CNN
@@
 AR Path="/5A33279F/5A380EE3" Ref="R15"  Part="1"
 AR Path="/5A340028/5A380EE3" Ref="R26"  Part="1"
-F 0 "R15" H 10270 3396 50  0000 L CNN
+F 0 "R26" H 10270 3396 50  0000 L CNN
 F 1 "47k" H 10270 3305 50  0000 L CNN
 F 2 "Resistors_SMD:R_0805_HandSoldering" V 10130 3350 50  0001 C CNN
@@
 AR Path="/5A33279F/5A380FEC" Ref="C25"  Part="1"
 AR Path="/5A340028/5A380FEC" Ref="C36"  Part="1"
-F 0 "C25" H 10765 3396 50  0000 L CNN
+F 0 "C36" H 10765 3396 50  0000 L CNN
 F 1 "DNP" H 10765 3305 50  0000 L CNN
 F 2 "Capacitors_SMD:C_0805_HandSoldering" H 10688 3200 50  0001 C CNN
@@
 AR Path="/5A33279F/5A38B1D4" Ref="C22"  Part="1"
 AR Path="/5A340028/5A38B1D4" Ref="C33"  Part="1"
-F 0 "C22" V 9598 3500 50  0000 C CNN
+F 0 "C33" V 9598 3500 50  0000 C CNN
 F 1 "10n" V 9689 3500 50  0000 C CNN
 F 2 "Capacitors_SMD:C_0805_HandSoldering" H 9888 3350 50  0001 C CNN
@@
 AR Path="/5A33279F/5A38B25E" Ref="C23"  Part="1"
 AR Path="/5A340028/5A38B25E" Ref="C34"  Part="1"
-F 0 "C23" V 9598 3950 50  0000 C CNN
+F 0 "C34" V 9598 3950 50  0000 C CNN
 F 1 "100n" V 9689 3950 50  0000 C CNN
 F 2 "Capacitors_SMD:C_0805_HandSoldering" H 9888 3800 50  0001 C CNN
@@
 AR Path="/5A340028/5A38B2B8" Ref="C35"  Part="1"
 AR Path="/5A33279F/5A38B2B8" Ref="C24"  Part="1"
-F 0 "C24" V 9598 4350 50  0000 C CNN
+F 0 "C35" V 9598 4350 50  0000 C CNN
 F 1 "10u" V 9689 4350 50  0000 C CNN
 F 2 "Resistors_SMD:R_1210_HandSoldering" H 9888 4200 50  0001 C CNN
@@
 AR Path="/5A33279F/5A3ACFE6" Ref="D10"  Part="1"
 AR Path="/5A340028/5A3ACFE6" Ref="D11"  Part="1"
-F 0 "D10" H 8900 2284 50  0000 C CNN
+F 0 "D11" H 8900 2284 50  0000 C CNN
 F 1 "D" H 8900 2375 50  0000 C CNN
 F 2 "Diodes_SMD:D_SMA_Handsoldering" H 8900 2500 50  0001 C CNN
@@
 AR Path="/5A340028/5A337FB6" Ref="R45"  Part="1"
 AR Path="/5A33279F/5A337FB6" Ref="R44"  Part="1"
-F 0 "R44" V 4293 3100 50  0000 C CNN
+F 0 "R45" V 4293 3100 50  0000 C CNN
 F 1 "DNP" V 4384 3100 50  0000 C CNN
 F 2 "Resistors_SMD:R_0805_HandSoldering" V 4430 3100 50  0001 C CNN

Commit message: PCB changes
Parts:
- U5: footprint Housings_SOIC:SOIC-8_3.9x4.9mm_Pitch1.27mm -> Housings_SOIC:SOIC-8-1EP_3.9x4.9mm_Pitch1.27mm
Changed lines of the file:
@@
 $Descr A4 11693 8268
 encoding utf-8
-Sheet 3 7
+Sheet 5 7
 Title ""
 Date ""
@@
 F 0 "U7" H 7950 3867 50  0000 C CNN
 F 1 "IXD-609" H 7950 3776 50  0000 C CNN
-F 2 "Housings_SOIC:SOIC-8_3.9x4.9mm_Pitch1.27mm" H 7950 3050 50  0001 C CIN
+F 2 "Housings_SOIC:SOIC-8-1EP_3.9x4.9mm_Pitch1.27mm" H 7950 3050 50  0001 C CIN
 F 3 "http://www.ixysic.com/home/pdfs.nsf/www/IXD_609.pdf/$file/IXD_609.pdf" H 7950 3400 50  0001 C CNN
 	1    7950 3400
