File: PCB/ENNOID Dual Gate Driver.kicad_pcb (KiCad board)
At the start: 2 copper layers, 133 parts, among them J1 Conn_02x08_Odd_Even, J2 Current, J3 TEMP, J4 PHASE, J5 Collector, J6 Gate_H, J7 G_L, J8 E, Q1 Q_NPN_CBE, Q2 Q_NPN_CBE, Q3 2N7002K-7, Q4 2N7002K-7, Q5 2N7002, Q6 2N7002, Q7 2N7002, Q8 2N7002, U1 MC7805, U2 MGJ2, U3 MGJ2, U4 1ED020I12-F2, U5 IXD-609, U6 1ED020I12-F2, U7 IXD-609, U8 AMC1301, U9 4069

Commit message: PCB half-done
Parts:
- added R44: DNP, Resistors_SMD:R_0805_HandSoldering, F.Cu at (20.6, 35.7)
- added R45: DNP, Resistors_SMD:R_0805_HandSoldering, F.Cu at (54.7, 32.6)
- added REF**: MountingHole_2.2mm_M2_Pad_Via, Mounting_Holes:MountingHole_2.2mm_M2_Pad_Via, F.Cu at (5.00, 93.0)
- added REF**: MountingHole_2.2mm_M2_Pad_Via, Mounting_Holes:MountingHole_2.2mm_M2_Pad_Via, F.Cu at (55.0, 93.0)
- Q1, Q2: value Q_NPN_CBE -> Q_NPN_BCE
- U1: footprint TO_SOT_Packages_SMD:TO-263-3_TabPin4 -> TO_SOT_Packages_SMD:TO-252-3_TabPin2
- U8: footprint Housings_SOIC:SOIC-8_3.9x4.9mm_Pitch1.27mm -> Housings_SOIC:SSO-8_6.8x5.9mm_Pitch1.27mm_Clearance8mm
- moved D10 304.9 mm to (17.9, 19.8)
- moved D11 303.7 mm to (39.9, 20.9), turned to 180 degrees
- moved D17 299.7 mm to (12.1, 78.5), turned to 270 degrees
- moved D14 293.4 mm to (3.04, 74.1), turned to 270 degrees
- moved R43 289.9 mm to (12.8, 69.6)
- moved C45 289.4 mm to (5.42, 87.3)
- moved R41 288.9 mm to (12.0, 83.3), turned to 90 degrees
- moved U4 284.8 mm to (16.6, 49.9), turned to 270 degrees
- moved D16 284.3 mm to (17.3, 82.7), turned to 270 degrees
- moved D15 279.6 mm to (5.51, 74.1), turned to 270 degrees
- moved R42 279.5 mm to (12.8, 71.6)
- moved R40 277.2 mm to (18.7, 86.4), turned to 180 degrees
- moved R39 275.3 mm to (17.4, 74.0), turned to 90 degrees
- moved U6 273.1 mm to (52.3, 48.7), turned to 270 degrees
- moved Q8 272.3 mm to (13.0, 74.3), turned to 270 degrees
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Connections:
- Q1 pad 1: /GD_HIGH/+VCC -> Net-(Q1-Pad1)
- Q1 pad 2: Net-(Q1-Pad2) -> /GD_LOW/+VCC
- Q1 pad 3: /GD_HIGH/VCC_REG -> /GD_LOW/VCC_REG
- Q2 pad 1: /GD_LOW/+VCC -> Net-(Q2-Pad1)
- Q2 pad 2: Net-(Q2-Pad2) -> /GD_HIGH/+VCC
- Q2 pad 3: /GD_LOW/VCC_REG -> /GD_HIGH/VCC_REG
- R16 pad 2: /GD_LOW/FLT_ALL -> FLT_ALL
- R2 pad 2: Net-(Q1-Pad2) -> Net-(Q2-Pad1)
- R4 pad 2: Net-(Q2-Pad2) -> Net-(Q1-Pad1)
- R5 pad 2: /GD_HIGH/FLT_ALL -> FLT_ALL
- U4 pad 13: (no net) -> FLT_H
- U6 pad 13: (no net) -> FLT_L
Other:
- board outline added: 60 x 98 mm

Commit message: Routing has started
Parts:
- added REF**: MountingHole_2.2mm_M2_Pad_Via, Mounting_Holes:MountingHole_2.2mm_M2_Pad_Via, F.Cu at (30.0, 4.00)
- J1: footprint Connectors_IDC:IDC-Header_2x08_Pitch2.54mm_Straight -> Connectors_Multicomp:Multicomp_MC9A12-1634_2x08x2.54mm_Straight
- J5: moved to B.Cu
- moved C21 16.4 mm to (23.9, 16.3)
- moved C20 16.2 mm to (23.9, 26.4)
- moved U5 16.2 mm to (23.8, 21.6)
- moved R27 9.99 mm to (33.6, 16.6)
- moved R29 9.99 mm to (33.6, 21.5)
- moved D1 9.55 mm to (23.6, 31.7)
- moved C24 8.56 mm to (23.9, 13.6), turned to 0 degrees
- moved C23 8.34 mm to (24.0, 11.0), turned to 0 degrees
- moved C22 8.34 mm to (24.0, 9.13), turned to 0 degrees
- moved J2 7.77 mm to (11.5, 88.3), turned to 270 degrees
- moved R15 7.22 mm to (15.7, 11.0)
- moved C25 7.16 mm to (15.8, 9.13)
- moved D10 7.13 mm to (12.6, 24.6)
- moved R13 7.13 mm to (10.8, 18.8)
- moved R12 7.13 mm to (14.2, 18.8)
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Routing:
- net +5V: track 0.00 -> 34.9 mm, vias 0 -> 19
- added copper zone on B.Cu, net +5V
- added copper zone on F.Cu, net GND

Commit message: PCB completed with readme update
Parts:
- FL1, FL2: value ACM4520-142-2P-T000 -> ACM4520
- J1: footprint Connectors_Multicomp:Multicomp_MC9A12-1634_2x08x2.54mm_Straight -> ENNOID:Multicomp_MC9A12-1634_2x08x2.54mm_Straight
- J4, J6, J7, J8: moved to B.Cu
- J5: moved to F.Cu
- U8: footprint Housings_SOIC:SSO-8_6.8x5.9mm_Pitch1.27mm_Clearance8mm -> ENNOID:SSO-8_6.8x5.9mm_Pitch1.27mm_Clearance8mm
- moved R11 9.94 mm to (7.57, 18.8)
- moved R14 9.87 mm to (17.4, 18.8)
- moved C10 9.18 mm to (38.7, 58.7), turned to 0 degrees
- moved C5 7.19 mm to (3.12, 61.2)
- moved C6 7.19 mm to (3.13, 59.2)
- moved C11 6.11 mm to (38.7, 60.7), turned to 0 degrees
- moved J7 6.00 mm to (43.5, 4.00), turned to 270 degrees
- moved J8 6.00 mm to (37.5, 4.00), turned to 270 degrees
- moved R12 3.36 mm to (10.8, 18.8)
- moved R13 3.28 mm to (14.1, 18.8)
- moved FL1 2.39 mm to (3.15, 66.0)
- moved C20 2.07 mm to (24.5, 28.4)
- moved C31 2.01 mm to (56.7, 27.8)
- moved R18 1.96 mm to (56.3, 57.9)
- moved R20 1.93 mm to (54.3, 57.9)
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- renumbered REF** to M1, REF** to M2, REF** to M3
Connections:
- FL1 pad 2: Net-(C5-Pad1) -> GND
- FL1 pad 3: GND -> Net-(C5-Pad2)
- FL1 pad 4: Net-(C5-Pad2) -> Net-(C5-Pad1)
- FL2 pad 2: Net-(C10-Pad1) -> GND
- FL2 pad 3: GND -> Net-(C10-Pad2)
- FL2 pad 4: Net-(C10-Pad2) -> Net-(C10-Pad1)
Routing:
- net /GD_HIGH/+VCC: track 0.00 -> 195.4 mm, vias 0 -> 16
- net VCC_IN: track 0.00 -> 192.6 mm, vias 0 -> 12
- net /GD_LOW/+VCC: track 0.00 -> 167.7 mm, vias 0 -> 16
- net /GD_LOW/E: track 0.00 -> 123.8 mm, vias 0 -> 10
- net FLT_ALL: track 0.00 -> 89.7 mm, vias 0 -> 4
- net PHASE: track 0.00 -> 87.9 mm, vias 0 -> 7
- net RST: track 0.00 -> 83.2 mm, vias 0 -> 5
- net GND: track 0.00 -> 80.5 mm, vias 0 -> 15
- net FLT_L: track 0.00 -> 78.1 mm, vias 0 -> 4
- net /GD_LOW/G: track 0.00 -> 69.2 mm, vias 0 -> 4
- net /GD_LOW/-VEE: track 0.00 -> 66.3 mm
- net PWM_H: track 0.00 -> 55.4 mm, vias 0 -> 4
- net FLT_H: track 0.00 -> 54.3 mm, vias 0 -> 2
- net Net-(R38-Pad1): track 0.00 -> 51.4 mm, vias 0 -> 2
- net Vout+: track 0.00 -> 44.1 mm, vias 0 -> 2
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- added copper zone on F.Cu, net /GD_HIGH/-VEE
- added copper zone on F.Cu, net /GD_LOW/-VEE
- added copper zone on B.Cu, net /GD_LOW/E
- added copper zone on B.Cu, net PHASE
Other:
- board text added: "E1"
- board text added: "E2"
- board text added: "G1"
- board text added: "G2"

Commit message: Minor updates
Parts:
- moved C42 7.82 mm to (32.9, 85.2), turned to 270 degrees
- moved C41 7.11 mm to (40.3, 83.7)
- moved R32 5.44 mm to (47.1, 88.1), turned to 270 degrees
- moved C44 4.49 mm to (47.1, 83.4), turned to 90 degrees
- moved R41 0.71 mm to (12.8, 83.3)
- moved D17 0.67 mm to (12.8, 78.4)
Connections:
- C41 pad 1: PWM_H -> PWM_L
- C42 pad 1: PWM_L -> PWM_H
- J1 pad 11: PWM_H -> PWM_L
- J1 pad 12: PWM_L -> PWM_H
Routing:
- net /GD_LOW/G: track 69.2 -> 144.7 mm, vias 4 -> 15
- net /GD_HIGH/G: track 28.7 -> 93.5 mm, vias 0 -> 11
- net GND: track 80.5 -> 62.2 mm, vias 15 -> 11
- net VCC_IN: track 192.6 -> 182.9 mm
- net TEMP: track 25.9 -> 19.4 mm
- net FLT_L: track 78.1 -> 81.8 mm, vias 4 -> 3
- net +5V: track 58.2 -> 61.7 mm, vias 20 -> 22
- net PWM_H: track 55.4 -> 52.2 mm
- net FLT_ALL: track 89.7 -> 91.8 mm
- net PWM_L: track 42.4 -> 44.0 mm, vias 2 -> 4
- net FLT_H: track 54.3 -> 55.9 mm
- net RST: track 83.2 -> 84.5 mm
- net PHASE: track 87.9 -> 87.2 mm
- net Net-(R38-Pad1): track 51.4 -> 50.7 mm
- net Vout-: track 41.9 -> 41.2 mm
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
Commit message: Minor changes
Connections:
- C21 pad 1: Net-(C21-Pad1) -> /GD_HIGH/+VCC
- C32 pad 1: Net-(C32-Pad1) -> /GD_LOW/+VCC
- D10 pad 1: Net-(C21-Pad1) -> Net-(D10-Pad1)
- D11 pad 1: Net-(C32-Pad1) -> Net-(D11-Pad1)
- R13 pad 1: Net-(C21-Pad1) -> Net-(D10-Pad1)
- R14 pad 1: Net-(C21-Pad1) -> Net-(D10-Pad1)
- R24 pad 1: Net-(C32-Pad1) -> Net-(D11-Pad1)
- R25 pad 1: Net-(C32-Pad1) -> Net-(D11-Pad1)
- U5 pad 6: Net-(C21-Pad1) -> Net-(D10-Pad1)
- U5 pad 7: Net-(C21-Pad1) -> Net-(D10-Pad1)
- U7 pad 6: Net-(C32-Pad1) -> Net-(D11-Pad1)
- U7 pad 7: Net-(C32-Pad1) -> Net-(D11-Pad1)
Routing:
- net Net-(C21-Pad1): track 31.1 -> 0.00 mm
- net Net-(C32-Pad1): track 28.6 -> 0.00 mm
- net Net-(D10-Pad1): track 0.00 -> 24.8 mm
- net Net-(D11-Pad1): track 0.00 -> 22.6 mm
- net /GD_HIGH/+VCC: track 195.4 -> 209.5 mm
- net /GD_LOW/+VCC: track 167.7 -> 181.8 mm
- net PHASE: track 87.2 -> 89.1 mm
- net Net-(C19-Pad1): track 34.1 -> 35.5 mm

Commit message: Small changes
Parts:
- moved U2 0.05 mm to (3.10, 55.0)
Changed lines of the file:
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@@
     )
   )
-  (module ENNOID:DCDC-Conv_muRata_MGJ2 (layer F.Cu)
-    (at 3.0988 54.9148 180)
-    (tags "muRata MGJ2DCDC-Converter")
-    (fp_text reference U2 (at -5.6896 -3.0988 180) (layer F.SilkS)
-      (effects (font (size 1 1) (thickness 0.15)))
-    )
-    (fp_text value MGJ2 (at -1 19 180) (layer F.Fab)
-      (effects (font (size 1 1) (thickness 0.15)))
-    )
-    (fp_text user %R (at -2.25 6 270) (layer F.Fab)
-      (effects (font (size 1 1) (thickness 0.15)))
-    )
-    (fp_line (start 2.6 -2.28) (end -7.6 -2.28) (layer F.CrtYd) (width 0.05))
-    (fp_line (start 2.6 17.72) (end 2.6 -2.28) (layer F.CrtYd) (width 0.05))
-    (fp_line (start -7.6 17.72) (end 2.6 17.72) (layer F.CrtYd) (width 0.05))
-    (fp_line (start -7.6 -2.28) (end -7.6 17.72) (layer F.CrtYd) (width 0.05))
-    (fp_line (start 2.5 -2.15) (end -7.5 -2.15) (layer F.SilkS) (width 0.12))
-    (fp_line (start 2.5 17.59) (end 2.5 -2.15) (layer F.SilkS) (width 0.12))
-    (fp_line (start -7.5 17.59) (end 2.5 17.59) (layer F.SilkS) (width 0.12))
-    (fp_line (start -7.5 -2.15) (end -7.5 17.59) (layer F.SilkS) (width 0.12))
-    (fp_line (start 1.4 -2.03) (end -7.5 -2.03) (layer F.Fab) (width 0.1))
-    (fp_line (start 2.4 17.47) (end 2.4 -1.03) (layer F.Fab) (width 0.1))
-    (fp_line (start -7.4 17.47) (end 2.4 17.47) (layer F.Fab) (width 0.1))
-    (fp_line (start -7.4 -2.03) (end -7.4 17.47) (layer F.Fab) (width 0.1))
-    (fp_line (start 2.8 -2.53) (end 2.8 -0.5) (layer F.SilkS) (width 0.1))
-    (fp_line (start 2.8 -2.53) (end 0.5 -2.53) (layer F.SilkS) (width 0.1))
-    (fp_line (start 1.4 -2.03) (end 2.4 -1.03) (layer F.Fab) (width 0.1))
-    (pad 7 thru_hole oval (at 0 15.24 180) (size 1.5 1.5) (drill 0.7) (layers *.Cu *.Mask)
-      (net 6 /GD_HIGH/+VCC))
-    (pad 6 thru_hole oval (at 0 12.7 180) (size 1.5 1.5) (drill 0.7) (layers *.Cu *.Mask)
-      (net 5 PHASE))
-    (pad 5 thru_hole oval (at 0 10.16 180) (size 1.5 1.5) (drill 0.7) (layers *.Cu *.Mask)
-      (net 7 /GD_HIGH/-VEE))
-    (pad 2 thru_hole oval (at 0 2.54 180) (size 1.5 1.5) (drill 0.7) (layers *.Cu *.Mask)
-      (net 4 "Net-(C5-Pad2)"))
-    (pad 1 thru_hole rect (at 0 0 180) (size 1.5 1.5) (drill 0.7) (layers *.Cu *.Mask)
-      (net 3 "Net-(C5-Pad1)"))
-    (model ${ENNOID}/mgj2.step
-      (offset (xyz 2.6 2.75 0))
-      (scale (xyz 1 1 1))
-      (rotate (xyz 0 0 180))
-    )
-  )
   (module Resistors_SMD:R_0805_HandSoldering (layer F.Cu)
     (at 20.5359 67.4878 270)
@@
     )
   )
-  (module ENNOID:DCDC-Conv_muRata_MGJ2 (layer F.Cu)
-    (at 38.7858 55.0037 180)
-    (tags "muRata MGJ2DCDC-Converter")
-    (fp_text reference U3 (at -6.5786 -3.1623 180) (layer F.SilkS)
-      (effects (font (size 1 1) (thickness 0.15)))
-    )
-    (fp_text value MGJ2 (at -1 19 180) (layer F.Fab)
-      (effects (font (size 1 1) (thickness 0.15)))
-    )
-    (fp_line (start 1.4 -2.03) (end 2.4 -1.03) (layer F.Fab) (width 0.1))
-    (fp_line (start 2.8 -2.53) (end 0.5 -2.53) (layer F.SilkS) (width 0.1))
-    (fp_line (start 2.8 -2.53) (end 2.8 -0.5) (layer F.SilkS) (width 0.1))
-    (fp_line (start -7.4 -2.03) (end -7.4 17.47) (layer F.Fab) (width 0.1))
-    (fp_line (start -7.4 17.47) (end 2.4 17.47) (layer F.Fab) (width 0.1))
-    (fp_line (start 2.4 17.47) (end 2.4 -1.03) (layer F.Fab) (width 0.1))
-    (fp_line (start 1.4 -2.03) (end -7.5 -2.03) (layer F.Fab) (width 0.1))
-    (fp_line (start -7.5 -2.15) (end -7.5 17.59) (layer F.SilkS) (width 0.12))
-    (fp_line (start -7.5 17.59) (end 2.5 17.59) (layer F.SilkS) (width 0.12))
-    (fp_line (start 2.5 17.59) (end 2.5 -2.15) (layer F.SilkS) (width 0.12))
-    (fp_line (start 2.5 -2.15) (end -7.5 -2.15) (layer F.SilkS) (width 0.12))
-    (fp_line (start -7.6 -2.28) (end -7.6 17.72) (layer F.CrtYd) (width 0.05))
-    (fp_line (start -7.6 17.72) (end 2.6 17.72) (layer F.CrtYd) (width 0.05))
-    (fp_line (start 2.6 17.72) (end 2.6 -2.28) (layer F.CrtYd) (width 0.05))
-    (fp_line (start 2.6 -2.28) (end -7.6 -2.28) (layer F.CrtYd) (width 0.05))
-    (fp_text user %R (at -2.25 6 270) (layer F.Fab)
-      (effects (font (size 1 1) (thickness 0.15)))
-    )
-    (pad 1 thru_hole rect (at 0 0 180) (size 1.5 1.5) (drill 0.7) (layers *.Cu *.Mask)
-      (net 9 "Net-(C10-Pad1)"))
-    (pad 2 thru_hole oval (at 0 2.54 180) (size 1.5 1.5) (drill 0.7) (layers *.Cu *.Mask)
-      (net 10 "Net-(C10-Pad2)"))
-    (pad 5 thru_hole oval (at 0 10.16 180) (size 1.5 1.5) (drill 0.7) (layers *.Cu *.Mask)
-      (net 13 /GD_LOW/-VEE))
-    (pad 6 thru_hole oval (at 0 12.7 180) (size 1.5 1.5) (drill 0.7) (layers *.Cu *.Mask)
-      (net 11 /GD_LOW/E))
-    (pad 7 thru_hole oval (at 0 15.24 180) (size 1.5 1.5) (drill 0.7) (layers *.Cu *.Mask)
-      (net 12 /GD_LOW/+VCC))
-    (model ${ENNOID}/mgj2.step
-      (offset (xyz 2.6 2.75 0))
-      (scale (xyz 1 1 1))
-      (rotate (xyz 0 0 180))
-    )
-  )
   (module ENNOID:SSO-8_6.8x5.9mm_Pitch1.27mm_Clearance8mm (layer F.Cu)
     (at 29.9974 47.6504 270)
@@
     )
   )
+  (module ENNOID:DCDC-Conv_muRata_MGJ2 (layer F.Cu)
+    (at 3.0988 54.9656 180)
+    (tags "muRata MGJ2DCDC-Converter")
+    (fp_text reference U2 (at -3 -3 180) (layer F.SilkS)
+      (effects (font (size 1 1) (thickness 0.15)))
+    )
+    (fp_text value MGJ2 (at -1 19 180) (layer F.Fab)
+      (effects (font (size 1 1) (thickness 0.15)))
+    )
+    (fp_text user %R (at -2.25 6 270) (layer F.Fab)
+      (effects (font (size 1 1) (thickness 0.15)))
+    )
+    (fp_line (start 2.6 -2.28) (end -7.6 -2.28) (layer F.CrtYd) (width 0.05))
+    (fp_line (start 2.6 17.72) (end 2.6 -2.28) (layer F.CrtYd) (width 0.05))
+    (fp_line (start -7.6 17.72) (end 2.6 17.72) (layer F.CrtYd) (width 0.05))
+    (fp_line (start -7.6 -2.28) (end -7.6 17.72) (layer F.CrtYd) (width 0.05))
+    (fp_line (start 2.5 -2.15) (end -7.5 -2.15) (layer F.SilkS) (width 0.12))
+    (fp_line (start 2.5 17.59) (end 2.5 -2.15) (layer F.SilkS) (width 0.12))
+    (fp_line (start -7.5 17.59) (end 2.5 17.59) (layer F.SilkS) (width 0.12))
+    (fp_line (start -7.5 -2.15) (end -7.5 17.59) (layer F.SilkS) (width 0.12))
+    (fp_line (start 1.4 -2.03) (end -7.5 -2.03) (layer F.Fab) (width 0.1))
+    (fp_line (start 2.4 17.47) (end 2.4 -1.03) (layer F.Fab) (width 0.1))
+    (fp_line (start -7.4 17.47) (end 2.4 17.47) (layer F.Fab) (width 0.1))
+    (fp_line (start -7.4 -2.03) (end -7.4 17.47) (layer F.Fab) (width 0.1))
+    (fp_line (start 2.8 -2.53) (end 2.8 -0.5) (layer F.SilkS) (width 0.1))
+    (fp_line (start 2.8 -2.53) (end 0.5 -2.53) (layer F.SilkS) (width 0.1))
+    (fp_line (start 1.4 -2.03) (end 2.4 -1.03) (layer F.Fab) (width 0.1))
+    (pad 7 thru_hole oval (at 0 15.24 180) (size 1.5 1.5) (drill 0.7) (layers *.Cu *.Mask)
+      (net 6 /GD_HIGH/+VCC))
+    (pad 6 thru_hole oval (at 0 12.7 180) (size 1.5 1.5) (drill 0.7) (layers *.Cu *.Mask)
+      (net 5 PHASE))
+    (pad 5 thru_hole oval (at 0 10.16 180) (size 1.5 1.5) (drill 0.7) (layers *.Cu *.Mask)
+      (net 7 /GD_HIGH/-VEE))
+    (pad 2 thru_hole oval (at 0 2.54 180) (size 1.5 1.5) (drill 0.7) (layers *.Cu *.Mask)
+      (net 4 "Net-(C5-Pad2)"))
+    (pad 1 thru_hole rect (at 0 0 180) (size 1.5 1.5) (drill 0.7) (layers *.Cu *.Mask)
+      (net 3 "Net-(C5-Pad1)"))
+    (model ${ENNOID}/MGJ2.step
+      (offset (xyz 0 0 -4))
+      (scale (xyz 1 1 1))
+      (rotate (xyz -90 0 90))
+    )
+  )
+  (module ENNOID:DCDC-Conv_muRata_MGJ2 (layer F.Cu)
+    (at 38.7858 55.0037 180)
+    (tags "muRata MGJ2DCDC-Converter")
+    (fp_text reference U3 (at -3 -3 180) (layer F.SilkS)
+      (effects (font (size 1 1) (thickness 0.15)))
+    )
+    (fp_text value MGJ2 (at -1 19 180) (layer F.Fab)
+      (effects (font (size 1 1) (thickness 0.15)))
+    )
+    (fp_line (start 1.4 -2.03) (end 2.4 -1.03) (layer F.Fab) (width 0.1))
+    (fp_line (start 2.8 -2.53) (end 0.5 -2.53) (layer F.SilkS) (width 0.1))
+    (fp_line (start 2.8 -2.53) (end 2.8 -0.5) (layer F.SilkS) (width 0.1))
+    (fp_line (start -7.4 -2.03) (end -7.4 17.47) (layer F.Fab) (width 0.1))
+    (fp_line (start -7.4 17.47) (end 2.4 17.47) (layer F.Fab) (width 0.1))
+    (fp_line (start 2.4 17.47) (end 2.4 -1.03) (layer F.Fab) (width 0.1))
+    (fp_line (start 1.4 -2.03) (end -7.5 -2.03) (layer F.Fab) (width 0.1))
+    (fp_line (start -7.5 -2.15) (end -7.5 17.59) (layer F.SilkS) (width 0.12))
+    (fp_line (start -7.5 17.59) (end 2.5 17.59) (layer F.SilkS) (width 0.12))
+    (fp_line (start 2.5 17.59) (end 2.5 -2.15) (layer F.SilkS) (width 0.12))
+    (fp_line (start 2.5 -2.15) (end -7.5 -2.15) (layer F.SilkS) (width 0.12))
+    (fp_line (start -7.6 -2.28) (end -7.6 17.72) (layer F.CrtYd) (width 0.05))
+    (fp_line (start -7.6 17.72) (end 2.6 17.72) (layer F.CrtYd) (width 0.05))
+    (fp_line (start 2.6 17.72) (end 2.6 -2.28) (layer F.CrtYd) (width 0.05))
+    (fp_line (start 2.6 -2.28) (end -7.6 -2.28) (layer F.CrtYd) (width 0.05))
+    (fp_text user %R (at -2.25 6 270) (layer F.Fab)
+      (effects (font (size 1 1) (thickness 0.15)))
+    )
+    (pad 1 thru_hole rect (at 0 0 180) (size 1.5 1.5) (drill 0.7) (layers *.Cu *.Mask)
+      (net 9 "Net-(C10-Pad1)"))
+    (pad 2 thru_hole oval (at 0 2.54 180) (size 1.5 1.5) (drill 0.7) (layers *.Cu *.Mask)
+      (net 10 "Net-(C10-Pad2)"))
+    (pad 5 thru_hole oval (at 0 10.16 180) (size 1.5 1.5) (drill 0.7) (layers *.Cu *.Mask)
+      (net 13 /GD_LOW/-VEE))
+    (pad 6 thru_hole oval (at 0 12.7 180) (size 1.5 1.5) (drill 0.7) (layers *.Cu *.Mask)
+      (net 11 /GD_LOW/E))
+    (pad 7 thru_hole oval (at 0 15.24 180) (size 1.5 1.5) (drill 0.7) (layers *.Cu *.Mask)
+      (net 12 /GD_LOW/+VCC))
+    (model ${ENNOID}/MGJ2.step
+      (offset (xyz 0 0 -4))
+      (scale (xyz 1 1 1))
+      (rotate (xyz -90 0 90))
+    )
+  )

Commit message: pcb error correction
Parts:
- moved C42 7.64 mm to (40.4, 83.6)
- moved C41 7.52 mm to (32.9, 85.2)
Connections:
- C41 pad 1: PWM_L -> PWM_H
- C42 pad 1: PWM_H -> PWM_L
- J1 pad 11: PWM_L -> PWM_H
- J1 pad 12: PWM_H -> PWM_L
Routing:
- net PWM_L: track 44.0 -> 41.4 mm
- net PWM_H: track 52.2 -> 54.2 mm
Other:
- board text added: "FLT_H"
- board text added: "FLT_L"
- board text added: "RDY_H"
- board text added: "RDY_L"

Commit message: PCB changes
Parts:
- C12, C13, C14, C20, C21, C22, C23, C31, C32, C38, C7, C8, C9, D9, Q1, Q2, R1, R2, R22, R23, R27, R28, R29, R3, R4, R44, R45: moved to B.Cu
- R19, R8: value 1k -> 47k
- U5, U7: footprint Housings_SOIC:SOIC-8_3.9x4.9mm_Pitch1.27mm -> Housings_SOIC:SOIC-8-1EP_3.9x4.9mm_Pitch1.27mm
- moved D6 26.0 mm to (57.0, 37.5)
- moved D3 21.2 mm to (23.0, 37.5), turned to 180 degrees
- moved C33 19.8 mm to (41.5, 23.4), turned to 270 degrees
- moved C35 19.1 mm to (39.0, 22.4), turned to 270 degrees
- moved C34 17.1 mm to (43.3, 23.4), turned to 270 degrees
- moved D11 15.1 mm to (57.9, 18.5), turned to 270 degrees
- moved C22 14.4 mm to (24.3, 23.5), turned to 270 degrees
- moved C21 13.8 mm to (17.5, 28.5)
- moved C23 12.6 mm to (22.3, 23.5), turned to 270 degrees
- moved R23 12.3 mm to (54.3, 15.7)
- moved R22 12.1 mm to (50.8, 15.7)
- moved D1 11.9 mm to (11.0, 33.0), turned to 270 degrees
- moved U5 11.3 mm to (17.5, 31.0)
- moved D2 10.8 mm to (46.2, 33.3), turned to 270 degrees
- moved R3 10.6 mm to (38.7, 29.5)
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Connections:
- R28 pad 2: /GD_LOW/VCC_REG -> /GD_LOW/+VCC
Routing:
- net /GD_HIGH/+VCC: track 209.5 -> 5.02 mm, vias 16 -> 2
- net VCC_IN: track 182.9 -> 0.00 mm, vias 12 -> 0
- net /GD_LOW/+VCC: track 181.8 -> 25.1 mm, vias 16 -> 4
- net /GD_LOW/G: track 144.7 -> 0.00 mm, vias 15 -> 0
- net /GD_LOW/E: track 123.8 -> 15.8 mm, vias 10 -> 1
- net /GD_HIGH/G: track 93.5 -> 0.00 mm, vias 11 -> 0
- net FLT_ALL: track 91.8 -> 0.00 mm, vias 4 -> 0
- net RST: track 84.5 -> 0.00 mm, vias 5 -> 0
- net FLT_L: track 81.8 -> 0.00 mm, vias 3 -> 0
- net GND: track 62.1 -> 0.00 mm, vias 11 -> 0
- net +5V: track 61.7 -> 0.00 mm, vias 22 -> 0
- net FLT_H: track 55.9 -> 0.00 mm, vias 2 -> 0
- net PWM_H: track 54.2 -> 0.00 mm, vias 4 -> 0
- net (no net): track 0.00 -> 53.0 mm
- net Net-(R38-Pad1): track 50.7 -> 0.00 mm, vias 2 -> 0
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- added copper zone on B.Cu, net /GD_HIGH/+VCC
- added copper zone on B.Cu, net /GD_HIGH/-VEE
- added copper zone on B.Cu, net /GD_HIGH/G
- added copper zone on F.Cu, net /GD_HIGH/G
- added copper zone on B.Cu, net /GD_LOW/+VCC
- added copper zone on B.Cu, net /GD_LOW/-VEE
- added copper zone on F.Cu, net /GD_LOW/E
- added copper zone on B.Cu, net /GD_LOW/G
- added copper zone on F.Cu, net /GD_LOW/G
- added copper zone on F.Cu, net PHASE
- removed copper zone on F.Cu, net /GD_HIGH/-VEE
- removed copper zone on F.Cu, net /GD_LOW/-VEE
- removed copper zone on B.Cu, net /GD_LOW/E
- removed copper zone on B.Cu, net PHASE
