File: PCB/ENNOID Dual Gate Driver.kicad_pcb (KiCad board)
At the start: 2 copper layers, 60 x 98 mm, 138 parts, among them J1 Conn_02x08_Odd_Even, J2 Current, J3 TEMP, J4 PHASE, J5 Collector, J6 Gate_H, J7 G_L, J8 E, M1 MountingHole_2.2mm_M2_Pad_Via, M2 MountingHole_2.2mm_M2_Pad_Via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

Commit message: PCB changes
Parts:
- C24, R11, R12: moved to B.Cu
- moved R1 7.50 mm to (4.39, 29.4)
- moved D10 5.59 mm to (9.25, 19.2), turned to 270 degrees
- moved C20 4.26 mm to (16.9, 29.3)
- moved C21 4.26 mm to (16.9, 24.3)
- moved U5 4.26 mm to (16.9, 26.8)
- moved C22 4.06 mm to (21.3, 20.7)
- moved C23 4.06 mm to (19.3, 20.7)
- moved R11 3.66 mm to (12.8, 15.5)
- moved R12 3.66 mm to (16.3, 15.5)
- moved R13 3.35 mm to (12.8, 15.5)
- moved R14 3.35 mm to (16.3, 15.5)
- moved C24 3.30 mm to (23.7, 20.2)
- moved R10 1.90 mm to (3.86, 25.7), turned to 0 degrees
- moved R2 1.70 mm to (10.3, 29.4), turned to 0 degrees
- moved D1 1.33 mm to (12.2, 33.5)
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Routing:
- net Net-(D11-Pad2): track 0.00 -> 11.2 mm, vias 0 -> 2
- net /GD_HIGH/+VCC: track 5.02 -> 16.2 mm, vias 2 -> 4
- net /GD_HIGH/-VEE: track 28.5 -> 22.9 mm, vias 9 -> 11
- net Net-(D1-Pad1): track 3.78 -> 9.16 mm
- net Net-(D10-Pad1): track 22.3 -> 18.0 mm
- net Net-(R44-Pad2): track 12.0 -> 15.9 mm
- net PHASE: track 45.0 -> 48.0 mm, vias 11 -> 15
- net Net-(Q2-Pad1): track 2.88 -> 5.56 mm
- net Net-(C19-Pad1): track 37.2 -> 38.9 mm
- net Net-(D10-Pad2): track 11.5 -> 11.0 mm, vias 0 -> 2
