File: PCB/ENNOID Dual Gate Driver.sch (KiCad schematic (older format))
At the start: 15 parts, among them J1 Conn_02x08_Odd_Even, U1 MC7805

Commit message: Schematics & footprints completed
Ready for PCBnew
Parts:
- added C41, C42: 100n, Capacitors_SMD:C_0805_HandSoldering, symbol device:C
- added F1: Fuse, Resistors_SMD:R_0805_HandSoldering, symbol device:Fuse
- added J7: G_L, ENNOID:Quick_fit_terminal, symbol Connector:Conn_01x01_Female
- added J8: E, ENNOID:Quick_fit_terminal, symbol Connector:Conn_01x01_Female
- C1: footprint (none) -> Capacitors_SMD:C_1210_HandSoldering
- C2, C3, C4: footprint (none) -> Capacitors_SMD:C_0805_HandSoldering
- C43, C44: renamed from C?; footprint (none) -> Capacitors_SMD:C_0805_HandSoldering
- J2: renamed from J?; value Phase_Current -> Current; footprint (none) -> Connectors_Molex:Molex_KK-6410-04_04x2.54mm_Straight
- J3: renamed from J?; value Phase_Temp -> TEMP; footprint (none) -> Connectors_Molex:Molex_KK-6410-02_02x2.54mm_Straight
- J4, J5, J6: renamed from J?; footprint (none) -> ENNOID:Quick_fit_terminal
- R32, R33: renamed from R?; footprint (none) -> Resistors_SMD:R_0805_HandSoldering
- U1: footprint (none) -> TO_SOT_Packages_SMD:TO-263-3_TabPin4
Connections:
- net labels added: +24V, FLT_ALL, RST
- net labels removed: C, E, G_H, G_L, RST_H, RST_L
- wire segments 81 -> 114
- no-connect marks 0 -> 2

Commit message: PCB half-done
Parts:
- U1: footprint TO_SOT_Packages_SMD:TO-263-3_TabPin4 -> TO_SOT_Packages_SMD:TO-252-3_TabPin2
Connections:
- wire segments 114 -> 119
Changed lines of the file:
@@
 F7 "PHASE" O R 2700 1100 60
 $EndSheet
-Text GLabel 1350 850  0    60   Input ~ 0
-VCC_IN
 Wire Wire Line
 	1350 850  1500 850
@@
 Wire Wire Line
 	1300 1050 1300 1100
-Text GLabel 1150 2900 0    60   Input ~ 0
-VCC_IN
 $Comp
 L power:GND #PWR02
@@
 F7 "PHASE" O R 2500 3150 60
 $EndSheet
-Text GLabel 1000 5400 0    60   Input ~ 0
-VCC_IN
 $Comp
 L device:C C1
@@
 $EndComp
 Wire Wire Line
-	1000 5400 1200 5400
-Wire Wire Line
-	1200 5400 1650 5400
-Connection ~ 1200 5400
+	1200 5400 1500 5400
 $Comp
 L device:C C3
@@
 F 0 "U1" H 2350 5642 50  0000 C CNN
 F 1 "MC7805" H 2350 5551 50  0000 C CNN
-F 2 "TO_SOT_Packages_SMD:TO-263-3_TabPin4" H 2375 5250 50  0001 L CIN
+F 2 "TO_SOT_Packages_SMD:TO-252-3_TabPin2" H 2375 5250 50  0001 L CIN
 F 3 "" H 2350 5350 50  0001 C CNN
 	1    2350 5400
@@
 Text GLabel 2700 6800 2    60   Input ~ 0
 PWM_L
-Text GLabel 1200 7400 0    60   Input ~ 0
-VCC_IN
 Wire Wire Line
 	4400 1250 4900 1250
@@
 Text GLabel 1550 6500 0    60   Input ~ 0
 RST
-Text GLabel 2300 6500 2    60   Output ~ 0
+Text GLabel 2300 6500 2    60   Input ~ 0
 FLT_ALL
 Wire Wire Line
@@
 Wire Wire Line
 	2500 7100 2500 7150
-Connection ~ 1300 7400
-Wire Wire Line
-	1200 7400 1300 7400
 Connection ~ 1100 6800
 Wire Wire Line
@@
 Wire Wire Line
 	2300 6400 2200 6400
-Wire Wire Line
-	2200 6500 2300 6500
 NoConn ~ 2200 6600
 NoConn ~ 1700 6600
@@
 Wire Wire Line
 	2500 2950 3350 2950
-Wire Wire Line
-	4900 5200 3350 5200
-Wire Wire Line
-	3350 5200 3350 2950
-Connection ~ 3350 2950
 Wire Wire Line
 	3350 2950 4950 2950
@@
 FLT_ALL
 Wire Wire Line
-	10100 5550 10650 5550
-Text GLabel 8650 5200 0    60   Input ~ 0
-VCC_IN
-Wire Wire Line
-	8650 5200 8900 5200
+	8450 5200 8900 5200
 Text GLabel 8650 5300 0    60   Input ~ 0
 RDY_L
@@
 Wire Wire Line
 	8900 5750 8750 5750
+Text GLabel 4600 3600 0    60   Input ~ 0
+FLT_ALL
+Wire Wire Line
+	4600 3600 4950 3600
+Wire Wire Line
+	10100 5550 10650 5550
+Wire Wire Line
+	2200 6500 2300 6500
+Text GLabel 4400 1650 0    60   Input ~ 0
+FLT_ALL
+Wire Wire Line
+	4400 1650 4900 1650
+$Comp
+L power:+24V #PWR047
+U 1 1 5A3C8158
+P 1500 5400
+F 0 "#PWR047" H 1500 5250 50  0001 C CNN
+F 1 "+24V" H 1515 5573 50  0000 C CNN
+F 2 "" H 1500 5400 50  0001 C CNN
+F 3 "" H 1500 5400 50  0001 C CNN
+	1    1500 5400
+	1    0    0    -1
+$EndComp
+Connection ~ 1500 5400
+Wire Wire Line
+	1500 5400 1650 5400
+$Comp
+L power:+24V #PWR045
+U 1 1 5A3CC538
+P 1150 2900
+F 0 "#PWR045" H 1150 2750 50  0001 C CNN
+F 1 "+24V" H 1165 3073 50  0000 C CNN
+F 2 "" H 1150 2900 50  0001 C CNN
+F 3 "" H 1150 2900 50  0001 C CNN
+	1    1150 2900
+	1    0    0    -1
+$EndComp
+$Comp
+L power:+24V #PWR046
+U 1 1 5A3CC6A9
+P 1350 850
+F 0 "#PWR046" H 1350 700 50  0001 C CNN
+F 1 "+24V" H 1365 1023 50  0000 C CNN
+F 2 "" H 1350 850 50  0001 C CNN
+F 3 "" H 1350 850 50  0001 C CNN
+	1    1350 850
+	1    0    0    -1
+$EndComp
+$Comp
+L power:+24V #PWR048
+U 1 1 5A3D1FFC
+P 8450 5200
+F 0 "#PWR048" H 8450 5050 50  0001 C CNN
+F 1 "+24V" H 8465 5373 50  0000 C CNN
+F 2 "" H 8450 5200 50  0001 C CNN
+F 3 "" H 8450 5200 50  0001 C CNN
+	1    8450 5200
+	1    0    0    -1
+$EndComp
+Text GLabel 1050 7400 0    60   Input ~ 0
+VCC_IN
+Wire Wire Line
+	1300 7400 1050 7400
+Connection ~ 1300 7400
+Text GLabel 8350 5200 0    60   Input ~ 0
+VCC_IN
+Wire Wire Line
+	8350 5200 8450 5200
+Connection ~ 8450 5200
+Text GLabel 1050 2900 0    60   Input ~ 0
+VCC_IN
+Wire Wire Line
+	1150 2900 1050 2900
+Connection ~ 1150 2900
+Text GLabel 1150 850  0    60   Input ~ 0
+VCC_IN
+Wire Wire Line
+	1350 850  1150 850
+Connection ~ 1350 850
+Wire Wire Line
+	4900 5200 3350 5200
+Connection ~ 3350 2950
+Wire Wire Line
+	3350 5200 3350 2950
 $EndSCHEMATC

Commit message: Routing has started
Parts:
- J1: footprint Connectors_IDC:IDC-Header_2x08_Pitch2.54mm_Straight -> Connectors_Multicomp:Multicomp_MC9A12-1634_2x08x2.54mm_Straight
Changed lines of the file:
@@
 F 0 "J1" H 1950 7025 50  0000 C CNN
 F 1 "Conn_02x08_Odd_Even" H 1950 7026 50  0001 C CNN
-F 2 "Connectors_IDC:IDC-Header_2x08_Pitch2.54mm_Straight" H 1900 6600 50  0001 C CNN
+F 2 "Connectors_Multicomp:Multicomp_MC9A12-1634_2x08x2.54mm_Straight" H 1900 6600 50  0001 C CNN
 F 3 "~" H 1900 6600 50  0001 C CNN
 	1    1900 6600

Commit message: PCB completed with readme update
Parts:
- J1: footprint Connectors_Multicomp:Multicomp_MC9A12-1634_2x08x2.54mm_Straight -> ENNOID:Multicomp_MC9A12-1634_2x08x2.54mm_Straight
Changed lines of the file:
@@
 F 0 "J1" H 1950 7025 50  0000 C CNN
 F 1 "Conn_02x08_Odd_Even" H 1950 7026 50  0001 C CNN
-F 2 "Connectors_Multicomp:Multicomp_MC9A12-1634_2x08x2.54mm_Straight" H 1900 6600 50  0001 C CNN
+F 2 "ENNOID:Multicomp_MC9A12-1634_2x08x2.54mm_Straight" H 1900 6600 50  0001 C CNN
 F 3 "~" H 1900 6600 50  0001 C CNN
 	1    1900 6600

Commit message: Minor updates
Changed lines of the file:
@@
 FLT_H
 Text GLabel 2700 6800 2    60   Input ~ 0
-PWM_L
+PWM_H
 Wire Wire Line
 	4400 1250 4900 1250
@@
 	4550 3500 4950 3500
 Text GLabel 1000 6800 0    60   Input ~ 0
-PWM_H
+PWM_L
 Text GLabel 1550 6500 0    60   Input ~ 0
 RST

Commit message: pcb error correction
Changed lines of the file:
@@
 FLT_H
 Text GLabel 2700 6800 2    60   Input ~ 0
-PWM_H
+PWM_L
 Wire Wire Line
 	4400 1250 4900 1250
@@
 	4550 3500 4950 3500
 Text GLabel 1000 6800 0    60   Input ~ 0
-PWM_L
+PWM_H
 Text GLabel 1550 6500 0    60   Input ~ 0
 RST
@@
 	1    0    0    -1
 $EndComp
-$Comp
-L device:C C41
-U 1 1 5A3DD0B7
-P 1100 6950
-F 0 "C41" H 1215 6996 50  0000 L CNN
-F 1 "100n" H 1215 6905 50  0000 L CNN
-F 2 "Capacitors_SMD:C_0805_HandSoldering" H 1138 6800 50  0001 C CNN
-F 3 "" H 1100 6950 50  0001 C CNN
-	1    1100 6950
-	1    0    0    -1
-$EndComp
 Wire Wire Line
 	1300 7400 1350 7400
@@
 	1    0    0    -1
 $EndComp
-Wire Wire Line
-	2500 6800 2700 6800
-Connection ~ 2500 6800
 $Comp
 L power:GND #PWR026
@@
 Wire Wire Line
 	2500 7100 2500 7150
-Connection ~ 1100 6800
 Wire Wire Line
 	1100 6800 1700 6800
-Wire Wire Line
-	1000 6800 1100 6800
 Wire Wire Line
 	1550 6700 1700 6700
@@
 Wire Wire Line
 	3350 5200 3350 2950
+$Comp
+L device:C C41
+U 1 1 5A3DD0B7
+P 1100 6950
+F 0 "C41" H 1215 6996 50  0000 L CNN
+F 1 "100n" H 1215 6905 50  0000 L CNN
+F 2 "Capacitors_SMD:C_0805_HandSoldering" H 1138 6800 50  0001 C CNN
+F 3 "" H 1100 6950 50  0001 C CNN
+	1    1100 6950
+	1    0    0    -1
+$EndComp
+Connection ~ 1100 6800
+Wire Wire Line
+	1000 6800 1100 6800
+Connection ~ 2500 6800
+Wire Wire Line
+	2500 6800 2700 6800
 $EndSCHEMATC

Commit message: PCB changes
Changed lines of the file:
@@
 	2700 1000 4900 1000
 Wire Wire Line
-	2500 2850 4950 2850
+	2500 2850 3150 2850
 Wire Wire Line
 	2500 3050 4950 3050
@@
 F6 "Vout-" O L 4900 5500 60
 F7 "GND" I L 4900 5650 60
-F8 "VCC_REG" I L 4900 5200 60
+F8 "+VCC" I L 4900 5200 60
 $EndSheet
 $Comp
@@
 Wire Wire Line
 	5350 6900 5450 6900
-Wire Wire Line
-	2500 2950 3350 2950
-Wire Wire Line
-	3350 2950 4950 2950
 $Comp
 L Connector:Conn_01x01_Female J7
@@
 	1350 850  1150 850
 Connection ~ 1350 850
-Wire Wire Line
-	4900 5200 3350 5200
-Connection ~ 3350 2950
-Wire Wire Line
-	3350 5200 3350 2950
 $Comp
 L device:C C41
@@
 Wire Wire Line
 	2500 6800 2700 6800
+Wire Wire Line
+	2500 2950 4950 2950
+Wire Wire Line
+	3150 5200 4900 5200
+Wire Wire Line
+	3150 2850 3150 5200
+Connection ~ 3150 2850
+Wire Wire Line
+	3150 2850 4950 2850
 $EndSCHEMATC
