File: PCB/V_PHASE.sch (KiCad schematic (older format))
At the start: 11 parts, among them U8 AMC1301

Commit message: Schematics & footprints completed
Ready for PCBnew
Parts:
- C37, C38, C39, C40: footprint (none) -> Capacitors_SMD:C_0805_HandSoldering
- D9: footprint (none) -> Diodes_SMD:D_SOT-23_ANK
- R27, R29, R30, R31: footprint (none) -> Resistors_SMD:R_0805_HandSoldering
- R28: value 12 -> 200; footprint (none) -> Resistors_SMD:R_0805_HandSoldering
Connections:
- net labels added: VCC_REG
Changed lines of the file:
@@
 $Descr A4 11693 8268
 encoding utf-8
-Sheet 8 6
+Sheet 6 7
 Title ""
 Date ""
@@
 F 0 "C37" H 5215 3346 50  0000 L CNN
 F 1 "100n" H 5215 3255 50  0000 L CNN
-F 2 "" H 5138 3150 50  0001 C CNN
+F 2 "Capacitors_SMD:C_0805_HandSoldering" H 5138 3150 50  0001 C CNN
 F 3 "" H 5100 3300 50  0001 C CNN
 	1    5100 3300
@@
 F 0 "C38" H 5265 3996 50  0000 L CNN
 F 1 "330p" H 5265 3905 50  0000 L CNN
-F 2 "" H 5188 3800 50  0001 C CNN
+F 2 "Capacitors_SMD:C_0805_HandSoldering" H 5188 3800 50  0001 C CNN
 F 3 "" H 5150 3950 50  0001 C CNN
 	1    5150 3950
@@
 	5500 3850 5500 4200
 Wire Wire Line
-	5500 4200 5150 4200
-Wire Wire Line
 	5150 4200 5150 4100
 $Comp
@@
 P 4200 3000
 F 0 "R28" V 3993 3000 50  0000 C CNN
-F 1 "12" V 4084 3000 50  0000 C CNN
-F 2 "" V 4130 3000 50  0001 C CNN
+F 1 "200" V 4084 3000 50  0000 C CNN
+F 2 "Resistors_SMD:R_0805_HandSoldering" V 4130 3000 50  0001 C CNN
 F 3 "" H 4200 3000 50  0001 C CNN
 	1    4200 3000
@@
 F 0 "R27" V 3593 3750 50  0000 C CNN
 F 1 "1M" V 3684 3750 50  0000 C CNN
-F 2 "" V 3730 3750 50  0001 C CNN
+F 2 "Resistors_SMD:R_0805_HandSoldering" V 3730 3750 50  0001 C CNN
 F 3 "" H 3800 3750 50  0001 C CNN
 	1    3800 3750
@@
 F 0 "R29" V 3993 3750 50  0000 C CNN
 F 1 "1M" V 4084 3750 50  0000 C CNN
-F 2 "" V 4130 3750 50  0001 C CNN
+F 2 "Resistors_SMD:R_0805_HandSoldering" V 4130 3750 50  0001 C CNN
 F 3 "" H 4200 3750 50  0001 C CNN
 	1    4200 3750
@@
 F 0 "R30" H 4430 3904 50  0000 R CNN
 F 1 "1k" H 4430 3995 50  0000 R CNN
-F 2 "" V 4430 3950 50  0001 C CNN
+F 2 "Resistors_SMD:R_0805_HandSoldering" V 4430 3950 50  0001 C CNN
 F 3 "" H 4500 3950 50  0001 C CNN
 	1    4500 3950
@@
 F 0 "R31" V 5007 4200 50  0000 C CNN
 F 1 "1k" V 4916 4200 50  0000 C CNN
-F 2 "" V 4730 4200 50  0001 C CNN
+F 2 "Resistors_SMD:R_0805_HandSoldering" V 4730 4200 50  0001 C CNN
 F 3 "" H 4800 4200 50  0001 C CNN
 	1    4800 4200
@@
 Wire Wire Line
 	5150 4200 4950 4200
-Connection ~ 5150 4200
 Wire Wire Line
 	4650 4200 4500 4200
@@
 F 0 "D9" V 4504 3329 50  0000 L CNN
 F 1 "5V" V 4595 3329 50  0000 L CNN
-F 2 "" H 4550 3250 50  0001 C CNN
+F 2 "Diodes_SMD:D_SOT-23_ANK" H 4550 3250 50  0001 C CNN
 F 3 "https://en.wikipedia.org/wiki/Zener_diode" H 4550 3250 50  0001 C CNN
 	1    4550 3250
@@
 F 0 "C39" H 6865 3346 50  0000 L CNN
 F 1 "100n" H 6865 3255 50  0000 L CNN
-F 2 "" H 6788 3150 50  0001 C CNN
+F 2 "Capacitors_SMD:C_0805_HandSoldering" H 6788 3150 50  0001 C CNN
 F 3 "" H 6750 3300 50  0001 C CNN
 	1    6750 3300
@@
 F 0 "C40" H 7315 3346 50  0000 L CNN
 F 1 "2.2u" H 7315 3255 50  0000 L CNN
-F 2 "" H 7238 3150 50  0001 C CNN
+F 2 "Capacitors_SMD:C_0805_HandSoldering" H 7238 3150 50  0001 C CNN
 F 3 "" H 7200 3300 50  0001 C CNN
 	1    7200 3300
@@
 Wire Wire Line
 	2950 4200 4500 4200
-Wire Wire Line
-	3950 3000 4050 3000
 Text HLabel 7950 3050 2    60   Input ~ 0
 +5V
@@
 Vout-
 $Comp
-L power:GND #PWR?
+L power:GND #PWR035
 U 1 1 5A34B574
 P 7600 3550
-F 0 "#PWR?" H 7600 3300 50  0001 C CNN
+F 0 "#PWR035" H 7600 3300 50  0001 C CNN
 F 1 "GND" H 7605 3377 50  0000 C CNN
 F 2 "" H 7600 3550 50  0001 C CNN
@@
 	7600 3550 7700 3550
 Connection ~ 7600 3550
+Text HLabel 3800 3000 0    60   Input ~ 0
+VCC_REG
+Wire Wire Line
+	4050 3000 3800 3000
+Wire Wire Line
+	5500 4200 5150 4200
+Connection ~ 5150 4200
 $EndSCHEMATC

Commit message: PCB half-done
Parts:
- U8: footprint Housings_SOIC:SOIC-8_3.9x4.9mm_Pitch1.27mm -> Housings_SOIC:SSO-8_6.8x5.9mm_Pitch1.27mm_Clearance8mm
Changed lines of the file:
@@
 F 0 "U8" H 5900 4117 50  0000 C CNN
 F 1 "AMC1301" H 5900 4026 50  0000 C CNN
-F 2 "Housings_SOIC:SOIC-8_3.9x4.9mm_Pitch1.27mm" H 5900 3300 50  0001 C CIN
+F 2 "Housings_SOIC:SSO-8_6.8x5.9mm_Pitch1.27mm_Clearance8mm" H 5900 3300 50  0001 C CIN
 F 3 "http://www.ti.com/lit/ds/symlink/amc1301.pdf" H 5900 3650 50  0001 C CNN
 	1    5900 3650

Commit message: PCB completed with readme update
Parts:
- U8: footprint Housings_SOIC:SSO-8_6.8x5.9mm_Pitch1.27mm_Clearance8mm -> ENNOID:SSO-8_6.8x5.9mm_Pitch1.27mm_Clearance8mm
Changed lines of the file:
@@
 F 0 "U8" H 5900 4117 50  0000 C CNN
 F 1 "AMC1301" H 5900 4026 50  0000 C CNN
-F 2 "Housings_SOIC:SSO-8_6.8x5.9mm_Pitch1.27mm_Clearance8mm" H 5900 3300 50  0001 C CIN
+F 2 "ENNOID:SSO-8_6.8x5.9mm_Pitch1.27mm_Clearance8mm" H 5900 3300 50  0001 C CIN
 F 3 "http://www.ti.com/lit/ds/symlink/amc1301.pdf" H 5900 3650 50  0001 C CNN
 	1    5900 3650

Commit message: PCB changes
Connections:
- net labels added: +VCC
- net labels removed: VCC_REG
Changed lines of the file:
@@
 Connection ~ 7600 3550
 Text HLabel 3800 3000 0    60   Input ~ 0
-VCC_REG
-Wire Wire Line
-	4050 3000 3800 3000
++VCC
 Wire Wire Line
 	5500 4200 5150 4200
 Connection ~ 5150 4200
+Wire Wire Line
+	4050 3000 3800 3000
 $EndSCHEMATC
