File: V0.1 - Wolfspeed/PCB/ENNOID Dual Gate Driver.kicad_pcb (KiCad board)
At the start: 2 copper layers, 60 x 98 mm, 118 parts, among them J1 Conn_02x08_Odd_Even, J2 Current, J3 TEMP, J4 PHASE, J5 Collector, J6 Gate_H, J7 G_L, J8 E, Q1 Q_NPN_BCE, Q2 Q_NPN_BCE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

Commit message: V0.1 wolfspeed
Routing:
- net VCC_IN: track 103.4 -> 98.2 mm
Changed lines of the file:
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@@
     (thickness 1.6)
     (drawings 15)
-    (tracks 785)
+    (tracks 781)
     (zones 0)
     (modules 118)
@@
   )
   (setup
-    (last_trace_width 2)
+    (last_trace_width 0.25)
     (user_trace_width 1)
     (user_trace_width 2)
@@
   (segment (start 13.5 70.339196) (end 14.663398 69.175798) (width 0.25) (layer F.Cu) (net 34))
   (segment (start 14.663398 69.175798) (end 17.4128 69.175798) (width 0.25) (layer F.Cu) (net 34))
-  (segment (start 41.9862 82.2452) (end 42.9514 82.2452) (width 2) (layer B.Cu) (net 55))
-  (segment (start 40.005 82.2452) (end 40.9956 82.2452) (width 2) (layer B.Cu) (net 55))
-  (segment (start 45.847 72.8472) (end 45.847 71.755) (width 2) (layer B.Cu) (net 55))
-  (segment (start 45.847 72.8472) (end 45.847 70.6882) (width 2) (layer B.Cu) (net 55))
   (segment (start 11.0236 74.2736) (end 11.0236 78.504515) (width 0.25) (layer F.Cu) (net 62))
   (segment (start 20.721981 84.8106) (end 13.0302 84.8106) (width 0.25) (layer B.Cu) (net 62))
