File: V0.2-IGBT/PCB/ENNOID Dual Gate Driver.kicad_pcb (KiCad board)
At the start: 2 copper layers, 60 x 98 mm, 118 parts, among them J1 Conn_02x08_Odd_Even, J2 Current, J3 TEMP, J4 PHASE, J5 Collector, J6 Gate_H, J7 G_L, J8 E, Q1 Q_NPN_BCE, Q2 Q_NPN_BCE, U1 MC7805, U2 MGJ2, U3 MGJ2, U4 1ED020I12-F2, U5 IXD-609, U6 1ED020I12-F2, U7 IXD-609, U8 AMC1301

Commit message: v0.2 PCB
Parts:
- removed D5, D8: D_Zener, Diodes_SMD:D_SOD-123
- removed R44, R45: DNP, Resistors_SMD:R_0805_HandSoldering
- removed REF** (x3): MountingHole_2.2mm_M2_DIN965_Pad, Mounting_Holes:MountingHole_2.2mm_M2_DIN965_Pad
- removed U6: 1ED020I12-F2, Housings_SOIC:SOIC-16W_7.5x10.3mm_Pitch1.27mm
- removed U7: IXD-609, Housings_SOIC:SOIC-8-1EP_3.9x4.9mm_Pitch1.27mm
- added C45: 100n, Capacitors_SMD:C_0805_HandSoldering, F.Cu at (57.3, 45.2)
- added C46: 1u, Capacitors_SMD:C_0805_HandSoldering, F.Cu at (52.6, 41.0)
- added C47: 1u, Capacitors_SMD:C_0805_HandSoldering, F.Cu at (57.7, 41.0)
- added C48: 220p, Capacitors_SMD:C_0805_HandSoldering, B.Cu at (42.1, 19.1)
- added C49: 10u, Capacitors_SMD:C_1206_HandSoldering, B.Cu at (51.7, 32.1)
- added C50: 100n, Capacitors_SMD:C_0805_HandSoldering, B.Cu at (54.4, 23.5)
- added C51: 100n, Capacitors_SMD:C_0805_HandSoldering, B.Cu at (48.2, 23.7)
- added C52: 1u, Capacitors_SMD:C_0805_HandSoldering, B.Cu at (54.5, 25.5)
- added C53: 1u, Capacitors_SMD:C_0805_HandSoldering, B.Cu at (48.1, 25.5)
- added C54: 10u, Capacitors_SMD:C_1206_HandSoldering, B.Cu at (54.7, 29.8)
- added C55: 10u, Capacitors_SMD:C_1206_HandSoldering, B.Cu at (48.2, 27.6)
- added C56: 10u, Capacitors_SMD:C_1206_HandSoldering, B.Cu at (54.8, 27.6)
- added C57: 10u, Capacitors_SMD:C_1206_HandSoldering, B.Cu at (48.2, 29.9)
- added C58: 0.22u, Capacitors_SMD:C_0805_HandSoldering, B.Cu at (42.1, 13.3)
- added D15: smcj440ca, Diodes_SMD:D_SMC_Handsoldering, F.Cu at (7.52, 4.62)
- added D16: es2j-ltp, Diodes_SMD:D_SMA_Handsoldering, B.Cu at (7.57, 4.62)
- added D17: 1N4148W, Diodes_SMD:D_SOD-123, F.Cu at (57.3, 62.8)
- added D18: MMSZ5242BS, Diodes_SMD:D_SOD-323, B.Cu at (42.4, 20.9)
- added D19: BAT54WS-7-F, Diodes_SMD:D_SOD-323_HandSoldering, B.Cu at (42.2, 17.1)
- added D20: SMAJ18CA, Diodes_SMD:D_SMA_Handsoldering, B.Cu at (40.9, 10.6)
- added D21: smcj440ca, Diodes_SMD:D_SMC_Handsoldering, F.Cu at (30.4, 7.21)
- added D22: es2j-ltp, Diodes_SMD:D_SMA_Handsoldering, B.Cu at (30.3, 7.16)
- added Q3: MJD44H11RLG, TO_SOT_Packages_SMD:TO-252-3_TabPin4, F.Cu at (18.3, 25.7)
- added Q4: MJD45H11RLG, TO_SOT_Packages_SMD:TO-252-3_TabPin4, F.Cu at (11.2, 25.7)
- added Q5: MJD44H11RLG, TO_SOT_Packages_SMD:TO-252-3_TabPin4, F.Cu at (55.4, 25.7)
- added Q6: MJD45H11RLG, TO_SOT_Packages_SMD:TO-252-3_TabPin4, F.Cu at (48.3, 25.7)
- added R35: 12, Resistors_SMD:R_0805_HandSoldering, F.Cu at (48.3, 43.3)
- added R36: 3, Resistors_SMD:R_2512_HandSoldering, F.Cu at (57.6, 14.4)
- added R37: 3, Resistors_SMD:R_2512_HandSoldering, F.Cu at (53.7, 14.4)
- added R38: 3, Resistors_SMD:R_2512_HandSoldering, F.Cu at (46.1, 14.4)
- added R39: 3, Resistors_SMD:R_2512_HandSoldering, F.Cu at (49.9, 14.4)
- added R40: 10k, Resistors_SMD:R_0805_HandSoldering, B.Cu at (42.2, 15.2)
- C17: value 100n -> 15n
- C19, C36: value DNP -> 100n
- C20: value 100n -> 1u
- C21: value 4.7u -> 1u; footprint Capacitors_SMD:C_1206_HandSoldering -> Capacitors_SMD:C_0805_HandSoldering
- C22: value 10n -> 220p
- C23, C31: value 100n -> 10u; footprint Capacitors_SMD:C_0805_HandSoldering -> Capacitors_SMD:C_1206_HandSoldering
- C24: value 10u -> 100n; footprint Resistors_SMD:R_1210_HandSoldering -> Capacitors_SMD:C_0805_HandSoldering
- C25: value DNP -> 100n; moved to B.Cu
- C28, C29: value 100n -> 1u; moved to B.Cu
- C30: value DNP -> 10u; footprint Capacitors_SMD:C_0805_HandSoldering -> Capacitors_SMD:C_1206_HandSoldering; moved to B.Cu
- C32: value 4.7u -> 10u
- C33: value 10n -> 10u; footprint Capacitors_SMD:C_0805_HandSoldering -> Capacitors_SMD:C_1206_HandSoldering; moved to B.Cu
- C34: value 100n -> 0.22u; moved to B.Cu
- C35: value 10u -> 15n; footprint Resistors_SMD:R_1210_HandSoldering -> Capacitors_SMD:C_0805_HandSoldering
- D10: value D -> BAT54WS-7-F; footprint Diodes_SMD:D_SMA_Handsoldering -> Diodes_SMD:D_SOD-323_HandSoldering; moved to B.Cu
- D11: value D -> SMAJ18CA; moved to B.Cu
- D3: value D_Zener -> 1N4148W
- D4, D7: value D -> sTth112
- D6: value D_Zener -> MMSZ5242BS; footprint Diodes_SMD:D_SOD-123 -> Diodes_SMD:D_SOD-323; moved to B.Cu
- R10: moved to B.Cu
- R11, R12: value DND -> 12; footprint Resistors_SMD:R_MELF_MMB-0207 -> Resistors_SMD:R_0805_HandSoldering
- R13, R25: value 20 -> 12; footprint Resistors_SMD:R_MELF_MMB-0207 -> Resistors_SMD:R_0805_HandSoldering
- R14: value 20 -> 3; footprint Resistors_SMD:R_MELF_MMB-0207 -> Resistors_SMD:R_2512_HandSoldering
- R15: value 47k -> 3; footprint Resistors_SMD:R_0805_HandSoldering -> Resistors_SMD:R_2512_HandSoldering
- R22, R23: value DND -> 3; footprint Resistors_SMD:R_MELF_MMB-0207 -> Resistors_SMD:R_2512_HandSoldering; moved to F.Cu
- R24: value 20 -> 10k; footprint Resistors_SMD:R_MELF_MMB-0207 -> Resistors_SMD:R_0805_HandSoldering; moved to B.Cu
- R26: value 47k -> 12
- U4: value 1ED020I12-F2 -> ISO5852SDWR
- U5: value IXD-609 -> ISO5852SDWR; footprint Housings_SOIC:SOIC-8-1EP_3.9x4.9mm_Pitch1.27mm -> Housings_SOIC:SOIC-16W_7.5x10.3mm_Pitch1.27mm
- moved R23 45.2 mm to (9.07, 14.5), turned to 270 degrees
- moved C29 43.6 mm to (11.5, 23.9), turned to 0 degrees
- moved U5 43.1 mm to (51.2, 52.9), turned to 270 degrees
- moved C30 40.8 mm to (18.1, 27.9)
- moved C31 40.1 mm to (11.4, 30.1)
- moved D6 38.1 mm to (22.5, 21.3), turned to 0 degrees
- moved R22 38.0 mm to (12.9, 14.5), turned to 270 degrees
- moved D11 36.6 mm to (22.3, 10.6), turned to 0 degrees
- moved C36 36.0 mm to (52.7, 44.8)
- moved R26 34.8 mm to (46.5, 43.3), turned to 270 degrees
- moved C32 34.0 mm to (18.0, 30.1), turned to 180 degrees
- moved C28 31.8 mm to (17.9, 25.8), turned to 180 degrees
- moved R24 31.6 mm to (22.6, 15.5), turned to 180 degrees
- moved C33 30.4 mm to (11.4, 27.9), turned to 0 degrees
- moved D3 25.2 mm to (22.9, 62.7), turned to 270 degrees
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Connections:
- C17 pad 1: /GD_HIGH/-VEE -> Net-(C17-Pad1)
- C17 pad 2: PHASE -> /GD_HIGH/-VEE
- C18 pad 1: PHASE -> /GD_HIGH/VCC_REG
- C18 pad 2: /GD_HIGH/VCC_REG -> Net-(C18-Pad2)
- C19 pad 1: Net-(C19-Pad1) -> Net-(C18-Pad2)
- C19 pad 2: PHASE -> /GD_HIGH/-VEE
- C20 pad 1: /GD_HIGH/+VCC -> /GD_HIGH/VCC_REG
- C20 pad 2: /GD_HIGH/-VEE -> Net-(C18-Pad2)
- C21 pad 1: /GD_HIGH/+VCC -> Net-(C18-Pad2)
- C22 pad 1: PHASE -> Net-(C22-Pad1)
- C22 pad 2: /GD_HIGH/-VEE -> PHASE
- C23 pad 1: PHASE -> /GD_HIGH/+VCC
- C24 pad 1: PHASE -> /GD_HIGH/+VCC
- C24 pad 2: /GD_HIGH/-VEE -> PHASE
- C25 pad 1: /GD_HIGH/G -> PHASE
- C25 pad 2: PHASE -> /GD_HIGH/-VEE
- C28 pad 1: /GD_LOW/-VEE -> /GD_HIGH/+VCC
- C28 pad 2: /GD_LOW/E -> PHASE
- C29 pad 1: /GD_LOW/E -> PHASE
- C29 pad 2: /GD_LOW/VCC_REG -> /GD_HIGH/-VEE
- C30 pad 1: Net-(C30-Pad1) -> /GD_HIGH/+VCC
- C30 pad 2: /GD_LOW/E -> PHASE
- C31 pad 1: /GD_LOW/+VCC -> PHASE
- C31 pad 2: /GD_LOW/-VEE -> /GD_HIGH/-VEE
- C32 pad 1: /GD_LOW/+VCC -> /GD_HIGH/+VCC
- C32 pad 2: /GD_LOW/-VEE -> PHASE
- C33 pad 1: /GD_LOW/E -> PHASE
- C33 pad 2: /GD_LOW/-VEE -> /GD_HIGH/-VEE
- C34 pad 1: /GD_LOW/E -> /GD_HIGH/G
- C34 pad 2: /GD_LOW/-VEE -> PHASE
- C35 pad 1: /GD_LOW/E -> Net-(C35-Pad1)
- C36 pad 1: /GD_LOW/G -> /GD_LOW/VCC_REG
- C36 pad 2: /GD_LOW/E -> Net-(C36-Pad2)
- D10 pad 1: Net-(D10-Pad1) -> Net-(C22-Pad1)
- D10 pad 2: Net-(D10-Pad2) -> PHASE
- D11 pad 1: Net-(D11-Pad1) -> /GD_HIGH/G
- D11 pad 2: Net-(D11-Pad2) -> PHASE
- D3 pad 1: Net-(C19-Pad1) -> FLT
- D3 pad 2: PHASE -> Net-(C15-Pad1)
- D4 pad 1: Net-(D4-Pad1) -> /GD_HIGH/C
- D6 pad 1: Net-(C30-Pad1) -> Net-(C22-Pad1)
- D6 pad 2: /GD_LOW/E -> PHASE
- D7 pad 1: Net-(D7-Pad1) -> PHASE
- J1 pad 7: Net-(J1-Pad7) -> (no net)
- J1 pad 8: Net-(J1-Pad8) -> (no net)
- R10 pad 2: Net-(C19-Pad1) -> Net-(C22-Pad1)
- R11 pad 1: Net-(D10-Pad2) -> Net-(C17-Pad1)
- R11 pad 2: /GD_HIGH/G -> Net-(R11-Pad2)
- R12 pad 1: Net-(D10-Pad2) -> Net-(Q3-Pad1)
- R12 pad 2: /GD_HIGH/G -> Net-(R12-Pad2)
- R13 pad 1: Net-(D10-Pad1) -> Net-(Q3-Pad1)
- R13 pad 2: /GD_HIGH/G -> Net-(R11-Pad2)
- R14 pad 1: Net-(D10-Pad1) -> /GD_HIGH/G
- R14 pad 2: /GD_HIGH/G -> Net-(Q3-Pad3)
- R15 pad 2: PHASE -> Net-(Q3-Pad3)
- R21 pad 2: Net-(C30-Pad1) -> Net-(C48-Pad1)
- R22 pad 1: Net-(D11-Pad2) -> /GD_HIGH/G
- R22 pad 2: /GD_LOW/G -> Net-(Q4-Pad3)
- R23 pad 1: Net-(D11-Pad2) -> /GD_HIGH/G
- R23 pad 2: /GD_LOW/G -> Net-(Q4-Pad3)
- R24 pad 1: Net-(D11-Pad1) -> PHASE
- R24 pad 2: /GD_LOW/G -> /GD_HIGH/G
- R25 pad 1: Net-(D11-Pad1) -> Net-(C35-Pad1)
- R25 pad 2: /GD_LOW/G -> Net-(R25-Pad2)
- R26 pad 1: /GD_LOW/G -> Net-(Q5-Pad1)
- R26 pad 2: /GD_LOW/E -> Net-(R26-Pad2)
- U4 pad 2: Net-(C19-Pad1) -> Net-(C22-Pad1)
- U4 pad 3: PHASE -> Net-(C18-Pad2)
- U4 pad 4: Net-(R44-Pad1) -> Net-(R12-Pad2)
- U4 pad 6: Net-(R44-Pad2) -> Net-(R11-Pad2)
- U4 pad 7: Net-(U4-Pad7) -> (no net)
- U5 pad 1: /GD_HIGH/+VCC -> /GD_LOW/-VEE
- U5 pad 2: Net-(R44-Pad2) -> Net-(C48-Pad1)
- U5 pad 3: Net-(U5-Pad3) -> Net-(C36-Pad2)
- U5 pad 4: /GD_HIGH/-VEE -> Net-(R26-Pad2)
- U5 pad 5: /GD_HIGH/-VEE -> /GD_LOW/VCC_REG
- U5 pad 6: Net-(D10-Pad1) -> Net-(R25-Pad2)
- U5 pad 7: Net-(D10-Pad1) -> (no net)
- U5 pad 8: /GD_HIGH/+VCC -> /GD_LOW/-VEE
- U5 pad 9: (no net) -> GND
Routing:
- net FLT: track 106.2 -> 0.00 mm, vias 4 -> 0
- net VCC_IN: track 103.4 -> 0.00 mm, vias 9 -> 0
- net RST: track 93.5 -> 0.00 mm, vias 3 -> 0
- net RDY: track 74.1 -> 0.00 mm, vias 4 -> 0
- net (no net): track 53.0 -> 0.00 mm
- net /GD_LOW/-VEE: track 51.6 -> 0.00 mm, vias 15 -> 0
- net PWM_H: track 50.4 -> 0.00 mm, vias 3 -> 0
- net PHASE: track 48.0 -> 0.00 mm, vias 15 -> 0
- net PWM_L: track 47.0 -> 0.00 mm, vias 1 -> 0
- net +5V: track 46.2 -> 0.00 mm, vias 13 -> 0
- net Vout+: track 44.1 -> 0.00 mm, vias 2 -> 0
- net Net-(C30-Pad1): track 41.7 -> 0.00 mm, vias 2 -> 0
- net Vout-: track 40.8 -> 0.00 mm, vias 2 -> 0
- net Net-(C19-Pad1): track 38.9 -> 0.00 mm, vias 2 -> 0
- net Net-(C38-Pad1): track 27.8 -> 0.00 mm, vias 1 -> 0
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- removed copper zone on B.Cu, net /GD_LOW/-VEE

Commit message: v0.2
Parts:
- C18, C35, C45, C47, R26, R35: moved to B.Cu
- C21, C22, C23, C49, D10, D6, R12: moved to F.Cu
- D15, D21: footprint Diodes_SMD:D_SMC_Handsoldering -> Diodes_SMD:D_SMC
- Q3, Q4, Q5, Q6: footprint TO_SOT_Packages_SMD:TO-252-3_TabPin4 -> TO_SOT_Packages_SMD:TO-252-2
- moved D10 25.9 mm to (2.16, 33.6), turned to 270 degrees
- moved C22 23.2 mm to (4.09, 33.5), turned to 270 degrees
- moved D6 20.5 mm to (5.99, 33.6), turned to 270 degrees
- moved R11 14.3 mm to (13.0, 43.6), turned to 270 degrees
- moved D19 13.8 mm to (34.6, 28.7), turned to 0 degrees
- moved C17 12.6 mm to (13.0, 43.6)
- moved C48 10.5 mm to (34.9, 26.8), turned to 0 degrees
- moved C50 9.48 mm to (47.8, 30.3), turned to 0 degrees
- moved C54 9.31 mm to (47.5, 24.0), turned to 0 degrees
- moved C29 9.30 mm to (18.0, 30.5)
- moved C24 9.13 mm to (11.6, 30.4), turned to 0 degrees
- moved C35 9.00 mm to (56.2, 41.6), turned to 0 degrees
- moved C31 8.96 mm to (18.1, 24.2)
- moved C32 8.90 mm to (11.4, 24.2), turned to 0 degrees
- moved C51 8.77 mm to (54.1, 30.1), turned to 0 degrees
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Connections:
- J1 pad 7: (no net) -> Net-(J1-Pad7)
- J1 pad 8: (no net) -> Net-(J1-Pad8)
- U4 pad 7: (no net) -> Net-(U4-Pad7)
- U5 pad 7: (no net) -> Net-(U5-Pad7)
Routing:
- net /GD_LOW/E: track 0.00 -> 97.2 mm, vias 0 -> 8
- net Net-(Q5-Pad1): track 0.00 -> 49.7 mm, vias 0 -> 2
- net /GD_LOW/-VEE: track 0.00 -> 28.2 mm, vias 0 -> 6
- net /GD_LOW/+VCC: track 0.00 -> 20.4 mm, vias 0 -> 4
- net PHASE: track 0.00 -> 17.3 mm
- net Net-(R25-Pad2): track 0.00 -> 17.0 mm, vias 0 -> 2
- net /GD_LOW/G: track 0.00 -> 16.7 mm
- net /GD_LOW/VCC_REG: track 0.00 -> 16.6 mm, vias 0 -> 1
- net Net-(Q5-Pad3): track 0.00 -> 12.9 mm
- net Net-(Q3-Pad3): track 0.00 -> 12.8 mm
- net Net-(D15-Pad2): track 0.00 -> 12.7 mm, vias 0 -> 1
- net Net-(Q6-Pad3): track 0.00 -> 12.2 mm
- net Net-(Q4-Pad3): track 0.00 -> 12.1 mm
- net Net-(D21-Pad2): track 0.00 -> 11.0 mm, vias 0 -> 1
- net Net-(C22-Pad1): track 0.00 -> 10.8 mm, vias 0 -> 1
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- added copper zone on B.Cu, net /GD_LOW/-VEE
- added copper zone on B.Cu, net /GD_LOW/E
- added copper zone on B.Cu, net PHASE

Commit message: v0.2 PCB POWER STAGE COMPLETED
Parts:
- removed C14, C9: 1u, Capacitors_SMD:C_0805_HandSoldering
- removed D1, D2: MMSZ5251B, Diodes_SMD:D_SOD-123
- removed Q1, Q2: Q_NPN_BCE, TO_SOT_Packages_SMD:SOT-89-3_Handsoldering
- removed R1, R3: 10k, Resistors_SMD:R_0805_HandSoldering
- removed R2, R4: 0, Resistors_SMD:R_0805_HandSoldering
- C17, C19, C21, R12, R13: moved to B.Cu
- C18, C20, C48, D18, D19, R11: moved to F.Cu
- moved D18 11.7 mm to (29.5, 35.4), turned to 270 degrees
- moved C17 9.83 mm to (22.6, 41.4), turned to 0 degrees
- moved C48 9.01 mm to (33.5, 35.7), turned to 270 degrees
- moved D19 7.44 mm to (31.5, 35.5), turned to 270 degrees
- moved R12 6.28 mm to (15.5, 37.8)
- moved R13 6.08 mm to (13.6, 37.8)
- moved D9 4.42 mm to (31.8, 38.5), turned to 0 degrees
- moved R11 4.18 mm to (16.5, 41.4), turned to 180 degrees
- moved C19 1.30 mm to (22.6, 45.0)
- moved C21 1.30 mm to (22.6, 43.2)
- moved C22 0.64 mm to (3.45, 33.5)
- moved D10 0.63 mm to (1.52, 33.6)
- moved D6 0.63 mm to (5.36, 33.6)
- moved C37 0.63 mm to (33.7, 42.9)
- moved R30 0.63 mm to (31.7, 42.9)
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Connections:
- C18 pad 1: /GD_HIGH/VCC_REG -> /GD_HIGH/+VCC
- C20 pad 1: /GD_HIGH/VCC_REG -> /GD_HIGH/+VCC
- C36 pad 1: /GD_LOW/VCC_REG -> /GD_LOW/+VCC
- C46 pad 1: /GD_LOW/VCC_REG -> /GD_LOW/+VCC
- J1 pad 7: Net-(J1-Pad7) -> (no net)
- J1 pad 8: Net-(J1-Pad8) -> (no net)
- U4 pad 5: /GD_HIGH/VCC_REG -> /GD_HIGH/+VCC
- U4 pad 7: Net-(U4-Pad7) -> (no net)
- U5 pad 5: /GD_LOW/VCC_REG -> /GD_LOW/+VCC
- U5 pad 7: Net-(U5-Pad7) -> (no net)
Routing:
- net PHASE: track 17.3 -> 130.9 mm, vias 0 -> 5
- net /GD_HIGH/+VCC: track 5.48 -> 58.0 mm, vias 0 -> 5
- net Net-(Q3-Pad1): track 0.00 -> 46.4 mm, vias 0 -> 2
- net /GD_HIGH/-VEE: track 3.22 -> 47.1 mm, vias 0 -> 6
- net Net-(C48-Pad1): track 0.00 -> 39.7 mm, vias 0 -> 2
- net /GD_LOW/+VCC: track 20.4 -> 56.3 mm, vias 4 -> 5
- net Net-(C22-Pad1): track 10.8 -> 42.2 mm, vias 1 -> 3
- net /GD_LOW/E: track 97.2 -> 125.8 mm, vias 8 -> 6
- net Net-(C38-Pad1): track 5.32 -> 27.9 mm
- net /GD_LOW/VCC_REG: track 16.6 -> 0.00 mm, vias 1 -> 0
- net Net-(R11-Pad2): track 0.00 -> 11.4 mm, vias 0 -> 2
- net Net-(C18-Pad2): track 0.00 -> 10.7 mm, vias 0 -> 1
- net Net-(R12-Pad2): track 0.00 -> 10.1 mm, vias 0 -> 1
- net Net-(D2-Pad1): track 8.00 -> 0.00 mm, vias 1 -> 0
- net /GD_HIGH/C: track 3.77 -> 11.2 mm
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
Commit message: v2.0 PCB SIGNAL SIDE
Parts:
- moved D14 14.1 mm to (17.5, 77.4)
- moved R34 14.1 mm to (17.5, 82.4)
- moved D12 13.7 mm to (26.0, 77.3)
- moved D13 13.7 mm to (21.5, 77.3)
- moved R16 13.7 mm to (21.5, 82.3)
- moved R5 13.7 mm to (26.0, 82.3)
- moved C41 3.80 mm to (35.6, 84.8)
- moved D3 1.73 mm to (21.2, 62.6)
- moved D17 1.37 mm to (55.9, 62.8)
- moved C42 0.36 mm to (33.7, 84.8)
- turned C27 to 0 degrees
Connections:
- C41 pad 1: PWM_H -> PWM_L
- C42 pad 1: PWM_L -> PWM_H
- J1 pad 11: PWM_H -> PWM_L
- J1 pad 12: PWM_L -> PWM_H
- J1 pad 3: Vout+ -> Vout-
- J1 pad 4: Vout- -> Vout+
Routing:
- net VCC_IN: track 0.00 -> 66.0 mm
- net Vout-: track 0.00 -> 39.6 mm, vias 0 -> 2
- net Vout+: track 0.00 -> 36.5 mm, vias 0 -> 2
- net PWM_L: track 0.00 -> 36.5 mm, vias 0 -> 1
- net RST: track 0.00 -> 35.8 mm
- net PWM_H: track 0.00 -> 35.4 mm, vias 0 -> 1
- net +5V: track 0.00 -> 24.1 mm, vias 0 -> 14
- net Net-(C26-Pad1): track 0.00 -> 20.5 mm, vias 0 -> 2
- net Net-(C15-Pad1): track 0.00 -> 20.4 mm, vias 0 -> 2
- net TEMP: track 0.00 -> 18.5 mm
- net GND: track 0.00 -> 18.1 mm, vias 0 -> 10
- net Net-(C10-Pad2): track 0.00 -> 16.3 mm
- net Net-(C5-Pad2): track 0.00 -> 16.1 mm
- net Net-(C10-Pad1): track 0.00 -> 12.0 mm
- net Net-(C5-Pad1): track 0.00 -> 11.9 mm
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
Commit message: SIGNAL PCV V0.2
Parts:
- R16, R34, R5: moved to B.Cu
- R19, R8: moved to F.Cu
- moved R34 24.1 mm to (25.4, 59.7), turned to 270 degrees
- moved D14 19.4 mm to (25.4, 59.7)
- moved D12 11.8 mm to (14.7, 80.6), turned to 180 degrees
- moved R5 11.5 mm to (14.7, 80.5), turned to 180 degrees
- moved D13 5.26 mm to (25.7, 80.5), turned to 0 degrees
- moved C42 4.84 mm to (31.5, 89.1), turned to 180 degrees
- moved R16 4.53 mm to (25.7, 80.5), turned to 0 degrees
- moved C41 4.32 mm to (36.1, 89.1), turned to 0 degrees
- moved R19 2.72 mm to (47.5, 63.9), turned to 90 degrees
- moved R8 2.55 mm to (13.6, 63.8), turned to 90 degrees
- moved R7 1.22 mm to (19.3, 63.8)
- moved R9 1.22 mm to (17.4, 63.8)
- moved D3 1.22 mm to (21.4, 63.8)
- moved R6 1.20 mm to (15.5, 63.8)
- moved C15 1.17 mm to (13.9, 57.7)
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Routing:
- net RDY: track 4.34 -> 38.4 mm
- net FLT: track 6.93 -> 29.6 mm, vias 0 -> 1
- net Net-(C15-Pad1): track 20.4 -> 0.01 mm, vias 2 -> 0
- net Net-(C26-Pad1): track 20.5 -> 0.27 mm, vias 2 -> 0
- net GND: track 18.1 -> 5.53 mm, vias 10 -> 3
- net RST: track 35.8 -> 26.1 mm, vias 0 -> 1
- net PWM_H: track 35.4 -> 44.4 mm, vias 1 -> 3
- net +5V: track 24.1 -> 15.5 mm, vias 14 -> 10
- net PWM_L: track 36.5 -> 43.3 mm
- net Net-(D14-Pad2): track 2.30 -> 0.00 mm
- net Net-(D13-Pad2): track 2.30 -> 0.00 mm
- net Net-(D12-Pad2): track 2.30 -> 0.00 mm
- net Vout+: track 36.5 -> 37.1 mm, vias 2 -> 1
- net Vout-: vias 2 -> 1

Commit message: V0.2 PCB completed
Parts:
- moved D13 11.8 mm to (13.9, 80.5), turned to 180 degrees
- moved R16 11.8 mm to (13.9, 80.5), turned to 180 degrees
- moved D12 8.26 mm to (23.0, 80.4), turned to 0 degrees
- moved R5 8.26 mm to (23.0, 80.4), turned to 0 degrees
Routing:
- net FLT: track 29.6 -> 104.0 mm, vias 1 -> 3
- net RST: track 26.1 -> 89.7 mm, vias 1 -> 3
- net Net-(C26-Pad1): track 0.27 -> 27.4 mm, vias 0 -> 3
- net Net-(C15-Pad1): track 0.01 -> 24.3 mm, vias 0 -> 2
- net +5V: track 15.5 -> 30.2 mm, vias 10 -> 13
- net RDY: track 38.4 -> 49.2 mm
- net GND: track 5.53 -> 15.9 mm, vias 3 -> 7
- net Net-(D13-Pad2): track 0.00 -> 3.13 mm, vias 0 -> 1
- net Net-(D12-Pad2): track 0.00 -> 3.04 mm, vias 0 -> 1
- net PWM_L: track 43.3 -> 42.3 mm
- net PWM_H: track 44.4 -> 43.7 mm
- net /GD_HIGH/+VCC: track 58.0 -> 57.5 mm

Commit message: V0.2 completed
Parts:
- added C9: 10u, Capacitors_SMD:C_0805_HandSoldering, B.Cu at (31.7, 43.0)
- added REF**: MountingHole_3.2mm_M3_ISO7380_Pad, Mounting_Holes:MountingHole_3.2mm_M3_ISO7380_Pad, F.Cu at (55.0, 93.0)
- added REF**: MountingHole_3.2mm_M3_ISO7380_Pad, Mounting_Holes:MountingHole_3.2mm_M3_ISO7380_Pad, F.Cu at (5.00, 93.0)
- D9: value 5V -> 5V
- R28: value 200 -> 800
- moved J3 0.31 mm to (48.2, 93.2)
- moved J2 0.19 mm to (11.7, 88.2)
Connections:
- J1 pad 7: (no net) -> Net-(J1-Pad7)
- J1 pad 8: (no net) -> Net-(J1-Pad8)
- U4 pad 7: (no net) -> Net-(U4-Pad7)
- U5 pad 7: (no net) -> Net-(U5-Pad7)
Routing:
- net /GD_HIGH/C: track 11.2 -> 14.9 mm
- net GND: track 15.9 -> 19.0 mm, vias 7 -> 8
- net Net-(D14-Pad2): track 0.00 -> 2.90 mm, vias 0 -> 1
- net /GD_LOW/E: track 125.8 -> 128.5 mm
- net FLT: track 104.0 -> 106.0 mm
- net Net-(C37-Pad1): track 13.0 -> 14.5 mm
- net PWM_H: track 43.7 -> 43.0 mm
- net Net-(C26-Pad1): track 27.4 -> 26.8 mm
