File: V0.2-IGBT/PCB/ENNOID Dual Gate Driver.kicad_pcb (KiCad board)
At the start: 2 copper layers, 60 x 98 mm, 134 parts, among them J1 Conn_02x08_Odd_Even, J2 Current, J3 TEMP, J4 PHASE, J5 Collector, J6 Gate_H, J7 G_L, J8 E, Q3 MJD44H11RLG, Q4 MJD45H11RLG, Q5 MJD44H11RLG, Q6 MJD45H11RLG, U1 MC7805, U2 MGJ2, U3 MGJ2, U4 ISO5852SDWR, U5 ISO5852SDWR, U8 AMC1301

Commit message: PCB V0.2
Routing:
- net /GD_LOW/G: vias 0 -> 45
- net /GD_HIGH/G: vias 0 -> 30
Changed lines of the file:
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@@
     (thickness 1.6)
     (drawings 15)
-    (tracks 816)
+    (tracks 891)
     (zones 0)
     (modules 134)
@@
   (segment (start 14.0282 57.5776) (end 14.0282 58.5544) (width 0.25) (layer F.Cu) (net 13))
   (segment (start 14.0208 57.585) (end 14.0282 57.5776) (width 0.25) (layer F.Cu) (net 13))
+  (via (at 16.7978 14.5984) (size 0.8) (drill 0.4) (layers F.Cu B.Cu) (net 14))
+  (via (at 15.7978 14.5984) (size 0.8) (drill 0.4) (layers F.Cu B.Cu) (net 14))
+  (via (at 14.7978 14.5984) (size 0.8) (drill 0.4) (layers F.Cu B.Cu) (net 14))
+  (via (at 13.7978 14.5984) (size 0.8) (drill 0.4) (layers F.Cu B.Cu) (net 14))
+  (via (at 12.7978 14.5984) (size 0.8) (drill 0.4) (layers F.Cu B.Cu) (net 14))
+  (via (at 11.7978 14.5984) (size 0.8) (drill 0.4) (layers F.Cu B.Cu) (net 14))
+  (via (at 10.7978 14.5984) (size 0.8) (drill 0.4) (layers F.Cu B.Cu) (net 14))
+  (via (at 9.7978 14.5984) (size 0.8) (drill 0.4) (layers F.Cu B.Cu) (net 14))
+  (via (at 8.7978 14.5984) (size 0.8) (drill 0.4) (layers F.Cu B.Cu) (net 14))
+  (via (at 7.7978 14.5984) (size 0.8) (drill 0.4) (layers F.Cu B.Cu) (net 14))
+  (via (at 16.7978 13.5984) (size 0.8) (drill 0.4) (layers F.Cu B.Cu) (net 14))
+  (via (at 15.7978 13.5984) (size 0.8) (drill 0.4) (layers F.Cu B.Cu) (net 14))
+  (via (at 14.7978 13.5984) (size 0.8) (drill 0.4) (layers F.Cu B.Cu) (net 14))
+  (via (at 13.7978 13.5984) (size 0.8) (drill 0.4) (layers F.Cu B.Cu) (net 14))
+  (via (at 12.7978 13.5984) (size 0.8) (drill 0.4) (layers F.Cu B.Cu) (net 14))
+  (via (at 11.7978 13.5984) (size 0.8) (drill 0.4) (layers F.Cu B.Cu) (net 14))
+  (via (at 10.7978 13.5984) (size 0.8) (drill 0.4) (layers F.Cu B.Cu) (net 14))
+  (via (at 9.7978 13.5984) (size 0.8) (drill 0.4) (layers F.Cu B.Cu) (net 14))
+  (via (at 8.7978 13.5984) (size 0.8) (drill 0.4) (layers F.Cu B.Cu) (net 14))
+  (via (at 7.7978 13.5984) (size 0.8) (drill 0.4) (layers F.Cu B.Cu) (net 14))
+  (via (at 16.7978 12.5984) (size 0.8) (drill 0.4) (layers F.Cu B.Cu) (net 14))
+  (via (at 15.7978 12.5984) (size 0.8) (drill 0.4) (layers F.Cu B.Cu) (net 14))
+  (via (at 14.7978 12.5984) (size 0.8) (drill 0.4) (layers F.Cu B.Cu) (net 14))
+  (via (at 13.7978 12.5984) (size 0.8) (drill 0.4) (layers F.Cu B.Cu) (net 14))
+  (via (at 12.7978 12.5984) (size 0.8) (drill 0.4) (layers F.Cu B.Cu) (net 14))
+  (via (at 11.7978 12.5984) (size 0.8) (drill 0.4) (layers F.Cu B.Cu) (net 14))
+  (via (at 10.7978 12.5984) (size 0.8) (drill 0.4) (layers F.Cu B.Cu) (net 14))
+  (via (at 9.7978 12.5984) (size 0.8) (drill 0.4) (layers F.Cu B.Cu) (net 14))
+  (via (at 8.7978 12.5984) (size 0.8) (drill 0.4) (layers F.Cu B.Cu) (net 14))
+  (via (at 7.7978 12.5984) (size 0.8) (drill 0.4) (layers F.Cu B.Cu) (net 14))
   (segment (start 49.4284 62.531) (end 49.4284 60.0964) (width 0.25) (layer F.Cu) (net 15))
   (segment (start 49.4284 60.0964) (end 48.977499 59.645499) (width 0.25) (layer F.Cu) (net 15))
@@
   (segment (start 47.5234 62.531) (end 49.4284 62.531) (width 0.25) (layer F.Cu) (net 15))
   (segment (start 49.4284 62.531) (end 49.4284 62.3856) (width 0.25) (layer F.Cu) (net 15))
+  (via (at 57.9674 14.7254) (size 0.8) (drill 0.4) (layers F.Cu B.Cu) (net 16))
+  (via (at 56.9674 14.7254) (size 0.8) (drill 0.4) (layers F.Cu B.Cu) (net 16))
+  (via (at 55.9674 14.7254) (size 0.8) (drill 0.4) (layers F.Cu B.Cu) (net 16))
+  (via (at 54.9674 14.7254) (size 0.8) (drill 0.4) (layers F.Cu B.Cu) (net 16))
+  (via (at 53.9674 14.7254) (size 0.8) (drill 0.4) (layers F.Cu B.Cu) (net 16))
+  (via (at 52.9674 14.7254) (size 0.8) (drill 0.4) (layers F.Cu B.Cu) (net 16))
+  (via (at 51.9674 14.7254) (size 0.8) (drill 0.4) (layers F.Cu B.Cu) (net 16))
+  (via (at 50.9674 14.7254) (size 0.8) (drill 0.4) (layers F.Cu B.Cu) (net 16))
+  (via (at 49.9674 14.7254) (size 0.8) (drill 0.4) (layers F.Cu B.Cu) (net 16))
+  (via (at 48.9674 14.7254) (size 0.8) (drill 0.4) (layers F.Cu B.Cu) (net 16))
+  (via (at 47.9674 14.7254) (size 0.8) (drill 0.4) (layers F.Cu B.Cu) (net 16))
+  (via (at 46.9674 14.7254) (size 0.8) (drill 0.4) (layers F.Cu B.Cu) (net 16))
+  (via (at 45.9674 14.7254) (size 0.8) (drill 0.4) (layers F.Cu B.Cu) (net 16))
+  (via (at 44.9674 14.7254) (size 0.8) (drill 0.4) (layers F.Cu B.Cu) (net 16))
+  (via (at 43.9674 14.7254) (size 0.8) (drill 0.4) (layers F.Cu B.Cu) (net 16))
+  (via (at 57.9674 13.7254) (size 0.8) (drill 0.4) (layers F.Cu B.Cu) (net 16))
+  (via (at 56.9674 13.7254) (size 0.8) (drill 0.4) (layers F.Cu B.Cu) (net 16))
+  (via (at 55.9674 13.7254) (size 0.8) (drill 0.4) (layers F.Cu B.Cu) (net 16))
+  (via (at 54.9674 13.7254) (size 0.8) (drill 0.4) (layers F.Cu B.Cu) (net 16))
+  (via (at 53.9674 13.7254) (size 0.8) (drill 0.4) (layers F.Cu B.Cu) (net 16))
+  (via (at 52.9674 13.7254) (size 0.8) (drill 0.4) (layers F.Cu B.Cu) (net 16))
+  (via (at 51.9674 13.7254) (size 0.8) (drill 0.4) (layers F.Cu B.Cu) (net 16))
+  (via (at 50.9674 13.7254) (size 0.8) (drill 0.4) (layers F.Cu B.Cu) (net 16))
+  (via (at 49.9674 13.7254) (size 0.8) (drill 0.4) (layers F.Cu B.Cu) (net 16))
+  (via (at 48.9674 13.7254) (size 0.8) (drill 0.4) (layers F.Cu B.Cu) (net 16))
+  (via (at 47.9674 13.7254) (size 0.8) (drill 0.4) (layers F.Cu B.Cu) (net 16))
+  (via (at 46.9674 13.7254) (size 0.8) (drill 0.4) (layers F.Cu B.Cu) (net 16))
+  (via (at 45.9674 13.7254) (size 0.8) (drill 0.4) (layers F.Cu B.Cu) (net 16))
+  (via (at 44.9674 13.7254) (size 0.8) (drill 0.4) (layers F.Cu B.Cu) (net 16))
+  (via (at 43.9674 13.7254) (size 0.8) (drill 0.4) (layers F.Cu B.Cu) (net 16))
+  (via (at 57.9674 12.7254) (size 0.8) (drill 0.4) (layers F.Cu B.Cu) (net 16))
+  (via (at 56.9674 12.7254) (size 0.8) (drill 0.4) (layers F.Cu B.Cu) (net 16))
+  (via (at 55.9674 12.7254) (size 0.8) (drill 0.4) (layers F.Cu B.Cu) (net 16))
+  (via (at 54.9674 12.7254) (size 0.8) (drill 0.4) (layers F.Cu B.Cu) (net 16))
+  (via (at 53.9674 12.7254) (size 0.8) (drill 0.4) (layers F.Cu B.Cu) (net 16))
+  (via (at 52.9674 12.7254) (size 0.8) (drill 0.4) (layers F.Cu B.Cu) (net 16))
+  (via (at 51.9674 12.7254) (size 0.8) (drill 0.4) (layers F.Cu B.Cu) (net 16))
+  (via (at 50.9674 12.7254) (size 0.8) (drill 0.4) (layers F.Cu B.Cu) (net 16))
+  (via (at 49.9674 12.7254) (size 0.8) (drill 0.4) (layers F.Cu B.Cu) (net 16))
+  (via (at 48.9674 12.7254) (size 0.8) (drill 0.4) (layers F.Cu B.Cu) (net 16))
+  (via (at 47.9674 12.7254) (size 0.8) (drill 0.4) (layers F.Cu B.Cu) (net 16))
+  (via (at 46.9674 12.7254) (size 0.8) (drill 0.4) (layers F.Cu B.Cu) (net 16))
+  (via (at 45.9674 12.7254) (size 0.8) (drill 0.4) (layers F.Cu B.Cu) (net 16))
+  (via (at 44.9674 12.7254) (size 0.8) (drill 0.4) (layers F.Cu B.Cu) (net 16))
+  (via (at 43.9674 12.7254) (size 0.8) (drill 0.4) (layers F.Cu B.Cu) (net 16))
   (segment (start 32.9692 44.466) (end 32.9692 45.7454) (width 0.25) (layer B.Cu) (net 17))
   (segment (start 32.7754 44.2722) (end 32.9692 44.466) (width 0.25) (layer B.Cu) (net 17))
@@
     (polygon
       (pts
-        (xy 44.958 50.7238) (xy 28.2956 50.7238) (xy 28.3464 35.56) (xy 34.798 35.56) (xy 34.798 0)
-        (xy 40.386 0.0508) (xy 40.4114 37.465) (xy 53.2892 37.4396) (xy 53.2892 39.5224) (xy 44.9326 39.497)
+        (xy 44.958 50.7238) (xy 28.2956 50.7238) (xy 28.3464 35.56) (xy 34.798 35.56) (xy 34.8488 -0.0254)
+        (xy 40.4368 0.0254) (xy 40.4114 37.465) (xy 53.2892 37.4396) (xy 53.2892 39.5224) (xy 44.9326 39.497)
       )
     )
@@
     (polygon
       (pts
-        (xy 40.9956 15.9258) (xy 40.9956 0.1524) (xy 60.0456 0) (xy 59.9948 15.9258)
+        (xy 40.9956 15.9258) (xy 40.9956 0.0762) (xy 60.0456 -0.0762) (xy 59.9948 15.9258)
       )
     )
@@
     (polygon
       (pts
-        (xy 40.9956 15.9258) (xy 40.9956 0.1016) (xy 60.0456 -0.0508) (xy 59.9694 15.9258)
+        (xy 40.9956 15.9258) (xy 40.9956 0.0254) (xy 60.0456 -0.127) (xy 59.9694 15.9258)
       )
     )
@@
     (polygon
       (pts
-        (xy 7.2644 13.2334) (xy 7.239 8.89) (xy 11.1252 8.8138) (xy 11.1252 0.4826) (xy 19.558 0.4826)
-        (xy 19.558 13.1826)
+        (xy 7.2136 15.9512) (xy 7.1628 8.8138) (xy 11.1252 8.8138) (xy 11.1506 0) (xy 19.5834 0)
+        (xy 19.5834 15.9004)
       )
     )
@@
     (polygon
       (pts
-        (xy 7.2644 16.383) (xy 7.2644 8.8646) (xy 11.1252 8.8138) (xy 11.1252 0.4826) (xy 19.558 0.4826)
-        (xy 19.5834 16.383)
+        (xy 7.2898 15.9004) (xy 7.2644 8.8138) (xy 11.1252 8.8138) (xy 11.1506 -0.0254) (xy 19.5834 -0.0254)
+        (xy 19.6088 15.9004)
       )
     )
@@
     (polygon
       (pts
-        (xy 20.32 0) (xy 25.4 0.0254) (xy 25.3746 16.4084) (xy 20.2946 16.4084)
+        (xy 20.32 0) (xy 25.4 0.0254) (xy 25.3746 15.9004) (xy 20.2946 15.9004)
       )
     )
