File: V0.2-IGBT/PCB/ENNOID Dual Gate Driver.kicad_pcb (KiCad board)
At the start: 2 copper layers, 60 x 98 mm, 134 parts, among them J1 Conn_02x08_Odd_Even, J2 Current, J3 TEMP, J4 PHASE, J5 Collector, J6 Gate_H, J7 G_L, J8 E, Q3 MJD44H11RLG, Q4 MJD45H11RLG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

Commit message: PCB V0.2
Routing:
- net /GD_HIGH/-VEE: track 47.1 -> 57.6 mm, vias 6 -> 12
- net /GD_LOW/-VEE: track 34.6 -> 43.6 mm, vias 6 -> 12
Changed lines of the file:
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@@
     (thickness 1.6)
     (drawings 15)
-    (tracks 891)
+    (tracks 923)
     (zones 0)
     (modules 134)
@@
   )
   (setup
-    (last_trace_width 0.25)
+    (last_trace_width 1)
     (user_trace_width 0.5)
     (user_trace_width 1)
@@
   (segment (start 16.5682 46.3678) (end 15.26 45.0596) (width 1) (layer F.Cu) (net 6))
   (segment (start 15.26 43.2308) (end 15.26 45.0596) (width 1) (layer F.Cu) (net 6))
+  (segment (start 22.8346 47.3108) (end 22.615 47.3108) (width 1) (layer F.Cu) (net 7))
+  (segment (start 22.615 47.3108) (end 21.6482 48.2776) (width 1) (layer F.Cu) (net 7))
+  (segment (start 23.8346 47.3108) (end 22.8346 47.3108) (width 1) (layer F.Cu) (net 7))
+  (segment (start 23.8346 48.3108) (end 23.8346 47.3108) (width 1) (layer F.Cu) (net 7))
+  (segment (start 22.8346 48.3108) (end 23.8346 48.3108) (width 1) (layer F.Cu) (net 7))
+  (via (at 23.8346 47.3108) (size 0.8) (drill 0.4) (layers F.Cu B.Cu) (net 7))
+  (via (at 22.8346 47.3108) (size 0.8) (drill 0.4) (layers F.Cu B.Cu) (net 7))
+  (via (at 23.8346 48.3108) (size 0.8) (drill 0.4) (layers F.Cu B.Cu) (net 7))
+  (segment (start 11.2268 48.26) (end 11.2268 47.26) (width 1) (layer F.Cu) (net 7))
+  (segment (start 11.2268 47.26) (end 11.7406 47.26) (width 1) (layer F.Cu) (net 7))
+  (segment (start 11.7406 47.26) (end 12.7582 48.2776) (width 1) (layer F.Cu) (net 7))
+  (segment (start 10.2268 47.26) (end 11.2268 47.26) (width 1) (layer F.Cu) (net 7))
+  (segment (start 10.2268 48.26) (end 10.2268 47.26) (width 1) (layer F.Cu) (net 7))
+  (segment (start 11.2268 48.26) (end 10.2268 48.26) (width 1) (layer F.Cu) (net 7))
+  (via (at 10.2268 47.26) (size 0.8) (drill 0.4) (layers F.Cu B.Cu) (net 7))
+  (via (at 11.2268 47.26) (size 0.8) (drill 0.4) (layers F.Cu B.Cu) (net 7))
+  (via (at 10.2268 48.26) (size 0.8) (drill 0.4) (layers F.Cu B.Cu) (net 7))
   (segment (start 18.8214 29.6418) (end 17.4178 31.0454) (width 2) (layer F.Cu) (net 7))
   (segment (start 17.4178 31.0454) (end 17.4178 31.75) (width 2) (layer F.Cu) (net 7))
@@
   (segment (start 36.4706 41.5506) (end 34.7472 41.5506) (width 0.25) (layer B.Cu) (net 11))
   (segment (start 37.2032 44.6876) (end 37.2032 42.2832) (width 0.25) (layer B.Cu) (net 11))
+  (via (at 44.7708 47.2854) (size 0.8) (drill 0.4) (layers F.Cu B.Cu) (net 12))
+  (via (at 44.7708 48.2854) (size 0.8) (drill 0.4) (layers F.Cu B.Cu) (net 12))
+  (segment (start 44.7708 47.2854) (end 45.7708 47.2854) (width 1) (layer F.Cu) (net 12))
+  (segment (start 44.7708 48.2854) (end 44.7708 47.2854) (width 1) (layer F.Cu) (net 12))
+  (segment (start 45.7708 48.2854) (end 44.7708 48.2854) (width 1) (layer F.Cu) (net 12))
+  (segment (start 56.7944 47.2854) (end 56.6404 47.2854) (width 1) (layer F.Cu) (net 12))
+  (segment (start 56.6404 47.2854) (end 55.6482 48.2776) (width 1) (layer F.Cu) (net 12))
+  (segment (start 57.7944 47.2854) (end 56.7944 47.2854) (width 1) (layer F.Cu) (net 12))
+  (segment (start 57.7944 48.2854) (end 57.7944 47.2854) (width 1) (layer F.Cu) (net 12))
+  (segment (start 56.7944 48.2854) (end 57.7944 48.2854) (width 1) (layer F.Cu) (net 12))
+  (segment (start 45.7708 47.2854) (end 45.7708 47.2902) (width 1) (layer F.Cu) (net 12))
+  (segment (start 45.7708 47.2902) (end 46.7582 48.2776) (width 1) (layer F.Cu) (net 12))
+  (via (at 57.7944 47.2854) (size 0.8) (drill 0.4) (layers F.Cu B.Cu) (net 12))
+  (via (at 56.7944 47.2854) (size 0.8) (drill 0.4) (layers F.Cu B.Cu) (net 12))
+  (via (at 57.7944 48.2854) (size 0.8) (drill 0.4) (layers F.Cu B.Cu) (net 12))
+  (via (at 45.7708 47.2854) (size 0.8) (drill 0.4) (layers F.Cu B.Cu) (net 12))
   (segment (start 52.7492 31.2674) (end 52.7492 29.8688) (width 1) (layer F.Cu) (net 12))
   (segment (start 52.831801 31.350001) (end 52.7492 31.2674) (width 1) (layer F.Cu) (net 12))
@@
   (via (at 53.3146 45.2628) (size 0.8) (drill 0.4) (layers F.Cu B.Cu) (net 44))
   (segment (start 54.9856 43.434) (end 54.9856 45.2374) (width 1) (layer B.Cu) (net 44))
+  (segment (start 33.4772 34.4116) (end 34.7418 34.4116) (width 0.25) (layer F.Cu) (net 45))
+  (segment (start 40.392401 40.062201) (end 40.7924 40.4622) (width 0.25) (layer F.Cu) (net 45))
+  (segment (start 40.894 40.5638) (end 40.7924 40.4622) (width 0.25) (layer B.Cu) (net 45))
+  (segment (start 46.6344 40.5638) (end 40.894 40.5638) (width 0.25) (layer B.Cu) (net 45))
+  (segment (start 34.7418 34.4116) (end 40.392401 40.062201) (width 0.25) (layer F.Cu) (net 45))
+  (via (at 40.7924 40.4622) (size 0.8) (drill 0.4) (layers F.Cu B.Cu) (net 45))
   (segment (start 54.3782 41.4877) (end 53.2765 40.386) (width 0.25) (layer F.Cu) (net 45))
   (segment (start 46.8122 40.386) (end 46.736 40.4622) (width 0.25) (layer F.Cu) (net 45))
@@
   (segment (start 53.2765 40.386) (end 46.8122 40.386) (width 0.25) (layer F.Cu) (net 45))
   (segment (start 46.736 40.4622) (end 46.6344 40.5638) (width 0.25) (layer F.Cu) (net 45))
-  (segment (start 40.5638 41.0464) (end 33.929 34.4116) (width 0.25) (layer F.Cu) (net 45))
-  (segment (start 41.1226 41.0464) (end 40.5638 41.0464) (width 0.25) (layer F.Cu) (net 45))
-  (segment (start 33.929 34.4116) (end 33.4772 34.4116) (width 0.25) (layer F.Cu) (net 45))
   (segment (start 32.719 30.8356) (end 32.719 33.6534) (width 0.25) (layer F.Cu) (net 45))
   (segment (start 32.719 33.6534) (end 33.4772 34.4116) (width 0.25) (layer F.Cu) (net 45))
@@
   (segment (start 29.5148 34.3322) (end 31.3722 34.3322) (width 0.25) (layer F.Cu) (net 45))
   (segment (start 31.3722 34.3322) (end 31.496 34.2084) (width 0.25) (layer F.Cu) (net 45))
-  (segment (start 46.6344 40.5638) (end 46.1518 41.0464) (width 0.25) (layer B.Cu) (net 45))
-  (segment (start 46.1518 41.0464) (end 41.688285 41.0464) (width 0.25) (layer B.Cu) (net 45))
-  (segment (start 41.688285 41.0464) (end 41.1226 41.0464) (width 0.25) (layer B.Cu) (net 45))
-  (via (at 41.1226 41.0464) (size 0.8) (drill 0.4) (layers F.Cu B.Cu) (net 45))
   (via (at 46.6344 40.5638) (size 0.8) (drill 0.4) (layers F.Cu B.Cu) (net 45))
   (segment (start 54.3782 48.2776) (end 54.3782 42.254798) (width 0.25) (layer F.Cu) (net 45))
@@
     (polygon
       (pts
-        (xy 44.958 50.7238) (xy 28.2956 50.7238) (xy 28.3464 35.56) (xy 34.798 35.56) (xy 34.8488 -0.0254)
-        (xy 40.4368 0.0254) (xy 40.4114 37.465) (xy 53.2892 37.4396) (xy 53.2892 39.5224) (xy 44.9326 39.497)
+        (xy 43.6626 50.7238) (xy 28.2956 50.7238) (xy 28.3464 35.56) (xy 34.798 35.56) (xy 34.8488 -0.0254)
+        (xy 40.4368 0.0254) (xy 40.4114 37.465) (xy 53.2892 37.4396) (xy 53.2892 39.5224) (xy 43.6626 39.497)
       )
     )
@@
     (polygon
       (pts
-        (xy 34.013577 50.714837) (xy 33.962777 46.142837) (xy 54.515794 46.266385) (xy 54.490394 21.704585) (xy 60.002194 21.729985)
+        (xy 34.013577 50.714837) (xy 34.0106 46.2788) (xy 54.515794 46.266385) (xy 54.490394 21.704585) (xy 60.002194 21.729985)
         (xy 60.027594 50.736785)
       )
@@
     (polygon
       (pts
-        (xy 9.8806 50.7238) (xy 0 50.7238) (xy 0 46.1772) (xy 0.0254 37.465) (xy 20.2184 37.465)
-        (xy 20.32 6.4516) (xy 20.32 0) (xy 25.4 0) (xy 25.4 39.497) (xy 9.8552 39.497)
+        (xy 9.2202 50.7238) (xy 0 50.7238) (xy 0 46.1772) (xy 0.0254 37.465) (xy 20.2184 37.465)
+        (xy 20.32 6.4516) (xy 20.32 0) (xy 25.4 0) (xy 25.4 39.497) (xy 9.1948 39.497)
       )
     )

Commit message: V0.2 PCB
Parts:
- moved C36 0.28 mm to (50.6, 45.2)
- moved C46 0.28 mm to (50.6, 43.4)
- moved R25 0.28 mm to (50.6, 41.5)
Routing:
- net /GD_LOW/+VCC: track 56.3 -> 57.3 mm, vias 5 -> 6
- net /GD_HIGH/+VCC: track 57.5 -> 58.5 mm, vias 5 -> 6
Changed lines of the file:
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@@
     (thickness 1.6)
     (drawings 15)
-    (tracks 923)
+    (tracks 930)
     (zones 0)
     (modules 134)
@@
   )
   (module Capacitors_SMD:C_0805_HandSoldering (layer F.Cu)
-    (at 50.3174 45.212)
+    (at 50.5968 45.1866)
     (descr "Capacitor SMD 0805, hand soldering")
     (tags "capacitor 0805")
@@
   )
   (module Capacitors_SMD:C_0805_HandSoldering (layer F.Cu)
-    (at 50.3174 43.3832)
+    (at 50.5968 43.3578)
     (descr "Capacitor SMD 0805, hand soldering")
     (tags "capacitor 0805")
@@
   )
   (module Resistors_SMD:R_0805_HandSoldering (layer F.Cu)
-    (at 50.3428 41.5544 180)
+    (at 50.6222 41.529 180)
     (descr "Resistor SMD 0805, hand soldering")
     (tags "resistor 0805")
@@
   (segment (start 3.2032 47.2276) (end 5.323 47.2276) (width 1) (layer B.Cu) (net 5))
   (segment (start 5.323 47.2276) (end 5.3594 47.264) (width 1) (layer B.Cu) (net 5))
+  (segment (start 11.5222 43.2054) (end 12.5222 43.2054) (width 1) (layer F.Cu) (net 6))
+  (via (at 11.5222 43.2054) (size 0.8) (drill 0.4) (layers F.Cu B.Cu) (net 6))
+  (segment (start 16.5682 46.5656) (end 15.26 45.2574) (width 1) (layer F.Cu) (net 6))
+  (segment (start 16.5682 48.2776) (end 16.5682 46.5656) (width 1) (layer F.Cu) (net 6))
+  (segment (start 15.26 45.2574) (end 15.26 45.0596) (width 1) (layer F.Cu) (net 6))
   (segment (start 10.6934 27.8048) (end 10.6934 30.3972) (width 1) (layer F.Cu) (net 6))
   (segment (start 10.6934 30.3972) (end 12.732 32.4358) (width 1) (layer F.Cu) (net 6))
@@
   (segment (start 12.5476 43.2308) (end 12.5222 43.2054) (width 1) (layer F.Cu) (net 6))
   (via (at 12.5222 43.2054) (size 0.8) (drill 0.4) (layers F.Cu B.Cu) (net 6))
-  (segment (start 16.5682 48.2776) (end 16.5682 46.3678) (width 1) (layer F.Cu) (net 6))
-  (segment (start 16.5682 46.3678) (end 15.26 45.0596) (width 1) (layer F.Cu) (net 6))
   (segment (start 15.26 43.2308) (end 15.26 45.0596) (width 1) (layer F.Cu) (net 6))
   (segment (start 22.8346 47.3108) (end 22.615 47.3108) (width 1) (layer F.Cu) (net 7))
@@
   (segment (start 52.8 38.3606) (end 50.7238 38.3606) (width 1) (layer F.Cu) (net 10))
   (segment (start 50.7238 38.3606) (end 49.8 37.4368) (width 1) (layer F.Cu) (net 10))
-  (segment (start 50.5682 46.809) (end 49.0674 45.3082) (width 1) (layer F.Cu) (net 11))
-  (segment (start 50.5682 48.2776) (end 50.5682 46.809) (width 1) (layer F.Cu) (net 11))
-  (segment (start 49.0674 45.3082) (end 49.0674 45.212) (width 1) (layer F.Cu) (net 11))
+  (segment (start 46.4472 43.4086) (end 47.4472 43.4086) (width 1) (layer F.Cu) (net 11))
+  (via (at 46.4472 43.4086) (size 0.8) (drill 0.4) (layers F.Cu B.Cu) (net 11))
+  (segment (start 50.5682 46.7328) (end 49.0674 45.232) (width 1) (layer F.Cu) (net 11))
+  (segment (start 50.5682 48.2776) (end 50.5682 46.7328) (width 1) (layer F.Cu) (net 11))
+  (segment (start 49.0674 45.232) (end 49.0674 45.212) (width 1) (layer F.Cu) (net 11))
   (segment (start 46.9674 31.75) (end 48.165 31.75) (width 1) (layer F.Cu) (net 11))
   (segment (start 48.165 31.75) (end 48.7492 32.3342) (width 1) (layer F.Cu) (net 11))
@@
   (segment (start 0.6858 30.0802) (end 0.6858 23.8506) (width 0.25) (layer F.Cu) (net 42))
   (via (at 0.762 23.7744) (size 0.8) (drill 0.4) (layers F.Cu B.Cu) (net 42))
-  (segment (start 53.2384 41.529) (end 54.9094 41.529) (width 1) (layer B.Cu) (net 43))
+  (segment (start 54.9094 41.529) (end 54.884 41.5036) (width 1) (layer B.Cu) (net 43))
+  (segment (start 54.884 41.5036) (end 54.058085 41.5036) (width 1) (layer B.Cu) (net 43))
+  (segment (start 53.2638 41.5036) (end 53.4924 41.5036) (width 0.25) (layer F.Cu) (net 43))
+  (segment (start 53.213 41.5544) (end 53.2638 41.5036) (width 0.25) (layer F.Cu) (net 43))
+  (segment (start 54.058085 41.5036) (end 53.4924 41.5036) (width 1) (layer B.Cu) (net 43))
+  (via (at 53.4924 41.5036) (size 0.8) (drill 0.4) (layers F.Cu B.Cu) (net 43))
   (segment (start 54.9094 41.529) (end 54.9856 41.6052) (width 0.25) (layer B.Cu) (net 43))
-  (segment (start 53.213 41.5544) (end 53.2384 41.529) (width 0.25) (layer F.Cu) (net 43))
   (segment (start 51.6928 41.5544) (end 53.213 41.5544) (width 1) (layer F.Cu) (net 43))
-  (via (at 53.2384 41.529) (size 0.8) (drill 0.4) (layers F.Cu B.Cu) (net 43))
   (segment (start 53.1082 48.2776) (end 53.1082 45.4692) (width 1) (layer F.Cu) (net 44))
   (segment (start 53.1082 45.4692) (end 53.3146 45.2628) (width 1) (layer F.Cu) (net 44))
@@
   (via (at 53.3146 45.2628) (size 0.8) (drill 0.4) (layers F.Cu B.Cu) (net 44))
   (segment (start 54.9856 43.434) (end 54.9856 45.2374) (width 1) (layer B.Cu) (net 44))
+  (segment (start 54.3782 42.254798) (end 54.3782 41.316396) (width 0.25) (layer F.Cu) (net 45))
+  (segment (start 54.3782 41.316396) (end 53.225605 40.163801) (width 0.25) (layer F.Cu) (net 45))
+  (segment (start 47.034399 40.163801) (end 46.6344 40.5638) (width 0.25) (layer F.Cu) (net 45))
+  (segment (start 53.225605 40.163801) (end 47.034399 40.163801) (width 0.25) (layer F.Cu) (net 45))
   (segment (start 33.4772 34.4116) (end 34.7418 34.4116) (width 0.25) (layer F.Cu) (net 45))
   (segment (start 40.392401 40.062201) (end 40.7924 40.4622) (width 0.25) (layer F.Cu) (net 45))
@@
   (segment (start 34.7418 34.4116) (end 40.392401 40.062201) (width 0.25) (layer F.Cu) (net 45))
   (via (at 40.7924 40.4622) (size 0.8) (drill 0.4) (layers F.Cu B.Cu) (net 45))
-  (segment (start 54.3782 41.4877) (end 53.2765 40.386) (width 0.25) (layer F.Cu) (net 45))
-  (segment (start 46.8122 40.386) (end 46.736 40.4622) (width 0.25) (layer F.Cu) (net 45))
-  (segment (start 54.3782 42.254798) (end 54.3782 41.4877) (width 0.25) (layer F.Cu) (net 45))
-  (segment (start 53.2765 40.386) (end 46.8122 40.386) (width 0.25) (layer F.Cu) (net 45))
-  (segment (start 46.736 40.4622) (end 46.6344 40.5638) (width 0.25) (layer F.Cu) (net 45))
   (segment (start 32.719 30.8356) (end 32.719 33.6534) (width 0.25) (layer F.Cu) (net 45))
   (segment (start 32.719 33.6534) (end 33.4772 34.4116) (width 0.25) (layer F.Cu) (net 45))
@@
   (via (at 17.8308 46.7106) (size 0.8) (drill 0.4) (layers F.Cu B.Cu) (net 53))
   (segment (start 17.8382 48.2776) (end 17.8382 46.718) (width 1) (layer F.Cu) (net 53))
-  (segment (start 49.2982 47.2662) (end 48.7426 46.7106) (width 1) (layer F.Cu) (net 54))
-  (segment (start 48.7426 46.7106) (end 48.133 46.7106) (width 1) (layer F.Cu) (net 54))
-  (segment (start 49.2982 48.2776) (end 49.2982 47.2662) (width 1) (layer F.Cu) (net 54))
+  (segment (start 49.2982 48.2776) (end 49.2982 47.183117) (width 1) (layer F.Cu) (net 54))
+  (segment (start 49.2982 47.183117) (end 48.724083 46.609) (width 1) (layer F.Cu) (net 54))
+  (segment (start 48.724083 46.609) (end 48.158398 46.609) (width 1) (layer F.Cu) (net 54))
+  (segment (start 49.8348 39.3484) (end 49.8348 44.932598) (width 1) (layer B.Cu) (net 54))
+  (segment (start 48.558397 46.209001) (end 48.158398 46.609) (width 1) (layer B.Cu) (net 54))
+  (segment (start 49.8348 44.932598) (end 48.558397 46.209001) (width 1) (layer B.Cu) (net 54))
+  (via (at 48.158398 46.609) (size 0.8) (drill 0.4) (layers F.Cu B.Cu) (net 54))
   (segment (start 47.4218 41.5544) (end 48.9928 41.5544) (width 1) (layer F.Cu) (net 54))
   (segment (start 49.8094 41.5544) (end 47.987485 41.5544) (width 1) (layer B.Cu) (net 54))
@@
   (segment (start 49.8348 41.5798) (end 49.8094 41.5544) (width 1) (layer B.Cu) (net 54))
   (via (at 47.4218 41.5544) (size 0.8) (drill 0.4) (layers F.Cu B.Cu) (net 54))
-  (via (at 48.133 46.7106) (size 0.8) (drill 0.4) (layers F.Cu B.Cu) (net 54))
-  (segment (start 49.8348 39.3484) (end 49.8348 45.0088) (width 1) (layer B.Cu) (net 54))
-  (segment (start 48.532999 46.310601) (end 48.133 46.7106) (width 1) (layer B.Cu) (net 54))
-  (segment (start 49.8348 45.0088) (end 48.532999 46.310601) (width 1) (layer B.Cu) (net 54))
   (segment (start 49.8348 39.3484) (end 49.8348 41.5798) (width 0.25) (layer B.Cu) (net 54))
   (segment (start 51.8414 46.6852) (end 51.8414 48.2744) (width 1) (layer F.Cu) (net 55))

Commit message: ENNOID LOGO on V0.2
Parts:
- added G***: LOGO, ENNOID:ENNOID-LOGO, B.Cu at (30.0, 72.5)

Commit message: logo
Parts:
- turned G*** to 180 degrees
Changed lines of the file:
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@@
   )
   (module ENNOID:ENNOID-LOGO (layer B.Cu)
-    (at 30 72.5)
-    (fp_text reference G*** (at 0 0) (layer B.SilkS) hide
+    (at 30 72.5 180)
+    (fp_text reference G*** (at 0 0 180) (layer B.SilkS) hide
       (effects (font (size 1.524 1.524) (thickness 0.3)) (justify mirror))
     )
-    (fp_text value LOGO (at 0.75 0) (layer B.SilkS) hide
+    (fp_text value LOGO (at 0.75 0 180) (layer B.SilkS) hide
       (effects (font (size 1.524 1.524) (thickness 0.3)) (justify mirror))
     )
