File: V0.2-IGBT/PCB/ENNOID Dual Gate Driver.kicad_pcb (KiCad board)
At the start: 2 copper layers, 60 x 98 mm, 142 parts, among them J1 Conn_02x08_Odd_Even, J2 Current, J3 TEMP, J4 PHASE, J5 Collector, J6 Gate_H, J7 G_L, J8 E, Q3 MJD3055T4G, Q4 MJD2955T4G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

Commit message: V0.2
Parts:
- R10: moved to F.Cu
- moved R10 6.55 mm to (3.25, 31.3), turned to 0 degrees
- moved D16 3.81 mm to (9.40, 21.0)
- moved D22 3.58 mm to (45.5, 20.8)
- moved C22 3.56 mm to (3.45, 37.1)
- moved D10 3.56 mm to (1.52, 37.1)
- moved D6 3.56 mm to (5.36, 37.1)
- moved D15 1.01 mm to (9.37, 4.50)
- moved D21 1.00 mm to (29.3, 4.50)
Routing:
- net PHASE: track 134.1 -> 117.1 mm
- net Net-(D21-Pad2): track 10.5 -> 18.2 mm, vias 1 -> 2
- net Net-(C22-Pad1): track 42.2 -> 35.3 mm, vias 3 -> 2
- net Net-(D15-Pad2): track 8.21 -> 13.1 mm, vias 1 -> 2
- net /GD_HIGH/G: track 5.27 -> 9.17 mm, vias 30 -> 29
- net /GD_HIGH/+VCC: track 64.3 -> 60.5 mm
- net /GD_LOW/G: track 14.9 -> 18.5 mm
- net /GD_LOW/+VCC: track 62.8 -> 59.2 mm
Other:
- outline, holes or cut-outs redrawn

Commit message: V0.2 completed
Parts:
- R10, R21: value 10k -> 1k
- R14, R15, R22, R23, R36, R37, R38, R39: footprint Resistors_SMD:R_2512_HandSoldering -> Resistors_SMD:R_2512
- moved D21 0.42 mm to (29.2, 4.09)
- moved D15 0.42 mm to (9.27, 4.09)
Routing:
- net /GD_HIGH/G: track 9.17 -> 15.5 mm, vias 29 -> 33
- net /GD_LOW/G: track 18.5 -> 22.5 mm
- net Net-(Q6-Pad3): track 12.2 -> 13.4 mm
- net Net-(Q3-Pad3): track 12.8 -> 14.0 mm
- net Net-(Q4-Pad3): track 12.1 -> 13.3 mm
- net Net-(Q5-Pad3): track 12.9 -> 14.1 mm

Commit message: Maintenance update
Parts:
- removed R31: 1k, Resistors_SMD:R_0805_HandSoldering
- moved D6 0.36 mm to (5.72, 37.1)
- moved D18 0.28 mm to (29.2, 35.4)
- moved R32 0.28 mm to (47.5, 90.4)
- moved C42 0.28 mm to (31.2, 89.1)
- moved C44 0.28 mm to (47.5, 86.1)
- moved C41 0.25 mm to (36.3, 89.1)
- moved C35 0.20 mm to (56.2, 41.4)
- moved R25 0.18 mm to (50.6, 41.4)
- moved C17 0.18 mm to (22.6, 41.2)
- moved R20 0.16 mm to (49.6, 63.2)
- moved R8 0.15 mm to (53.7, 63.2)
- moved R9 0.15 mm to (16.4, 63.4)
- moved D2 0.15 mm to (15.4, 66.6)
- moved C22 0.15 mm to (3.61, 37.1)
- moved R6 0.13 mm to (20.5, 63.4)
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Connections:
- C38 pad 2: Net-(C38-Pad2) -> /ISO_PSU_LOW/COM
- U8 pad 3: Net-(C38-Pad2) -> /ISO_PSU_LOW/COM
Routing:
- net /ISO_PSU_LOW/COM: track 128.5 -> 134.6 mm, vias 6 -> 7
- net Net-(C38-Pad2): track 5.60 -> 0.00 mm, vias 1 -> 0
- net /GD_LOW/G: track 22.5 -> 25.9 mm
- net /GD_HIGH/G: track 15.5 -> 18.9 mm
- net /GD_LOW/-VEE: vias 12 -> 40
- net /GD_LOW/+VCC: vias 6 -> 34
- net /GD_HIGH/-VEE: vias 12 -> 40
- net /GD_HIGH/+VCC: vias 6 -> 34
Other:
- outline, holes or cut-outs redrawn
- board text added: "Dual Gate Driver - V0.2 01/2018 https://github.com/EnnoidMe"

Commit message: Maintenance update
Parts:
- added REF**: MountingHole_3.2mm_M3_ISO14580_Pad, Mounting_Holes:MountingHole_3.2mm_M3_ISO14580_Pad, F.Cu at (55.0, 5.00)
- D18, D6: footprint Diodes_SMD:D_SOD-323 -> Diodes_SMD:D_SOD-323_HandSoldering
- moved D15 2.41 mm to (9.25, 6.50)
- moved D21 2.41 mm to (29.2, 6.50)
- moved D5 2.39 mm to (12.8, 9.70)
- moved R14 1.02 mm to (9.02, 15.5)
- moved R22 1.02 mm to (20.4, 15.5)
- moved R15 1.02 mm to (12.8, 15.5)
- moved R23 1.02 mm to (16.7, 15.5)
- moved R36 0.91 mm to (48.9, 15.2)
- moved R37 0.91 mm to (45.1, 15.2)
- moved R38 0.91 mm to (52.8, 15.2)
- moved R39 0.91 mm to (56.6, 15.2)
Connections:
- J1 pad 7: Net-(J1-Pad7) -> (no net)
- J1 pad 8: Net-(J1-Pad8) -> (no net)
- U4 pad 7: Net-(U4-Pad7) -> (no net)
- U5 pad 7: Net-(U5-Pad7) -> (no net)
Routing:
- net /GD_HIGH/C: track 14.9 -> 19.9 mm
- net /GD_HIGH/G: track 18.9 -> 14.9 mm
- net Net-(D15-Pad2): track 13.1 -> 16.8 mm
- net PHASE: track 117.1 -> 114.7 mm
- net /GD_LOW/G: track 25.9 -> 24.3 mm
- net Net-(Q4-Pad3): track 13.3 -> 11.9 mm
- net Net-(Q3-Pad3): track 14.0 -> 12.5 mm
- net Net-(Q6-Pad3): track 13.4 -> 12.1 mm
- net Net-(Q5-Pad3): track 14.1 -> 12.9 mm
- net Net-(D21-Pad2): track 18.2 -> 17.4 mm
Other:
- outline, holes or cut-outs redrawn

Commit message: PIC update
Parts:
- moved R27 3.55 mm to (27.6, 22.4), turned to 180 degrees
- moved R29 3.21 mm to (32.4, 22.4), turned to 180 degrees
Routing:
- net PHASE: track 114.7 -> 123.4 mm
- net Net-(R17-Pad1): track 23.4 -> 28.8 mm
Other:
- outline, holes or cut-outs redrawn

Commit message: Maintenance update
Parts:
- G1: renamed from G***; value LOGO -> Logo_ENNOID
- J10: renamed from REF**; value MountingHole_3.2mm_M3_ISO14580_Pad -> Mounting Hole 2
- J11: renamed from REF**; value MountingHole_3.2mm_M3_ISO14580_Pad -> Mounting Hole 3
- J9: renamed from REF**; value MountingHole_3.2mm_M3_ISO14580_Pad -> Mounting hole 1
Changed lines of the file:
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@@
     (tags "mounting hole 3.2mm m3 iso14580")
     (attr virtual)
-    (fp_text reference REF** (at 0 -3.75) (layer F.SilkS) hide
+    (fp_text reference J11 (at 0 -3.75) (layer F.SilkS) hide
       (effects (font (size 1 1) (thickness 0.15)))
     )
-    (fp_text value MountingHole_3.2mm_M3_ISO14580_Pad (at 0 3.75) (layer F.Fab)
+    (fp_text value "Mounting Hole 3" (at 0 3.75) (layer F.Fab)
       (effects (font (size 1 1) (thickness 0.15)))
     )
@@
     (tags "mounting hole 3.2mm m3 iso14580")
     (attr virtual)
-    (fp_text reference REF** (at 0 -3.75) (layer F.SilkS) hide
+    (fp_text reference J9 (at 0 -3.75) (layer F.SilkS) hide
       (effects (font (size 1 1) (thickness 0.15)))
     )
-    (fp_text value MountingHole_3.2mm_M3_ISO14580_Pad (at 0 3.75) (layer F.Fab)
+    (fp_text value "Mounting hole 1" (at 0 3.75) (layer F.Fab)
       (effects (font (size 1 1) (thickness 0.15)))
     )
@@
     (tags "mounting hole 3.2mm m3 iso14580")
     (attr virtual)
-    (fp_text reference REF** (at 0 -3.75) (layer F.SilkS) hide
+    (fp_text reference J10 (at 0 -3.75) (layer F.SilkS) hide
       (effects (font (size 1 1) (thickness 0.15)))
     )
-    (fp_text value MountingHole_3.2mm_M3_ISO14580_Pad (at 0 3.75) (layer F.Fab)
+    (fp_text value "Mounting Hole 2" (at 0 3.75) (layer F.Fab)
       (effects (font (size 1 1) (thickness 0.15)))
     )
@@
   (module ENNOID:ENNOID-LOGO (layer B.Cu)
     (at 30 74 180)
-    (fp_text reference G*** (at 0 0 180) (layer B.SilkS) hide
+    (fp_text reference G1 (at 0 0 180) (layer B.SilkS) hide
       (effects (font (size 1.524 1.524) (thickness 0.3)) (justify mirror))
     )
-    (fp_text value LOGO (at 0.75 0 180) (layer B.SilkS) hide
+    (fp_text value Logo_ENNOID (at 0.75 0 180) (layer B.SilkS) hide
       (effects (font (size 1.524 1.524) (thickness 0.3)) (justify mirror))
     )
