File: V0.2-IGBT/PCB/GD.sch (KiCad schematic (older format))
At the start: 28 parts, among them U4 1ED020I12-F2, U5 IXD-609

Commit message: v0.2 PCB
Parts:
- removed C35: 10u, Resistors_SMD:R_1210_HandSoldering, symbol device:C
- removed D10: D, Diodes_SMD:D_SMA_Handsoldering, symbol device:D
- removed D3, D5: D_Zener, Diodes_SMD:D_SOD-123, symbol device:D_Zener
- removed R45: DNP, Resistors_SMD:R_0805_HandSoldering, symbol device:R
- removed U4: 1ED020I12-F2, Housings_SOIC:SOIC-16W_7.5x10.3mm_Pitch1.27mm, symbol ENNOID:1ED020I12-F2
- removed U5: IXD-609, Housings_SOIC:SOIC-8-1EP_3.9x4.9mm_Pitch1.27mm, symbol ENNOID:IXD-609
- added C20, C28, C29: 1u, Capacitors_SMD:C_0805_HandSoldering, symbol device:C
- added C24: 100n, Capacitors_SMD:C_0805_HandSoldering, symbol device:C
- added C30, C32, C33: 10u, Capacitors_SMD:C_1206_HandSoldering, symbol device:C
- added C34: 0.22u, Capacitors_SMD:C_0805_HandSoldering, symbol device:C
- added D10: BAT54WS-7-F, Diodes_SMD:D_SOD-323_HandSoldering, symbol device:D_Schottky
- added D11: SMAJ18CA, Diodes_SMD:D_SMA_Handsoldering, symbol device:D_TVS
- added D15: smcj440ca, Diodes_SMD:D_SMC_Handsoldering, symbol device:D_TVS
- added D16: es2j-ltp, Diodes_SMD:D_SMA_Handsoldering, symbol device:D
- added D3: 1N4148W, Diodes_SMD:D_SOD-123, symbol device:D
- added D6: MMSZ5242BS, Diodes_SMD:D_SOD-323, symbol device:D_Zener
- added Q3: MJD44H11RLG, TO_SOT_Packages_SMD:TO-252-3_TabPin4, symbol device:Q_NPN_Darlington_BCEC
- added Q4: MJD45H11RLG, TO_SOT_Packages_SMD:TO-252-3_TabPin4, symbol device:Q_PNP_Darlington_BCEC
- added R22, R23: 3, Resistors_SMD:R_2512_HandSoldering, symbol device:R
- added R24: 10k, Resistors_SMD:R_0805_HandSoldering, symbol device:R
- added U4: ISO5852SDWR, Housings_SOIC:SOIC-16W_7.5x10.3mm_Pitch1.27mm, symbol ENNOID:ISO5852SDWR
- C17: value 100n -> 15n
- C19, C25: value DNP -> 100n
- C21: value 4.7u -> 1u; footprint Capacitors_SMD:C_1206_HandSoldering -> Capacitors_SMD:C_0805_HandSoldering
- C22: value 10n -> 220p
- C23, C31: value 100n -> 10u; footprint Capacitors_SMD:C_0805_HandSoldering -> Capacitors_SMD:C_1206_HandSoldering
- D4: value D -> sTth112
- R11, R12: value DND -> 12; footprint Resistors_SMD:R_MELF_MMB-0207 -> Resistors_SMD:R_0805_HandSoldering
- R13: value 20 -> 12; footprint Resistors_SMD:R_MELF_MMB-0207 -> Resistors_SMD:R_0805_HandSoldering
- R14: value 20 -> 3; footprint Resistors_SMD:R_MELF_MMB-0207 -> Resistors_SMD:R_2512_HandSoldering
- R15: value 47k -> 3; footprint Resistors_SMD:R_0805_HandSoldering -> Resistors_SMD:R_2512_HandSoldering
Connections:
- wire segments 124 -> 155

Commit message: v0.2
Parts:
- D15: footprint Diodes_SMD:D_SMC_Handsoldering -> Diodes_SMD:D_SMC
- Q3, Q4: footprint TO_SOT_Packages_SMD:TO-252-3_TabPin4 -> TO_SOT_Packages_SMD:TO-252-2
Changed lines of the file:
@@
 $Descr A4 11693 8268
 encoding utf-8
-Sheet 5 6
+Sheet 3 6
 Title ""
 Date ""
@@
 F 0 "Q6" H 6288 3654 50  0000 L CNN
 F 1 "MJD45H11RLG" H 6288 3745 50  0000 L CNN
-F 2 "TO_SOT_Packages_SMD:TO-252-3_TabPin4" H 6200 3800 50  0001 C CNN
+F 2 "TO_SOT_Packages_SMD:TO-252-2" H 6200 3800 50  0001 C CNN
 F 3 "" H 6000 3700 50  0001 C CNN
 	1    6000 3700
@@
 F 0 "Q5" H 6288 3146 50  0000 L CNN
 F 1 "MJD44H11RLG" H 6288 3055 50  0000 L CNN
-F 2 "TO_SOT_Packages_SMD:TO-252-3_TabPin4" H 6200 3200 50  0001 C CNN
+F 2 "TO_SOT_Packages_SMD:TO-252-2" H 6200 3200 50  0001 C CNN
 F 3 "" H 6000 3100 50  0001 C CNN
 	1    6000 3100
@@
 F 0 "D21" V 10204 1779 50  0000 L CNN
 F 1 "smcj440ca" V 10295 1779 50  0000 L CNN
-F 2 "Diodes_SMD:D_SMC_Handsoldering" H 10250 1700 50  0001 C CNN
+F 2 "Diodes_SMD:D_SMC" H 10250 1700 50  0001 C CNN
 F 3 "https://en.wikipedia.org/wiki/Transient-voltage-suppression_diode" H 10250 1700 50  0001 C CNN
 	1    10250 1700

Commit message: v2.0 PCB SIGNAL SIDE
Connections:
- net labels removed: VCC_REG
- wire segments 155 -> 156
Changed lines of the file:
@@
 $Descr A4 11693 8268
 encoding utf-8
-Sheet 3 6
+Sheet 5 6
 Title ""
 Date ""
@@
 Text HLabel 8100 2650 1    60   Input ~ 0
 +VCC
-Text HLabel 4200 1950 1    60   Input ~ 0
-VCC_REG
 Text HLabel 5300 2750 2    60   Input ~ 0
 -VEE
@@
 	5200 2750 5300 2750
 Connection ~ 5200 2650
-Connection ~ 4200 2000
-Wire Wire Line
-	4200 2000 4200 1950
 $Comp
 L device:C C22
@@
 Wire Wire Line
 	8500 1250 10250 1250
+Wire Wire Line
+	6100 2700 6100 2000
+Wire Wire Line
+	6100 2000 5650 2000
+Connection ~ 6100 2700
+Connection ~ 5650 2000
 $EndSCHEMATC

Commit message: V0.2 shoot through EMI protection added
In response to Marcos repply to my post on endless sphere https://endless-sphere.com/forums/viewtopic.php?f=30&t=89056&start=75
Parts:
- removed C15, C16: 100n, Capacitors_SMD:C_0805_HandSoldering, symbol device:C
- removed R6: 1k, Resistors_SMD:R_0805_HandSoldering, symbol device:R
- added C14, C26: 100n, Capacitors_SMD:C_0805_HandSoldering, symbol device:C
- added D2: GSOT03C, TO_SOT_Packages_SMD:SOT-23, symbol device:D_Schottky_x2_ACom_KKA
- added R3: 4.7k, Resistors_SMD:R_0805_HandSoldering, symbol device:R
- added R4: 1k, Resistors_SMD:R_0805_HandSoldering, symbol device:R
- R8: value 47k -> 10
Connections:
- net labels added: PWM+, PWM-
- net labels removed: PWM
- wire segments 156 -> 159

Commit message: Schematics update
Parts:
- C14, C18, C19, C24, C25, C26: Mfg.# (none) -> C0805C104J5RACAUTO
- C28, C29: Mfg.# (none) -> UMK212BJ105MG-T
- C30, C31, C32, C33: Mfg.# (none) -> UMK325BJ106KMHP
Connections:
- net labels added: GND_ISO
- wire segments 159 -> 160

Commit message: V0.2 BOM and schematics updated
Parts:
- C17: Mfg.# (none) -> CC0805KRX7R9BB153
- C23: Mfg.# (none) -> UMK325BJ106KMHP
- Q3: value MJD44H11RLG -> MJD3055T4G
- Q4: value MJD45H11RLG -> MJD2955T4G
- R10, R4: Mfg.# (none) -> RC0805JR-071KL
- R11, R12, R13: Mfg.# (none) -> RC0805JR-0712RL
- R24, R7, R9: Mfg.# (none) -> AC0805JR-0710KL
- R3: Mfg.# (none) -> RC0805FR-074K7L
- U4: Mfg.# (none) -> ISO5852SQDWRQ1

Commit message: V0.2 pcb changes
Connections:
- wire segments 160 -> 157
- no-connect marks 1 -> 3
