File: V0.2-IGBT/PCB/GD.sch (KiCad schematic (older format))
At the start: 44 parts, among them Q3 MJD3055T4G, Q4 MJD2955T4G, U4 ISO5852SDWR

Commit message: V0.2
Parts:
- R10: value 10k -> 1k

Commit message: V0.2 completed
Parts:
- R14, R15, R22, R23: footprint Resistors_SMD:R_2512_HandSoldering -> Resistors_SMD:R_2512
Connections:
- wire segments 159 -> 162
Changed lines of the file:
@@
 AR Path="/5A33279F/5A3180B4" Ref="#PWR08"  Part="1"
 AR Path="/5A340028/5A3180B4" Ref="#PWR015"  Part="1"
-F 0 "#PWR08" H 3200 3250 50  0001 C CNN
+F 0 "#PWR015" H 3200 3250 50  0001 C CNN
 F 1 "GND" H 3205 3327 50  0000 C CNN
 F 2 "" H 3200 3500 50  0001 C CNN
@@
 	1    0    0    -1
 $EndComp
-Text HLabel 4200 3500 3    60   Input ~ 0
--VEE
 Wire Wire Line
 	4200 3500 4100 3500
@@
 $EndComp
 Wire Wire Line
-	5300 3450 5300 3150
-Wire Wire Line
 	5800 3100 5800 3150
 Wire Wire Line
 	5300 3150 5800 3150
-Connection ~ 5300 3150
-Connection ~ 5800 3150
-Wire Wire Line
-	5800 3150 5800 3700
 $Comp
 L device:C C23
@@
 F 0 "R15" V 6943 3250 50  0000 C CNN
 F 1 "3" V 7034 3250 50  0000 C CNN
-F 2 "Resistors_SMD:R_2512_HandSoldering" V 7080 3250 50  0001 C CNN
+F 2 "Resistors_SMD:R_2512" V 7080 3250 50  0001 C CNN
 F 3 "" H 7150 3250 50  0001 C CNN
 	1    7150 3250
@@
 F 0 "R22" V 6943 3650 50  0000 C CNN
 F 1 "3" V 7034 3650 50  0000 C CNN
-F 2 "Resistors_SMD:R_2512_HandSoldering" V 7080 3650 50  0001 C CNN
+F 2 "Resistors_SMD:R_2512" V 7080 3650 50  0001 C CNN
 F 3 "" H 7150 3650 50  0001 C CNN
 	1    7150 3650
@@
 F 0 "R14" V 6943 2950 50  0000 C CNN
 F 1 "3" V 7034 2950 50  0000 C CNN
-F 2 "Resistors_SMD:R_2512_HandSoldering" V 7080 2950 50  0001 C CNN
+F 2 "Resistors_SMD:R_2512" V 7080 2950 50  0001 C CNN
 F 3 "" H 7150 2950 50  0001 C CNN
 	1    7150 2950
@@
 F 0 "R23" V 6943 3950 50  0000 C CNN
 F 1 "3" V 7034 3950 50  0000 C CNN
-F 2 "Resistors_SMD:R_2512_HandSoldering" V 7080 3950 50  0001 C CNN
+F 2 "Resistors_SMD:R_2512" V 7080 3950 50  0001 C CNN
 F 3 "" H 7150 3950 50  0001 C CNN
 	1    7150 3950
@@
 AR Path="/5A340028/5A572019" Ref="#PWR018"  Part="1"
 AR Path="/5A33279F/5A572019" Ref="#PWR013"  Part="1"
-F 0 "#PWR013" H 2550 4250 50  0001 C CNN
+F 0 "#PWR018" H 2550 4250 50  0001 C CNN
 F 1 "GND" H 2555 4327 50  0000 C CNN
 F 2 "" H 2550 4500 50  0001 C CNN
@@
 AR Path="/5A33279F/5A5EF2CA" Ref="#PWR017"  Part="1"
 AR Path="/5A340028/5A5EF2CA" Ref="#PWR019"  Part="1"
-F 0 "#PWR017" H 3050 2400 50  0001 C CNN
+F 0 "#PWR019" H 3050 2400 50  0001 C CNN
 F 1 "GND" H 3055 2477 50  0000 C CNN
 F 2 "" H 3050 2650 50  0001 C CNN
@@
 AR Path="/5A33279F/5A689130" Ref="#PWR020"  Part="1"
 AR Path="/5A340028/5A689130" Ref="#PWR038"  Part="1"
-F 0 "#PWR020" H 2350 2700 50  0001 C CNN
+F 0 "#PWR038" H 2350 2700 50  0001 C CNN
 F 1 "GND" H 2500 2900 50  0000 C CNN
 F 2 "" H 2350 2950 50  0001 C CNN
@@
 AR Path="/5A340028/5A30F6FF" Ref="#PWR014"  Part="1"
 AR Path="/5A33279F/5A30F6FF" Ref="#PWR07"  Part="1"
-F 0 "#PWR07" H 1350 4900 50  0001 C CNN
+F 0 "#PWR014" H 1350 4900 50  0001 C CNN
 F 1 "GND" H 1355 4977 50  0000 C CNN
 F 2 "" H 1350 5150 50  0001 C CNN
@@
 Wire Wire Line
 	6100 2700 7600 2700
+Wire Wire Line
+	9650 2700 10250 2700
+Connection ~ 10250 2700
+Wire Wire Line
+	10250 2700 10400 2700
+$Comp
+L device:D_Schottky D16
+U 1 1 5A56D823
+P 7600 3100
+AR Path="/5A33279F/5A56D823" Ref="D16"  Part="1"
+AR Path="/5A340028/5A56D823" Ref="D22"  Part="1"
+F 0 "D16" V 7554 3179 50  0000 L CNN
+F 1 "PMEG4010" V 7645 3179 50  0000 L CNN
+F 2 "Diodes_SMD:D_SOD-323_HandSoldering" H 7600 3100 50  0001 C CNN
+F 3 "" H 7600 3100 50  0001 C CNN
+	1    7600 3100
+	0    1    1    0
+$EndComp
+Connection ~ 7600 3250
+Wire Wire Line
+	7600 2950 7600 2700
+Connection ~ 7600 2700
+Wire Wire Line
+	7600 2700 8000 2700
+Wire Wire Line
+	4200 3500 4200 4450
+Wire Wire Line
+	4200 4450 4700 4450
+Connection ~ 4700 4450
+Wire Wire Line
+	5300 3450 5800 3450
+Wire Wire Line
+	5800 3450 5800 3700
+Wire Wire Line
+	5800 3450 5800 3150
+Connection ~ 5800 3450
+Connection ~ 5800 3150
+Wire Wire Line
+	10250 2300 10250 2700
+Wire Wire Line
+	10250 1850 10250 2000
 $Comp
 L device:D D8
@@
 	0    -1   -1   0
 $EndComp
-Wire Wire Line
-	10250 1850 10250 2000
-Wire Wire Line
-	10250 2300 10250 2700
-Wire Wire Line
-	9650 2700 10250 2700
-Connection ~ 10250 2700
-Wire Wire Line
-	10250 2700 10400 2700
-$Comp
-L device:D_Schottky D16
-U 1 1 5A56D823
-P 7600 3100
-AR Path="/5A33279F/5A56D823" Ref="D16"  Part="1"
-AR Path="/5A340028/5A56D823" Ref="D22"  Part="1"
-F 0 "D16" V 7554 3179 50  0000 L CNN
-F 1 "PMEG4010" V 7645 3179 50  0000 L CNN
-F 2 "Diodes_SMD:D_SOD-323_HandSoldering" H 7600 3100 50  0001 C CNN
-F 3 "" H 7600 3100 50  0001 C CNN
-	1    7600 3100
-	0    1    1    0
-$EndComp
-Connection ~ 7600 3250
-Wire Wire Line
-	7600 2950 7600 2700
-Connection ~ 7600 2700
-Wire Wire Line
-	7600 2700 8000 2700
 $EndSCHEMATC

Commit message: Maintenance update
Parts:
- C14, C17, C18, C19, C20, C21, C22, C23, C24, C25, C26, C28, C29, C30, C31, C32, C33, C34: symbol device:C -> ENNOID-Dual-Gate-Driver-rescue:C-device
- D10, D16: symbol device:D_Schottky -> ENNOID-Dual-Gate-Driver-rescue:D_Schottky-device
- D11, D15: symbol device:D_TVS -> ENNOID-Dual-Gate-Driver-rescue:D_TVS-device
- D2: symbol device:D_Schottky_x2_ACom_KKA -> ENNOID-Dual-Gate-Driver-rescue:D_Schottky_x2_ACom_KKA-device
- D3, D4, D8: symbol device:D -> ENNOID-Dual-Gate-Driver-rescue:D-device
- D6: symbol device:D_Zener -> ENNOID-Dual-Gate-Driver-rescue:D_Zener-device
- Q3: symbol device:Q_NPN_Darlington_BCEC -> ENNOID-Dual-Gate-Driver-rescue:Q_NPN_Darlington_BCEC-device
- Q4: symbol device:Q_PNP_Darlington_BCEC -> ENNOID-Dual-Gate-Driver-rescue:Q_PNP_Darlington_BCEC-device
- R10, R11, R12, R13, R14, R15, R22, R23, R24, R3, R4, R7, R8, R9: symbol device:R -> ENNOID-Dual-Gate-Driver-rescue:R-device
Connections:
- wire segments 162 -> 163
Other:
- note added: "Adj. soft turnoff\nSee tiduc70a.pdf"
- note added: "Desat see tiduc70a.pdf"
- note added: "Limit transcient\n here"
- note added: "Limit voltage and transcient here"
- note added: "Transcient suppression"
- note added: "basic clamping /\nIGBt overvoltage protection"
- note added: "gate/ emitter\ntranscient\novervoltage protection\n& Vg=Ve at standstill"
- note added: "when fault = mute input"

Commit message: Maintenance update
Parts:
- D6: footprint Diodes_SMD:D_SOD-323 -> Diodes_SMD:D_SOD-323_HandSoldering
