File: V0.2-IGBT/PCB/ENNOID Dual Gate Driver.sch (KiCad schematic (older format))
At the start: 26 parts, among them J1 Conn_02x08_Odd_Even, J2 Current, J3 TEMP, J4 PHASE, J5 Collector, J6 Gate_H, J7 G_L, J8 E, U1 MC7805

Commit message: v0.2 PCB
Changed lines of the file:
@@
 Text GLabel 1550 6500 0    60   Input ~ 0
 RST
-Text GLabel 2300 6500 2    60   Input ~ 0
+Text GLabel 2300 6500 2    60   Output ~ 0
 FLT
 Wire Wire Line
@@
 Wire Wire Line
 	2200 6500 2300 6500
-Text GLabel 4400 1550 0    60   Input ~ 0
+Text GLabel 4400 1550 0    60   Output ~ 0
 FLT
 $Comp
@@
 Text GLabel 1500 4700 3    60   Input ~ 0
 FLT
-Text GLabel 4550 3500 0    60   Input ~ 0
+Text GLabel 4550 3500 0    60   Output ~ 0
 FLT
 Wire Wire Line

Commit message: v2.0 PCB SIGNAL SIDE
Connections:
- wire segments 117 -> 115
Changed lines of the file:
@@
 F4 "+VCC" O R 2700 800 60
 F5 "-VEE" O R 2700 1000 60
-F6 "VCC_REG" O R 2700 900 60
-F7 "PHASE" O R 2700 1100 60
+F6 "PHASE" O R 2700 1100 60
 $EndSheet
 Wire Wire Line
@@
 F4 "RDY" I L 4900 1350 60
 F5 "PWM" I L 4900 1250 60
-F6 "VCC_REG" I L 4900 900 60
-F7 "-VEE" I L 4900 1000 60
-F8 "+VCC" I L 4900 800 60
-F9 "E" I R 6200 1700 60
-F10 "C" I R 6200 750 60
-F11 "G" I R 6200 1200 60
-F12 "+5V" I L 4900 700 60
-F13 "GND" I L 4900 1750 60
+F6 "-VEE" I L 4900 1000 60
+F7 "+VCC" I L 4900 800 60
+F8 "E" I R 6200 1700 60
+F9 "C" I R 6200 750 60
+F10 "G" I R 6200 1200 60
+F11 "+5V" I L 4900 700 60
+F12 "GND" I L 4900 1750 60
 $EndSheet
 $Sheet
@@
 F4 "+VCC" O R 2500 2850 60
 F5 "-VEE" O R 2500 3050 60
-F6 "VCC_REG" O R 2500 2950 60
-F7 "PHASE" O R 2500 3150 60
+F6 "PHASE" O R 2500 3150 60
 $EndSheet
 $Comp
@@
 F7 "GND" I L 4950 3700 60
 F8 "+VCC" I L 4950 2850 60
-F9 "VCC_REG" I L 4950 2950 60
-F10 "-VEE" I L 4950 3050 60
-F11 "C" I R 6200 2700 60
-F12 "G" I R 6200 3200 60
-F13 "E" I R 6200 3650 60
+F9 "-VEE" I L 4950 3050 60
+F10 "C" I R 6200 2700 60
+F11 "G" I R 6200 3200 60
+F12 "E" I R 6200 3650 60
 $EndSheet
 Wire Wire Line
@@
 Wire Wire Line
 	2700 800  4900 800
-Wire Wire Line
-	2700 900  4900 900
 Wire Wire Line
 	2700 1000 4900 1000
@@
 Text GLabel 4400 1350 0    60   Input ~ 0
 RDY
-Text GLabel 2700 6800 2    60   Input ~ 0
+Text GLabel 950  6800 0    60   Input ~ 0
 PWM_L
 Wire Wire Line
@@
 Text GLabel 4550 3300 0    60   Input ~ 0
 RDY
-Text GLabel 1000 6800 0    60   Input ~ 0
+Text GLabel 2650 6800 2    60   Input ~ 0
 PWM_H
 Text GLabel 1550 6500 0    60   Input ~ 0
@@
 Wire Wire Line
 	4900 5500 4550 5500
+Text GLabel 2300 6400 2    60   Output ~ 0
+Vout+
 Text GLabel 1550 6400 0    60   Output ~ 0
-Vout+
-Text GLabel 2300 6400 2    60   Output ~ 0
 Vout-
 $Comp
@@
 	1550 6300 1700 6300
 Wire Wire Line
-	1550 6400 1700 6400
-Wire Wire Line
 	1550 6500 1700 6500
 Wire Wire Line
 	2200 6300 2300 6300
-Wire Wire Line
-	2300 6400 2200 6400
 NoConn ~ 2200 6600
 NoConn ~ 1700 6600
@@
 	1    0    0    -1
 $EndComp
-Connection ~ 1100 6800
-Wire Wire Line
-	1000 6800 1100 6800
-Connection ~ 2500 6800
-Wire Wire Line
-	2500 6800 2700 6800
-Wire Wire Line
-	2500 2950 4950 2950
 Wire Wire Line
 	3150 5200 4900 5200
@@
 Wire Wire Line
 	1850 4600 1850 4700
+Wire Wire Line
+	2200 6400 2300 6400
+Wire Wire Line
+	1700 6400 1550 6400
+Wire Wire Line
+	950  6800 1100 6800
+Connection ~ 1100 6800
+Wire Wire Line
+	2650 6800 2500 6800
+Connection ~ 2500 6800
 $EndSCHEMATC

Commit message: V0.2 shoot through EMI protection added
In response to Marcos repply to my post on endless sphere https://endless-sphere.com/forums/viewtopic.php?f=30&t=89056&start=75
Connections:
- wire segments 115 -> 117
Changed lines of the file:
@@
 L power:GND #PWR02
 U 1 1 5A33266A
-P 1100 3150
-F 0 "#PWR02" H 1100 2900 50  0001 C CNN
-F 1 "GND" H 1105 2977 50  0001 C CNN
-F 2 "" H 1100 3150 50  0001 C CNN
-F 3 "" H 1100 3150 50  0001 C CNN
-	1    1100 3150
-	1    0    0    -1
-$EndComp
-Wire Wire Line
-	1300 2900 1150 2900
-Wire Wire Line
-	1100 3150 1100 3100
-Wire Wire Line
-	1100 3100 1300 3100
+P 1100 3100
+F 0 "#PWR02" H 1100 2850 50  0001 C CNN
+F 1 "GND" H 1105 2927 50  0001 C CNN
+F 2 "" H 1100 3100 50  0001 C CNN
+F 3 "" H 1100 3100 50  0001 C CNN
+	1    1100 3100
+	1    0    0    -1
+$EndComp
+Wire Wire Line
+	1300 2850 1150 2850
+Wire Wire Line
+	1100 3100 1100 3050
+Wire Wire Line
+	1100 3050 1300 3050
 $Sheet
 S 4900 650  1300 1150
@@
 F3 "FLT" O L 4900 1550 60
 F4 "RDY" I L 4900 1350 60
-F5 "PWM" I L 4900 1250 60
+F5 "PWM+" I L 4900 1150 60
 F6 "-VEE" I L 4900 1000 60
 F7 "+VCC" I L 4900 800 60
@@
 F11 "+5V" I L 4900 700 60
 F12 "GND" I L 4900 1750 60
+F13 "PWM-" I L 4900 1250 50
 $EndSheet
 $Sheet
-S 1300 2800 1200 400
+S 1300 2750 1200 400
 U 5A331F4C
 F0 "ISO_PSU_LOW" 60
 F1 "ISO_PSU.sch" 60
-F2 "VCC_IN" I L 1300 2900 60
-F3 "GND" I L 1300 3100 60
-F4 "+VCC" O R 2500 2850 60
-F5 "-VEE" O R 2500 3050 60
-F6 "PHASE" O R 2500 3150 60
+F2 "VCC_IN" I L 1300 2850 60
+F3 "GND" I L 1300 3050 60
+F4 "+VCC" O R 2500 2800 60
+F5 "-VEE" O R 2500 3000 60
+F6 "PHASE" O R 2500 3100 60
 $EndSheet
 $Comp
@@
 F0 "GD_LOW" 60
 F1 "GD.sch" 60
-F2 "+5V" I L 4950 2750 60
+F2 "+5V" I L 4950 2700 60
 F3 "RST" I L 4950 3400 60
 F4 "FLT" O L 4950 3500 60
 F5 "RDY" I L 4950 3300 60
-F6 "PWM" I L 4950 3200 60
+F6 "PWM+" I L 4950 3100 60
 F7 "GND" I L 4950 3700 60
-F8 "+VCC" I L 4950 2850 60
-F9 "-VEE" I L 4950 3050 60
+F8 "+VCC" I L 4950 2800 60
+F9 "-VEE" I L 4950 3000 60
 F10 "C" I R 6200 2700 60
 F11 "G" I R 6200 3200 60
 F12 "E" I R 6200 3650 60
+F13 "PWM-" I L 4950 3200 50
 $EndSheet
 Wire Wire Line
@@
 	2700 1000 4900 1000
 Wire Wire Line
-	2500 2850 3150 2850
-Wire Wire Line
-	2500 3050 4950 3050
+	2500 2800 3150 2800
+Wire Wire Line
+	2500 3000 4950 3000
 Wire Wire Line
 	2700 1100 3600 1100
@@
 	3600 2200 7200 2200
 Wire Wire Line
-	2500 3150 3550 3150
-Wire Wire Line
-	3550 3150 3550 4300
+	2500 3100 3550 3100
+Wire Wire Line
+	3550 3100 3550 4300
 Wire Wire Line
 	3550 4300 7200 4300
@@
 Text GLabel 4400 1450 0    60   Input ~ 0
 RST
-Text GLabel 4400 1250 0    60   Input ~ 0
+Text GLabel 4400 1150 0    60   Input ~ 0
 PWM_H
 Text GLabel 4400 1350 0    60   Input ~ 0
@@
 PWM_L
 Wire Wire Line
-	4400 1250 4900 1250
+	4400 1150 4900 1150
 Wire Wire Line
 	4400 1450 4900 1450
@@
 Wire Wire Line
 	4900 1550 4400 1550
-Text GLabel 4550 3200 0    60   Input ~ 0
+Text GLabel 4550 3100 0    60   Input ~ 0
 PWM_L
 Wire Wire Line
-	4550 3200 4950 3200
+	4550 3100 4950 3100
 Text GLabel 4550 3400 0    60   Input ~ 0
 RST
@@
 L power:+5V #PWR032
 U 1 1 5A344C1F
-P 4800 2750
-F 0 "#PWR032" H 4800 2600 50  0001 C CNN
-F 1 "+5V" H 4815 2923 50  0000 C CNN
-F 2 "" H 4800 2750 50  0001 C CNN
-F 3 "" H 4800 2750 50  0001 C CNN
-	1    4800 2750
-	1    0    0    -1
-$EndComp
-Wire Wire Line
-	4800 2750 4950 2750
+P 4800 2700
+F 0 "#PWR032" H 4800 2550 50  0001 C CNN
+F 1 "+5V" H 4815 2873 50  0000 C CNN
+F 2 "" H 4800 2700 50  0001 C CNN
+F 3 "" H 4800 2700 50  0001 C CNN
+	1    4800 2700
+	1    0    0    -1
+$EndComp
+Wire Wire Line
+	4800 2700 4950 2700
 $Comp
 L power:+5V #PWR029
@@
 L power:+24V #PWR045
 U 1 1 5A3CC538
-P 1150 2900
-F 0 "#PWR045" H 1150 2750 50  0001 C CNN
-F 1 "+24V" H 1165 3073 50  0000 C CNN
-F 2 "" H 1150 2900 50  0001 C CNN
-F 3 "" H 1150 2900 50  0001 C CNN
-	1    1150 2900
+P 1150 2850
+F 0 "#PWR045" H 1150 2700 50  0001 C CNN
+F 1 "+24V" H 1165 3023 50  0000 C CNN
+F 2 "" H 1150 2850 50  0001 C CNN
+F 3 "" H 1150 2850 50  0001 C CNN
+	1    1150 2850
 	1    0    0    -1
 $EndComp
@@
 	1300 7400 1050 7400
 Connection ~ 1300 7400
-Text GLabel 1050 2900 0    60   Input ~ 0
+Text GLabel 1050 2850 0    60   Input ~ 0
 VCC_IN
 Wire Wire Line
-	1150 2900 1050 2900
-Connection ~ 1150 2900
+	1150 2850 1050 2850
+Connection ~ 1150 2850
 Text GLabel 1150 850  0    60   Input ~ 0
 VCC_IN
@@
 	3150 5200 4900 5200
 Wire Wire Line
-	3150 2850 3150 5200
-Connection ~ 3150 2850
-Wire Wire Line
-	3150 2850 4950 2850
+	3150 2800 3150 5200
+Connection ~ 3150 2800
+Wire Wire Line
+	3150 2800 4950 2800
 $Comp
 L power:+5V #PWR012
@@
 	2650 6800 2500 6800
 Connection ~ 2500 6800
+Wire Notes Line
+	5350 500  5350 6100
+Wire Notes Line
+	5650 6100 5650 500
+Text GLabel 4400 1250 0    60   Input ~ 0
+PWM_L
+Wire Wire Line
+	4400 1250 4900 1250
+Text GLabel 4550 3200 0    60   Input ~ 0
+PWM_H
+Wire Wire Line
+	4550 3200 4950 3200
 $EndSCHEMATC

Commit message: Schematics update
Parts:
- C1: Mfg.# (none) -> UMK325BJ106KMHP
- C2, C3, C41, C42: Mfg.# (none) -> C0805C104J5RACAUTO
- C4, C43, C44: Mfg.# (none) -> UMK212BJ105MG-T
- F1: Mfg.# (none) -> MFU0805FF01000P100
- U1: Mfg.# (none) -> MC7805BDTRKG
Connections:
- net labels removed: VCC_IN
- wire segments 117 -> 123

Commit message: V0.2 BOM and schematics updated
Parts:
- D12, D13, D14: Mfg.# (none) -> LTW-170TK
- J1: Mfg.# (none) -> 30316-6002HB
- R16, R34, R5: value 1k -> 300; Mfg.# (none) -> RK73B2ATTDD301J
Changed lines of the file:
@@
 F 1 "Conn_02x08_Odd_Even" H 1950 7026 50  0001 C CNN
 F 2 "ENNOID:Multicomp_MC9A12-1634_2x08x2.54mm_Straight" H 1900 6600 50  0001 C CNN
-F 3 "~" H 1900 6600 50  0001 C CNN
+F 3 "http://www.mouser.com/ds/2/1/TS0818-221281.pdf" H 1900 6600 50  0001 C CNN
+F 4 "30316-6002HB " H 1900 6600 50  0001 C CNN "Mfg.#"
 	1    1900 6600
 	1    0    0    -1
@@
 P 1150 1400
 F 0 "R5" H 1220 1446 50  0000 L CNN
-F 1 "1k" H 1220 1355 50  0000 L CNN
+F 1 "300" H 1220 1355 50  0000 L CNN
 F 2 "Resistors_SMD:R_0805_HandSoldering" V 1080 1400 50  0001 C CNN
 F 3 "" H 1150 1400 50  0001 C CNN
+F 4 "RK73B2ATTDD301J" H 1150 1400 50  0001 C CNN "Mfg.#"
 	1    1150 1400
 	1    0    0    -1
@@
 P 1500 1400
 F 0 "R16" H 1570 1446 50  0000 L CNN
-F 1 "1k" H 1570 1355 50  0000 L CNN
+F 1 "300" H 1570 1355 50  0000 L CNN
 F 2 "Resistors_SMD:R_0805_HandSoldering" V 1430 1400 50  0001 C CNN
 F 3 "" H 1500 1400 50  0001 C CNN
+F 4 "RK73B2ATTDD301J" H 1500 1400 50  0001 C CNN "Mfg.#"
 	1    1500 1400
 	1    0    0    -1
@@
 P 1850 1400
 F 0 "R34" H 1920 1446 50  0000 L CNN
-F 1 "1k" H 1920 1355 50  0000 L CNN
+F 1 "300" H 1920 1355 50  0000 L CNN
 F 2 "Resistors_SMD:R_0805_HandSoldering" V 1780 1400 50  0001 C CNN
 F 3 "" H 1850 1400 50  0001 C CNN
+F 4 "RK73B2ATTDD301J" H 1850 1400 50  0001 C CNN "Mfg.#"
 	1    1850 1400
 	1    0    0    -1
@@
 F 1 "LED" V 1097 1733 50  0000 R CNN
 F 2 "LEDs:LED_0805_HandSoldering" H 1150 1850 50  0001 C CNN
-F 3 "~" H 1150 1850 50  0001 C CNN
+F 3 "http://www.mouser.com/ds/2/239/Lite-On-LTW-170TK-1175303.pdf" H 1150 1850 50  0001 C CNN
+F 4 "LTW-170TK " V 1150 1850 50  0001 C CNN "Mfg.#"
 	1    1150 1850
 	0    -1   -1   0
@@
 F 1 "LED" V 1447 1733 50  0000 R CNN
 F 2 "LEDs:LED_0805_HandSoldering" H 1500 1850 50  0001 C CNN
-F 3 "~" H 1500 1850 50  0001 C CNN
+F 3 "http://www.mouser.com/ds/2/239/Lite-On-LTW-170TK-1175303.pdf" H 1500 1850 50  0001 C CNN
+F 4 "LTW-170TK " V 1500 1850 50  0001 C CNN "Mfg.#"
 	1    1500 1850
 	0    -1   -1   0
@@
 F 1 "LED" V 1797 1733 50  0000 R CNN
 F 2 "LEDs:LED_0805_HandSoldering" H 1850 1850 50  0001 C CNN
-F 3 "~" H 1850 1850 50  0001 C CNN
+F 3 "http://www.mouser.com/ds/2/239/Lite-On-LTW-170TK-1175303.pdf" H 1850 1850 50  0001 C CNN
+F 4 "LTW-170TK " V 1850 1850 50  0001 C CNN "Mfg.#"
 	1    1850 1850
 	0    -1   -1   0

Commit message: V0.2 PCB
Parts:
- U1: footprint TO_SOT_Packages_SMD:TO-252-3_TabPin2 -> TO_SOT_Packages_SMD:TO-252-2
Changed lines of the file:
@@
 F 0 "U1" H 2050 3442 50  0000 C CNN
 F 1 "MC7805" H 2050 3351 50  0000 C CNN
-F 2 "TO_SOT_Packages_SMD:TO-252-3_TabPin2" H 2075 3050 50  0001 L CIN
+F 2 "TO_SOT_Packages_SMD:TO-252-2" H 2075 3050 50  0001 L CIN
 F 3 "http://www.mouser.com/ds/2/308/MC7800-D-94905.pdf" H 2050 3150 50  0001 C CNN
 F 4 "MC7805BDTRKG" H 2050 3200 50  0001 C CNN "Mfg.#"

Commit message: Maintenance update
Parts:
- C1, C2, C3, C4, C41, C42, C43, C44: symbol device:C -> ENNOID-Dual-Gate-Driver-rescue:C-device
- D12, D13, D14: symbol device:LED -> ENNOID-Dual-Gate-Driver-rescue:LED-device
- F1: symbol device:Fuse -> ENNOID-Dual-Gate-Driver-rescue:Fuse-device
- J1: symbol Connector:Conn_02x08_Odd_Even -> ENNOID-Dual-Gate-Driver-rescue:Conn_02x08_Odd_Even-Connector
- J2: symbol Connector:Conn_01x04 -> ENNOID-Dual-Gate-Driver-rescue:Conn_01x04-Connector
- J3: symbol Connector:Conn_01x02 -> ENNOID-Dual-Gate-Driver-rescue:Conn_01x02-Connector
- J4, J5, J6, J7, J8: symbol Connector:Conn_01x01_Female -> ENNOID-Dual-Gate-Driver-rescue:Conn_01x01_Female-Connector
- R16, R32, R33, R34, R5: symbol device:R -> ENNOID-Dual-Gate-Driver-rescue:R-device
- U1: symbol regul:L7805 -> ENNOID-Dual-Gate-Driver-rescue:L7805-regul
Changed lines of the file:
@@
 $EndDescr
 $Comp
-L Connector:Conn_02x08_Odd_Even J1
+L ENNOID-Dual-Gate-Driver-rescue:Conn_02x08_Odd_Even-Connector J1
 U 1 1 5A3005AC
 P 1900 6600
@@
 Wire Wire Line
 	4750 2200 4900 2200
-$Comp
-L power:GND #PWR01
-U 1 1 5A300A30
-P 4700 2450
-F 0 "#PWR01" H 4700 2200 50  0001 C CNN
-F 1 "GND" H 4705 2277 50  0001 C CNN
-F 2 "" H 4700 2450 50  0001 C CNN
-F 3 "" H 4700 2450 50  0001 C CNN
-	1    4700 2450
-	1    0    0    -1
-$EndComp
 Wire Wire Line
 	4900 2400 4700 2400
 Wire Wire Line
 	4700 2400 4700 2450
-$Comp
-L power:GND #PWR02
-U 1 1 5A33266A
-P 4700 3200
-F 0 "#PWR02" H 4700 2950 50  0001 C CNN
-F 1 "GND" H 4705 3027 50  0001 C CNN
-F 2 "" H 4700 3200 50  0001 C CNN
-F 3 "" H 4700 3200 50  0001 C CNN
-	1    4700 3200
-	1    0    0    -1
-$EndComp
 Wire Wire Line
 	4900 2950 4750 2950
@@
 $EndSheet
 $Comp
-L device:C C1
+L ENNOID-Dual-Gate-Driver-rescue:C-device C1
 U 1 1 5A33DEE4
 P 900 3350
@@
 $EndComp
 $Comp
-L device:C C2
+L ENNOID-Dual-Gate-Driver-rescue:C-device C2
 U 1 1 5A33DFE6
 P 1350 3350
@@
 	900  3200 1200 3200
 $Comp
-L device:C C3
+L ENNOID-Dual-Gate-Driver-rescue:C-device C3
 U 1 1 5A33E247
 P 2500 3350
@@
 $EndComp
 $Comp
-L device:C C4
+L ENNOID-Dual-Gate-Driver-rescue:C-device C4
 U 1 1 5A33E2F7
 P 2950 3350
@@
 $EndComp
 $Comp
-L regul:L7805 U1
+L ENNOID-Dual-Gate-Driver-rescue:L7805-regul U1
 U 1 1 5A33E500
 P 2050 3200
@@
 	1350 3500 900  3500
 Connection ~ 1350 3500
-$Comp
-L power:GND #PWR03
-U 1 1 5A33ED69
-P 2050 3550
-F 0 "#PWR03" H 2050 3300 50  0001 C CNN
-F 1 "GND" H 2055 3377 50  0001 C CNN
-F 2 "" H 2050 3550 50  0001 C CNN
-F 3 "" H 2050 3550 50  0001 C CNN
-	1    2050 3550
-	1    0    0    -1
-$EndComp
 Wire Wire Line
 	2050 3550 2050 3500
@@
 Wire Wire Line
 	4500 4300 4900 4300
-$Comp
-L power:GND #PWR06
-U 1 1 5A3D9814
-P 4800 4700
-F 0 "#PWR06" H 4800 4450 50  0001 C CNN
-F 1 "GND" H 4805 4527 50  0001 C CNN
-F 2 "" H 4800 4700 50  0001 C CNN
-F 3 "" H 4800 4700 50  0001 C CNN
-	1    4800 4700
-	1    0    0    -1
-$EndComp
-$Comp
-L power:GND #PWR05
-U 1 1 5A3D9C57
-P 4800 1750
-F 0 "#PWR05" H 4800 1500 50  0001 C CNN
-F 1 "GND" H 4805 1577 50  0001 C CNN
-F 2 "" H 4800 1750 50  0001 C CNN
-F 3 "" H 4800 1750 50  0001 C CNN
-	1    4800 1750
-	1    0    0    -1
-$EndComp
 Wire Wire Line
 	4800 1750 4900 1750
@@
 	4900 4700 4800 4700
 $Comp
-L Connector:Conn_01x04 J2
+L ENNOID-Dual-Gate-Driver-rescue:Conn_01x04-Connector J2
 U 1 1 5A320690
 P 2150 4450
@@
 $EndComp
 $Comp
-L device:C C43
+L ENNOID-Dual-Gate-Driver-rescue:C-device C43
 U 1 1 5A320A25
 P 1250 4500
@@
 	1    0    0    -1
 $EndComp
-$Comp
-L power:GND #PWR028
-U 1 1 5A320B77
-P 1250 4750
-F 0 "#PWR028" H 1250 4500 50  0001 C CNN
-F 1 "GND" H 1255 4577 50  0001 C CNN
-F 2 "" H 1250 4750 50  0001 C CNN
-F 3 "" H 1250 4750 50  0001 C CNN
-	1    1250 4750
-	1    0    0    -1
-$EndComp
 Wire Wire Line
 	1250 4650 1250 4750
@@
 	1250 4650 1950 4650
 $Comp
-L Connector:Conn_01x02 J3
+L ENNOID-Dual-Gate-Driver-rescue:Conn_01x02-Connector J3
 U 1 1 5A3298CC
 P 4600 7100
@@
 $EndComp
 $Comp
-L device:C C44
+L ENNOID-Dual-Gate-Driver-rescue:C-device C44
 U 1 1 5A329B46
 P 4050 7300
@@
 	4350 7450 4050 7450
 $Comp
-L device:R R33
+L ENNOID-Dual-Gate-Driver-rescue:R-device R33
 U 1 1 5A32DB7E
 P 4050 6850
@@
 $EndComp
 $Comp
-L device:R R32
+L ENNOID-Dual-Gate-Driver-rescue:R-device R32
 U 1 1 5A32DDF0
 P 3800 7100
@@
 	1    0    0    -1
 $EndComp
-$Comp
-L power:GND #PWR034
-U 1 1 5A330589
-P 4050 7500
-F 0 "#PWR034" H 4050 7250 50  0001 C CNN
-F 1 "GND" H 4055 7327 50  0001 C CNN
-F 2 "" H 4050 7500 50  0001 C CNN
-F 3 "" H 4050 7500 50  0001 C CNN
-	1    4050 7500
-	1    0    0    -1
-$EndComp
 Wire Wire Line
 	4050 7500 4050 7450
@@
 Wire Wire Line
 	4900 5200 4750 5200
-$Comp
-L power:GND #PWR031
-U 1 1 5A34C1EE
-P 4750 5850
-F 0 "#PWR031" H 4750 5600 50  0001 C CNN
-F 1 "GND" H 4755 5677 50  0001 C CNN
-F 2 "" H 4750 5850 50  0001 C CNN
-F 3 "" H 4750 5850 50  0001 C CNN
-	1    4750 5850
-	1    0    0    -1
-$EndComp
-Wire Wire Line
-	4750 5850 4900 5850
 Text GLabel 4550 5600 0    60   Output ~ 0
 Vout+
@@
 $EndComp
 $Comp
-L Connector:Conn_01x01_Female J5
+L ENNOID-Dual-Gate-Driver-rescue:Conn_01x01_Female-Connector J5
 U 1 1 5A33A1F4
 P 8400 750
@@
 $EndComp
 $Comp
-L Connector:Conn_01x01_Female J6
+L ENNOID-Dual-Gate-Driver-rescue:Conn_01x01_Female-Connector J6
 U 1 1 5A33C74C
 P 8400 1150
@@
 PHASE
 $Comp
-L Connector:Conn_01x01_Female J4
+L ENNOID-Dual-Gate-Driver-rescue:Conn_01x01_Female-Connector J4
 U 1 1 5A3425E9
 P 8350 2950
@@
 Connection ~ 2200 7000
 $Comp
-L device:Fuse F1
+L ENNOID-Dual-Gate-Driver-rescue:Fuse-device F1
 U 1 1 5A3CFD36
 P 1500 7400
@@
 	1300 7400 1350 7400
 $Comp
-L power:GND #PWR022
-U 1 1 5A3E96FC
-P 1100 7200
-F 0 "#PWR022" H 1100 6950 50  0001 C CNN
-F 1 "GND" H 1105 7027 50  0001 C CNN
-F 2 "" H 1100 7200 50  0001 C CNN
-F 3 "" H 1100 7200 50  0001 C CNN
-	1    1100 7200
-	1    0    0    -1
-$EndComp
-$Comp
-L device:C C42
+L ENNOID-Dual-Gate-Driver-rescue:C-device C42
 U 1 1 5A3EC109
 P 2500 6950
@@
 	1    0    0    -1
 $EndComp
-$Comp
-L power:GND #PWR026
-U 1 1 5A3F1B0E
-P 2500 7150
-F 0 "#PWR026" H 2500 6900 50  0001 C CNN
-F 1 "GND" H 2505 6977 50  0001 C CNN
-F 2 "" H 2500 7150 50  0001 C CNN
-F 3 "" H 2500 7150 50  0001 C CNN
-	1    2500 7150
-	1    0    0    -1
-$EndComp
 Wire Wire Line
 	2500 7100 2500 7150
@@
 	3550 7100 3650 7100
 $Comp
-L Connector:Conn_01x01_Female J7
+L ENNOID-Dual-Gate-Driver-rescue:Conn_01x01_Female-Connector J7
 U 1 1 5A338421
 P 8350 4300
@@
 $EndComp
 $Comp
-L Connector:Conn_01x01_Female J8
+L ENNOID-Dual-Gate-Driver-rescue:Conn_01x01_Female-Connector J8
 U 1 1 5A33858B
 P 8400 4700
@@
 $EndComp
 $Comp
-L device:C C41
+L ENNOID-Dual-Gate-Driver-rescue:C-device C41
 U 1 1 5A3DD0B7
 P 1100 6950
@@
 $EndComp
 $Comp
-L device:R R5
+L ENNOID-Dual-Gate-Driver-rescue:R-device R5
 U 1 1 5A4D972A
 P 1150 1400
@@
 $EndComp
 $Comp
-L device:R R16
+L ENNOID-Dual-Gate-Driver-rescue:R-device R16
 U 1 1 5A4D9A5E
 P 1500 1400
@@
 $EndComp
 $Comp
-L device:R R34
+L ENNOID-Dual-Gate-Driver-rescue:R-device R34
 U 1 1 5A4D9BE2
 P 1850 1400
@@
 	1500 1250 1850 1250
 $Comp
-L device:LED D12
+L ENNOID-Dual-Gate-Driver-rescue:LED-device D12
 U 1 1 5A4F44B8
 P 1150 1850
@@
 $EndComp
 $Comp
-L device:LED D13
+L ENNOID-Dual-Gate-Driver-rescue:LED-device D13
 U 1 1 5A4F4A2D
 P 1500 1850
@@
 $EndComp
 $Comp
-L device:LED D14
+L ENNOID-Dual-Gate-Driver-rescue:LED-device D14
 U 1 1 5A4F4BC5
 P 1850 1850
@@
 	6200 5500 6750 5500
 Connection ~ 6750 4300
+$Comp
+L power:GND #PWR01
+U 1 1 5A60DF81
+P 2050 3550
+F 0 "#PWR01" H 2050 3300 50  0001 C CNN
+F 1 "GND" H 2055 3377 50  0000 C CNN
+F 2 "" H 2050 3550 50  0001 C CNN
+F 3 "" H 2050 3550 50  0001 C CNN
+	1    2050 3550
+	1    0    0    -1
+$EndComp
+$Comp
+L power:GND #PWR02
+U 1 1 5A60E0BD
+P 1250 4750
+F 0 "#PWR02" H 1250 4500 50  0001 C CNN
+F 1 "GND" H 1255 4577 50  0000 C CNN
+F 2 "" H 1250 4750 50  0001 C CNN
+F 3 "" H 1250 4750 50  0001 C CNN
+	1    1250 4750
+	1    0    0    -1
+$EndComp
+$Comp
+L power:GND #PWR03
+U 1 1 5A60E40B
+P 1100 7200
+F 0 "#PWR03" H 1100 6950 50  0001 C CNN
+F 1 "GND" H 1105 7027 50  0000 C CNN
+F 2 "" H 1100 7200 50  0001 C CNN
+F 3 "" H 1100 7200 50  0001 C CNN
+	1    1100 7200
+	1    0    0    -1
+$EndComp
+$Comp
+L power:GND #PWR05
+U 1 1 5A60E44A
+P 2500 7150
+F 0 "#PWR05" H 2500 6900 50  0001 C CNN
+F 1 "GND" H 2505 6977 50  0000 C CNN
+F 2 "" H 2500 7150 50  0001 C CNN
+F 3 "" H 2500 7150 50  0001 C CNN
+	1    2500 7150
+	1    0    0    -1
+$EndComp
+$Comp
+L power:GND #PWR06
+U 1 1 5A60E489
+P 4050 7500
+F 0 "#PWR06" H 4050 7250 50  0001 C CNN
+F 1 "GND" H 4055 7327 50  0000 C CNN
+F 2 "" H 4050 7500 50  0001 C CNN
+F 3 "" H 4050 7500 50  0001 C CNN
+	1    4050 7500
+	1    0    0    -1
+$EndComp
+$Comp
+L power:GND #PWR09
+U 1 1 5A60E66C
+P 4700 2450
+F 0 "#PWR09" H 4700 2200 50  0001 C CNN
+F 1 "GND" H 4705 2277 50  0000 C CNN
+F 2 "" H 4700 2450 50  0001 C CNN
+F 3 "" H 4700 2450 50  0001 C CNN
+	1    4700 2450
+	1    0    0    -1
+$EndComp
+$Comp
+L power:GND #PWR010
+U 1 1 5A60E7E4
+P 4800 1750
+F 0 "#PWR010" H 4800 1500 50  0001 C CNN
+F 1 "GND" H 4805 1577 50  0000 C CNN
+F 2 "" H 4800 1750 50  0001 C CNN
+F 3 "" H 4800 1750 50  0001 C CNN
+	1    4800 1750
+	1    0    0    -1
+$EndComp
+$Comp
+L power:GND #PWR011
+U 1 1 5A60E823
+P 4700 3200
+F 0 "#PWR011" H 4700 2950 50  0001 C CNN
+F 1 "GND" H 4705 3027 50  0000 C CNN
+F 2 "" H 4700 3200 50  0001 C CNN
+F 3 "" H 4700 3200 50  0001 C CNN
+	1    4700 3200
+	1    0    0    -1
+$EndComp
+$Comp
+L power:GND #PWR016
+U 1 1 5A60E8A1
+P 4800 4700
+F 0 "#PWR016" H 4800 4450 50  0001 C CNN
+F 1 "GND" H 4805 4527 50  0000 C CNN
+F 2 "" H 4800 4700 50  0001 C CNN
+F 3 "" H 4800 4700 50  0001 C CNN
+	1    4800 4700
+	1    0    0    -1
+$EndComp
+Wire Wire Line
+	4750 5850 4900 5850
+$Comp
+L power:GND #PWR021
+U 1 1 5A60E862
+P 4750 5850
+F 0 "#PWR021" H 4750 5600 50  0001 C CNN
+F 1 "GND" H 4755 5677 50  0000 C CNN
+F 2 "" H 4750 5850 50  0001 C CNN
+F 3 "" H 4750 5850 50  0001 C CNN
+	1    4750 5850
+	1    0    0    -1
+$EndComp
 $EndSCHEMATC
