File: V0.2-IGBT/PCB/ISO_PSU.sch (KiCad schematic (older format))
At the start: 11 parts, among them Q1 Q_NPN_BCE, U2 MGJ2

Commit message: v2.0 PCB SIGNAL SIDE
Parts:
- removed C9: 1u, Capacitors_SMD:C_0805_HandSoldering, symbol device:C
- removed D1: MMSZ5251B, Diodes_SMD:D_SOD-123, symbol device:D_Zener
- removed Q1: Q_NPN_BCE, TO_SOT_Packages_SMD:SOT-89-3_Handsoldering, symbol device:Q_NPN_BCE
- removed R1: 10k, Resistors_SMD:R_0805_HandSoldering, symbol device:R
- removed R2: 0, Resistors_SMD:R_0805_HandSoldering, symbol device:R
Connections:
- net labels removed: VCC_REG
- wire segments 42 -> 29
Changed lines of the file:
@@
 AR Path="/5A300795/5A301108" Ref="C6"  Part="1"
 AR Path="/5A331F4C/5A301108" Ref="C11"  Part="1"
-F 0 "C11" H 5015 2600 50  0000 L CNN
+F 0 "C6" H 5015 2600 50  0000 L CNN
 F 1 "1u" H 5015 2555 50  0000 L CNN
 F 2 "Capacitors_SMD:C_0805_HandSoldering" H 4938 2450 50  0001 C CNN
@@
 AR Path="/5A300795/5A301151" Ref="C5"  Part="1"
 AR Path="/5A331F4C/5A301151" Ref="C10"  Part="1"
-F 0 "C10" H 4515 2600 50  0000 L CNN
+F 0 "C5" H 4515 2600 50  0000 L CNN
 F 1 "100n" H 4515 2555 50  0000 L CNN
 F 2 "Capacitors_SMD:C_0805_HandSoldering" H 4438 2450 50  0001 C CNN
@@
 AR Path="/5A300795/5A3089F3" Ref="U2"  Part="1"
 AR Path="/5A331F4C/5A3089F3" Ref="U3"  Part="1"
-F 0 "U3" H 5700 3067 50  0000 C CNN
+F 0 "U2" H 5700 3067 50  0000 C CNN
 F 1 "MGJ2" H 5700 2976 50  0000 C CNN
 F 2 "ENNOID:DCDC-Conv_muRata_MGJ2" H 5700 2250 50  0001 C CIN
@@
 AR Path="/5A300795/5A308BE5" Ref="C7"  Part="1"
 AR Path="/5A331F4C/5A308BE5" Ref="C12"  Part="1"
-F 0 "C12" H 6815 2350 50  0000 L CNN
+F 0 "C7" H 6815 2350 50  0000 L CNN
 F 1 "1u" H 6815 2305 50  0000 L CNN
 F 2 "Capacitors_SMD:C_0805_HandSoldering" H 6738 2200 50  0001 C CNN
@@
 AR Path="/5A300795/5A308C45" Ref="C8"  Part="1"
 AR Path="/5A331F4C/5A308C45" Ref="C13"  Part="1"
-F 0 "C13" H 6815 2850 50  0000 L CNN
+F 0 "C8" H 6815 2850 50  0000 L CNN
 F 1 "1u" H 6815 2805 50  0000 L CNN
 F 2 "Capacitors_SMD:C_0805_HandSoldering" H 6738 2700 50  0001 C CNN
@@
 Text HLabel 6700 3200 3    60   Output ~ 0
 -VEE
-$Comp
-L device:R R1
-U 1 1 5A30AA71
-P 7600 2400
-AR Path="/5A300795/5A30AA71" Ref="R1"  Part="1"
-AR Path="/5A331F4C/5A30AA71" Ref="R3"  Part="1"
-F 0 "R3" H 7530 2354 50  0000 R CNN
-F 1 "10k" H 7530 2445 50  0000 R CNN
-F 2 "Resistors_SMD:R_0805_HandSoldering" V 7530 2400 50  0001 C CNN
-F 3 "" H 7600 2400 50  0001 C CNN
-	1    7600 2400
-	-1   0    0    1
-$EndComp
-$Comp
-L device:R R2
-U 1 1 5A30AEBF
-P 8050 2600
-AR Path="/5A300795/5A30AEBF" Ref="R2"  Part="1"
-AR Path="/5A331F4C/5A30AEBF" Ref="R4"  Part="1"
-F 0 "R4" V 8257 2600 50  0000 C CNN
-F 1 "0" V 8166 2600 50  0000 C CNN
-F 2 "Resistors_SMD:R_0805_HandSoldering" V 7980 2600 50  0001 C CNN
-F 3 "" H 8050 2600 50  0001 C CNN
-	1    8050 2600
-	0    -1   -1   0
-$EndComp
-$Comp
-L device:C C9
-U 1 1 5A30AF37
-P 8250 2950
-AR Path="/5A300795/5A30AF37" Ref="C9"  Part="1"
-AR Path="/5A331F4C/5A30AF37" Ref="C14"  Part="1"
-F 0 "C14" H 8365 2950 50  0000 L CNN
-F 1 "1u" H 8365 2905 50  0000 L CNN
-F 2 "Capacitors_SMD:C_0805_HandSoldering" H 8288 2800 50  0001 C CNN
-F 3 "" H 8250 2950 50  0001 C CNN
-	1    8250 2950
-	1    0    0    -1
-$EndComp
-Wire Wire Line
-	8200 2600 8300 2600
-Wire Wire Line
-	8600 2800 8250 2800
-Wire Wire Line
-	7900 2600 7600 2600
 Connection ~ 6700 3100
 Wire Wire Line
@@
 Wire Wire Line
 	6700 3100 6700 3200
-Wire Wire Line
-	8600 2400 8600 2200
-Wire Wire Line
-	7600 2600 7600 2550
-Wire Wire Line
-	7600 2250 7600 2200
-Connection ~ 7600 2200
-Wire Wire Line
-	7600 2200 8600 2200
-Text HLabel 8600 3150 3    60   Output ~ 0
-VCC_REG
-Wire Wire Line
-	8600 3150 8600 2800
 Text HLabel 6950 2600 2    60   Output ~ 0
 PHASE
 Wire Wire Line
-	6700 2200 7600 2200
-Wire Wire Line
-	6700 3100 7600 3100
-Wire Wire Line
 	6950 2600 6700 2600
-$Comp
-L device:D_Zener D1
-U 1 1 5A310D6B
-P 7600 2850
-AR Path="/5A300795/5A310D6B" Ref="D1"  Part="1"
-AR Path="/5A331F4C/5A310D6B" Ref="D2"  Part="1"
-F 0 "D2" V 7554 2929 50  0000 L CNN
-F 1 "MMSZ5251B" V 7645 2929 50  0000 L CNN
-F 2 "Diodes_SMD:D_SOD-123" H 7600 2850 50  0001 C CNN
-F 3 "https://en.wikipedia.org/wiki/Zener_diode" H 7600 2850 50  0001 C CNN
-	1    7600 2850
-	0    1    1    0
-$EndComp
-Wire Wire Line
-	7600 2700 7600 2600
-Connection ~ 7600 2600
-Wire Wire Line
-	7600 3000 7600 3100
-Connection ~ 7600 3100
-Wire Wire Line
-	7600 3100 8250 3100
 $Comp
 L power:GND #PWR036
@@
 AR Path="/5A300795/5A57221A" Ref="#PWR036"  Part="1"
 AR Path="/5A331F4C/5A57221A" Ref="#PWR037"  Part="1"
-F 0 "#PWR037" H 3600 2450 50  0001 C CNN
+F 0 "#PWR036" H 3600 2450 50  0001 C CNN
 F 1 "GND" H 3605 2527 50  0000 C CNN
 F 2 "" H 3600 2700 50  0001 C CNN
@@
 AR Path="/5A331F4C/5A415966" Ref="#PWR011"  Part="1"
 AR Path="/5A300795/5A415966" Ref="#PWR010"  Part="1"
-F 0 "#PWR011" H 3600 2350 50  0001 C CNN
+F 0 "#PWR010" H 3600 2350 50  0001 C CNN
 F 1 "+24V" H 3615 2673 50  0000 C CNN
 F 2 "" H 3600 2500 50  0001 C CNN
@@
 $EndComp
 $Comp
-L device:Q_NPN_BCE Q1
-U 1 1 5A34237B
-P 8500 2600
-AR Path="/5A331F4C/5A34237B" Ref="Q1"  Part="1"
-AR Path="/5A300795/5A34237B" Ref="Q2"  Part="1"
-F 0 "Q1" H 8691 2646 50  0000 L CNN
-F 1 "Q_NPN_BCE" H 8691 2555 50  0000 L CNN
-F 2 "TO_SOT_Packages_SMD:SOT-89-3_Handsoldering" H 8700 2700 50  0001 C CNN
-F 3 "" H 8500 2600 50  0001 C CNN
-	1    8500 2600
-	1    0    0    -1
-$EndComp
-Connection ~ 8600 2800
-$Comp
 L ENNOID:ACM4520 FL2
 U 1 1 5A376789
@@
 AR Path="/5A331F4C/5A376789" Ref="FL2"  Part="1"
 AR Path="/5A300795/5A376789" Ref="FL1"  Part="1"
-F 0 "FL2" H 3850 2878 50  0000 C CNN
+F 0 "FL1" H 3850 2878 50  0000 C CNN
 F 1 "ACM4520" H 3850 2787 50  0000 C CNN
 F 2 "ENNOID:ACM4520" H 3850 2787 50  0001 C CNN

Commit message: Schematics update
Parts:
- C5: Mfg.# (none) -> C0805C104J5RACAUTO
- C6, C7, C8: Mfg.# (none) -> UMK212BJ105MG-T
- FL2: Mfg. # (none) -> ACM4520-142-2P-TL000
- U2: Mfg. # (none) -> MGJ2D241509SC
Connections:
- net labels added: COM
- net labels removed: +24V, PHASE
Changed lines of the file:
@@
 $Descr A4 11693 8268
 encoding utf-8
-Sheet 4 6
+Sheet 2 6
 Title ""
 Date ""
@@
 AR Path="/5A300795/5A301108" Ref="C6"  Part="1"
 AR Path="/5A331F4C/5A301108" Ref="C11"  Part="1"
-F 0 "C11" H 5015 2600 50  0000 L CNN
+F 0 "C6" H 5015 2600 50  0000 L CNN
 F 1 "1u" H 5015 2555 50  0000 L CNN
 F 2 "Capacitors_SMD:C_0805_HandSoldering" H 4938 2450 50  0001 C CNN
-F 3 "" H 4900 2600 50  0001 C CNN
+F 3 "http://www.mouser.com/ds/2/396/mlcc_all_e-1149778.pdf" H 4900 2600 50  0001 C CNN
+F 4 "UMK212BJ105MG-T " H 4900 2600 50  0001 C CNN "Mfg.#"
 	1    4900 2600
 	1    0    0    -1
@@
 AR Path="/5A300795/5A301151" Ref="C5"  Part="1"
 AR Path="/5A331F4C/5A301151" Ref="C10"  Part="1"
-F 0 "C10" H 4515 2600 50  0000 L CNN
+F 0 "C5" H 4515 2600 50  0000 L CNN
 F 1 "100n" H 4515 2555 50  0000 L CNN
 F 2 "Capacitors_SMD:C_0805_HandSoldering" H 4438 2450 50  0001 C CNN
-F 3 "" H 4400 2600 50  0001 C CNN
+F 3 "http://www.mouser.com/ds/2/212/KEM_C1023_X7R_AUTO_SMD-1093309.pdf" H 4400 2600 50  0001 C CNN
+F 4 "C0805C104J5RACAUTO " H 4400 2600 50  0001 C CNN "Mfg.#"
 	1    4400 2600
 	1    0    0    -1
@@
 AR Path="/5A300795/5A3089F3" Ref="U2"  Part="1"
 AR Path="/5A331F4C/5A3089F3" Ref="U3"  Part="1"
-F 0 "U3" H 5700 3067 50  0000 C CNN
+F 0 "U2" H 5700 3067 50  0000 C CNN
 F 1 "MGJ2" H 5700 2976 50  0000 C CNN
 F 2 "ENNOID:DCDC-Conv_muRata_MGJ2" H 5700 2250 50  0001 C CIN
 F 3 "https://power.murata.com/data/power/ncl/kdc_mgj2.pdf" H 5700 2600 50  0001 C CNN
+F 4 "MGJ2D241509SC " H 5700 2600 50  0001 C CNN "Mfg. #"
 	1    5700 2600
 	1    0    0    -1
@@
 AR Path="/5A300795/5A308BE5" Ref="C7"  Part="1"
 AR Path="/5A331F4C/5A308BE5" Ref="C12"  Part="1"
-F 0 "C12" H 6815 2350 50  0000 L CNN
+F 0 "C7" H 6815 2350 50  0000 L CNN
 F 1 "1u" H 6815 2305 50  0000 L CNN
 F 2 "Capacitors_SMD:C_0805_HandSoldering" H 6738 2200 50  0001 C CNN
-F 3 "" H 6700 2350 50  0001 C CNN
+F 3 "http://www.mouser.com/ds/2/396/mlcc_all_e-1149778.pdf" H 6700 2350 50  0001 C CNN
+F 4 "UMK212BJ105MG-T " H 6700 2350 50  0001 C CNN "Mfg.#"
 	1    6700 2350
 	1    0    0    -1
@@
 AR Path="/5A300795/5A308C45" Ref="C8"  Part="1"
 AR Path="/5A331F4C/5A308C45" Ref="C13"  Part="1"
-F 0 "C13" H 6815 2850 50  0000 L CNN
+F 0 "C8" H 6815 2850 50  0000 L CNN
 F 1 "1u" H 6815 2805 50  0000 L CNN
 F 2 "Capacitors_SMD:C_0805_HandSoldering" H 6738 2700 50  0001 C CNN
-F 3 "" H 6700 2850 50  0001 C CNN
+F 3 "http://www.mouser.com/ds/2/396/mlcc_all_e-1149778.pdf" H 6700 2850 50  0001 C CNN
+F 4 "UMK212BJ105MG-T " H 6700 2850 50  0001 C CNN "Mfg.#"
 	1    6700 2850
 	1    0    0    -1
@@
 	6700 3100 6700 3200
 Text HLabel 6950 2600 2    60   Output ~ 0
-PHASE
+COM
 Wire Wire Line
 	6950 2600 6700 2600
-$Comp
-L power:GND #PWR036
-U 1 1 5A57221A
-P 3600 2700
-AR Path="/5A300795/5A57221A" Ref="#PWR036"  Part="1"
-AR Path="/5A331F4C/5A57221A" Ref="#PWR037"  Part="1"
-F 0 "#PWR037" H 3600 2450 50  0001 C CNN
-F 1 "GND" H 3605 2527 50  0000 C CNN
-F 2 "" H 3600 2700 50  0001 C CNN
-F 3 "" H 3600 2700 50  0001 C CNN
-	1    3600 2700
-	1    0    0    -1
-$EndComp
-Connection ~ 3600 2700
 Wire Wire Line
 	3600 2700 3500 2700
-$Comp
-L power:+24V #PWR011
-U 1 1 5A415966
-P 3600 2500
-AR Path="/5A331F4C/5A415966" Ref="#PWR011"  Part="1"
-AR Path="/5A300795/5A415966" Ref="#PWR010"  Part="1"
-F 0 "#PWR011" H 3600 2350 50  0001 C CNN
-F 1 "+24V" H 3615 2673 50  0000 C CNN
-F 2 "" H 3600 2500 50  0001 C CNN
-F 3 "" H 3600 2500 50  0001 C CNN
-	1    3600 2500
-	1    0    0    -1
-$EndComp
 $Comp
 L ENNOID:ACM4520 FL2
@@
 AR Path="/5A331F4C/5A376789" Ref="FL2"  Part="1"
 AR Path="/5A300795/5A376789" Ref="FL1"  Part="1"
-F 0 "FL2" H 3850 2878 50  0000 C CNN
+F 0 "FL1" H 3850 2878 50  0000 C CNN
 F 1 "ACM4520" H 3850 2787 50  0000 C CNN
 F 2 "ENNOID:ACM4520" H 3850 2787 50  0001 C CNN
-F 3 "" V 3850 2640 50  0000 C CNN
+F 3 "http://www.mouser.com/ds/2/400/mf_commercial_power_acm4520_en-837180.pdf" V 3850 2640 50  0001 C CNN
+F 4 "ACM4520-142-2P-TL000" H 3850 2600 50  0001 C CNN "Mfg. #"
 	1    3850 2600
 	1    0    0    -1
@@
 Wire Wire Line
 	3600 2500 3500 2500
-Connection ~ 3600 2500
 $EndSCHEMATC

Commit message: V0.2 BOM and schematics updated
Connections:
- wire segments 29 -> 27
Changed lines of the file:
@@
 	4400 2750 4900 2750
-Wire Wire Line
-	3650 2700 3600 2700
 Wire Wire Line
 	4050 2500 4250 2500
@@
 Wire Wire Line
 	6950 2600 6700 2600
-Wire Wire Line
-	3600 2700 3500 2700
 $Comp
 L ENNOID:ACM4520 FL2
@@
 $EndComp
 Wire Wire Line
-	3650 2500 3600 2500
+	3500 2700 3650 2700
 Wire Wire Line
-	3600 2500 3500 2500
+	3500 2500 3650 2500
 $EndSCHEMATC

Commit message: Maintenance update
Parts:
- C5, C6, C7, C8: symbol device:C -> ENNOID-Dual-Gate-Driver-rescue:C-device
Changed lines of the file:
@@
 $Descr A4 11693 8268
 encoding utf-8
-Sheet 2 6
+Sheet 4 6
 Title ""
 Date ""
@@
 GND
 $Comp
-L device:C C6
+L ENNOID-Dual-Gate-Driver-rescue:C-device C6
 U 1 1 5A301108
 P 4900 2600
@@
 $EndComp
 $Comp
-L device:C C5
+L ENNOID-Dual-Gate-Driver-rescue:C-device C5
 U 1 1 5A301151
 P 4400 2600
@@
 Connection ~ 4900 2750
 $Comp
-L device:C C7
+L ENNOID-Dual-Gate-Driver-rescue:C-device C7
 U 1 1 5A308BE5
 P 6700 2350
@@
 $EndComp
 $Comp
-L device:C C8
+L ENNOID-Dual-Gate-Driver-rescue:C-device C8
 U 1 1 5A308C45
 P 6700 2850
