File: V0.2-IGBT/PCB/V_PHASE.sch (KiCad schematic (older format))
At the start: 11 parts, among them U8 AMC1301

Commit message: V0.2 completed
Parts:
- added C9: 10u, Capacitors_SMD:C_0805_HandSoldering, symbol device:C
- D9: value 5V -> 5V
- R28: value 200 -> 800
Connections:
- wire segments 45 -> 49
Changed lines of the file:
@@
 L device:C C37
 U 1 1 5A30FC69
-P 5100 3300
-F 0 "C37" H 5215 3346 50  0000 L CNN
-F 1 "100n" H 5215 3255 50  0000 L CNN
-F 2 "Capacitors_SMD:C_0805_HandSoldering" H 5138 3150 50  0001 C CNN
-F 3 "" H 5100 3300 50  0001 C CNN
-	1    5100 3300
+P 5150 3300
+F 0 "C37" H 5265 3346 50  0000 L CNN
+F 1 "100n" H 5265 3255 50  0000 L CNN
+F 2 "Capacitors_SMD:C_0805_HandSoldering" H 5188 3150 50  0001 C CNN
+F 3 "" H 5150 3300 50  0001 C CNN
+	1    5150 3300
 	1    0    0    -1
 $EndComp
@@
 $EndComp
 Wire Wire Line
-	5500 3550 5100 3550
-Wire Wire Line
-	5100 3550 5100 3450
-Wire Wire Line
-	5500 3000 5100 3000
-Wire Wire Line
-	5100 3000 5100 3150
+	5500 3550 5150 3550
+Wire Wire Line
+	5150 3550 5150 3450
+Wire Wire Line
+	5500 3000 5150 3000
+Wire Wire Line
+	5150 3000 5150 3150
 Wire Wire Line
 	5500 3000 5500 3450
@@
 P 4200 3000
 F 0 "R28" V 3993 3000 50  0000 C CNN
-F 1 "200" V 4084 3000 50  0000 C CNN
+F 1 "800" V 4084 3000 50  0000 C CNN
 F 2 "Resistors_SMD:R_0805_HandSoldering" V 4130 3000 50  0001 C CNN
 F 3 "" H 4200 3000 50  0001 C CNN
@@
 	4050 3750 3950 3750
 Wire Wire Line
-	5100 3000 4550 3000
-Connection ~ 5100 3000
+	5150 3000 4800 3000
+Connection ~ 5150 3000
 $Comp
 L device:D_Zener D9
 U 1 1 5A3109F4
-P 4550 3250
-F 0 "D9" V 4504 3329 50  0000 L CNN
-F 1 "5V" V 4595 3329 50  0000 L CNN
-F 2 "Diodes_SMD:D_SOT-23_ANK" H 4550 3250 50  0001 C CNN
-F 3 "https://en.wikipedia.org/wiki/Zener_diode" H 4550 3250 50  0001 C CNN
-	1    4550 3250
-	0    1    1    0
-$EndComp
-Wire Wire Line
-	4550 3100 4550 3000
-Connection ~ 4550 3000
-Wire Wire Line
-	4550 3000 4350 3000
-Wire Wire Line
-	5100 3550 4550 3550
-Wire Wire Line
-	4550 3550 4550 3450
-Connection ~ 5100 3550
-Connection ~ 4550 3450
-Wire Wire Line
-	4550 3450 4550 3400
+P 4500 3250
+F 0 "D9" V 4454 3329 50  0000 L CNN
+F 1 "5V " V 4545 3329 50  0000 L CNN
+F 2 "Diodes_SMD:D_SOT-23_ANK" H 4500 3250 50  0001 C CNN
+F 3 "https://en.wikipedia.org/wiki/Zener_diode" H 4500 3250 50  0001 C CNN
+	1    4500 3250
+	0    1    1    0
+$EndComp
+Wire Wire Line
+	4500 3100 4500 3000
+Connection ~ 4500 3000
+Wire Wire Line
+	4500 3000 4350 3000
+Wire Wire Line
+	5150 3550 4800 3550
+Wire Wire Line
+	4500 3550 4500 3450
+Connection ~ 5150 3550
+Connection ~ 4500 3450
+Wire Wire Line
+	4500 3450 4500 3400
 $Comp
 L device:C C39
@@
 	2950 3450 2950 4200
 Wire Wire Line
-	2950 3450 4550 3450
+	2950 3450 4500 3450
 Wire Wire Line
 	2550 4200 2950 4200
@@
 Wire Wire Line
 	4050 3000 3800 3000
+$Comp
+L device:C C9
+U 1 1 5A4DF1BA
+P 4800 3300
+F 0 "C9" H 4915 3346 50  0000 L CNN
+F 1 "10u" H 4915 3255 50  0000 L CNN
+F 2 "Capacitors_SMD:C_0805_HandSoldering" H 4838 3150 50  0001 C CNN
+F 3 "" H 4800 3300 50  0001 C CNN
+	1    4800 3300
+	1    0    0    -1
+$EndComp
+Wire Wire Line
+	4800 3150 4800 3000
+Connection ~ 4800 3000
+Wire Wire Line
+	4800 3000 4500 3000
+Wire Wire Line
+	4800 3450 4800 3550
+Connection ~ 4800 3550
+Wire Wire Line
+	4800 3550 4500 3550
 $EndSCHEMATC

Commit message: VBUS sensor & voltage sense circuit changes
Parts:
- R27, R29: footprint Resistors_SMD:R_0805_HandSoldering -> Resistors_SMD:R_1206
Changed lines of the file:
@@
 F 0 "R27" V 3593 3750 50  0000 C CNN
 F 1 "1M" V 3684 3750 50  0000 C CNN
-F 2 "Resistors_SMD:R_0805_HandSoldering" V 3730 3750 50  0001 C CNN
+F 2 "Resistors_SMD:R_1206" V 3730 3750 50  0001 C CNN
 F 3 "" H 3800 3750 50  0001 C CNN
 	1    3800 3750
@@
 F 0 "R29" V 3993 3750 50  0000 C CNN
 F 1 "1M" V 4084 3750 50  0000 C CNN
-F 2 "Resistors_SMD:R_0805_HandSoldering" V 4130 3750 50  0001 C CNN
+F 2 "Resistors_SMD:R_1206" V 4130 3750 50  0001 C CNN
 F 3 "" H 4200 3750 50  0001 C CNN
 	1    4200 3750

Commit message: Schematics update
Parts:
- C37, C39: Mfg.# (none) -> C0805C104J5RACAUTO
- C9: Mfg.# (none) -> UMK325BJ106KMHP
Connections:
- wire segments 49 -> 46
Changed lines of the file:
@@
 F 1 "100n" H 5265 3255 50  0000 L CNN
 F 2 "Capacitors_SMD:C_0805_HandSoldering" H 5188 3150 50  0001 C CNN
-F 3 "" H 5150 3300 50  0001 C CNN
+F 3 "http://www.mouser.com/ds/2/212/KEM_C1023_X7R_AUTO_SMD-1093309.pdf" H 5150 3300 50  0001 C CNN
+F 4 "C0805C104J5RACAUTO" H 5150 3300 50  0001 C CNN "Mfg.#"
 	1    5150 3300
 	1    0    0    -1
@@
 F 1 "100n" H 6865 3255 50  0000 L CNN
 F 2 "Capacitors_SMD:C_0805_HandSoldering" H 6788 3150 50  0001 C CNN
-F 3 "" H 6750 3300 50  0001 C CNN
+F 3 "http://www.mouser.com/ds/2/212/KEM_C1023_X7R_AUTO_SMD-1093309.pdf" H 6750 3300 50  0001 C CNN
+F 4 "C0805C104J5RACAUTO" H 6750 3300 50  0001 C CNN "Mfg.#"
 	1    6750 3300
 	1    0    0    -1
@@
 Wire Wire Line
 	6750 3550 6300 3550
-Wire Wire Line
-	7600 3550 7200 3550
 Connection ~ 7200 3050
 Connection ~ 7200 3550
@@
 Text HLabel 7950 3050 2    60   Input ~ 0
 +5V
-Wire Wire Line
-	7200 3050 7700 3050
-$Comp
-L power:+5V #PWR021
-U 1 1 5A31BC2D
-P 7700 3000
-F 0 "#PWR021" H 7700 2850 50  0001 C CNN
-F 1 "+5V" H 7715 3173 50  0000 C CNN
-F 2 "" H 7700 3000 50  0001 C CNN
-F 3 "" H 7700 3000 50  0001 C CNN
-	1    7700 3000
-	1    0    0    -1
-$EndComp
-Wire Wire Line
-	7700 3000 7700 3050
-Connection ~ 7700 3050
-Wire Wire Line
-	7700 3050 7950 3050
 Text HLabel 6650 3750 2    60   Output ~ 0
 Vout+
 Text HLabel 6650 3850 2    60   Output ~ 0
 Vout-
-$Comp
-L power:GND #PWR035
-U 1 1 5A34B574
-P 7600 3550
-F 0 "#PWR035" H 7600 3300 50  0001 C CNN
-F 1 "GND" H 7605 3377 50  0000 C CNN
-F 2 "" H 7600 3550 50  0001 C CNN
-F 3 "" H 7600 3550 50  0001 C CNN
-	1    7600 3550
-	1    0    0    -1
-$EndComp
 Text HLabel 7700 3550 2    60   Input ~ 0
 GND
-Wire Wire Line
-	7600 3550 7700 3550
-Connection ~ 7600 3550
 Text HLabel 3800 3000 0    60   Input ~ 0
 +VCC
@@
 F 1 "10u" H 4915 3255 50  0000 L CNN
 F 2 "Capacitors_SMD:C_0805_HandSoldering" H 4838 3150 50  0001 C CNN
-F 3 "" H 4800 3300 50  0001 C CNN
+F 3 "http://www.mouser.com/ds/2/396/mlcc11_hq_e-541564.pdf" H 4800 3300 50  0001 C CNN
+F 4 "UMK325BJ106KMHP" H 4800 3300 50  0001 C CNN "Mfg.#"
 	1    4800 3300
 	1    0    0    -1
@@
 Wire Wire Line
 	4800 3550 4500 3550
+Wire Wire Line
+	7200 3550 7700 3550
+Wire Wire Line
+	7200 3050 7950 3050
 $EndSCHEMATC

Commit message: V0.2 BOM and schematics updated
Parts:
- C38: Mfg.# (none) -> C0805C331J5GACTU
- C40: Mfg.# (none) -> UMK212ABJ225KG-T
- D9: Mfg.# (none) -> BZX84-A5V1,215
- R27, R29: Mfg.# (none) -> CHV1206-FX-1004ELF
- R28: Mfg.# (none) -> RK73H2ATTDD8060F
- R30: Mfg.# (none) -> RC0805JR-071KL
- U8: Mfg.# (none) -> AMC1301QDWVRQ1
Changed lines of the file:
@@
 F 2 "ENNOID:SSO-8_6.8x5.9mm_Pitch1.27mm_Clearance8mm" H 5900 3300 50  0001 C CIN
 F 3 "http://www.ti.com/lit/ds/symlink/amc1301.pdf" H 5900 3650 50  0001 C CNN
+F 4 "AMC1301QDWVRQ1" H 5900 3650 50  0001 C CNN "Mfg.#"
 	1    5900 3650
 	1    0    0    -1
@@
 F 1 "330p" H 5265 3905 50  0000 L CNN
 F 2 "Capacitors_SMD:C_0805_HandSoldering" H 5188 3800 50  0001 C CNN
-F 3 "" H 5150 3950 50  0001 C CNN
+F 3 "http://www.mouser.com/ds/2/212/KEM_C1003_C0G_SMD-1101588.pdf" H 5150 3950 50  0001 C CNN
+F 4 "C0805C331J5GACTU " H 5150 3950 50  0001 C CNN "Mfg.#"
 	1    5150 3950
 	1    0    0    -1
@@
 F 1 "800" V 4084 3000 50  0000 C CNN
 F 2 "Resistors_SMD:R_0805_HandSoldering" V 4130 3000 50  0001 C CNN
-F 3 "" H 4200 3000 50  0001 C CNN
+F 3 "http://www.mouser.com/ds/2/219/RK73H-5715.pdf" H 4200 3000 50  0001 C CNN
+F 4 "RK73H2ATTDD8060F" V 4200 3000 50  0001 C CNN "Mfg.#"
 	1    4200 3000
 	0    1    1    0
@@
 F 1 "1M" V 3684 3750 50  0000 C CNN
 F 2 "Resistors_SMD:R_1206" V 3730 3750 50  0001 C CNN
-F 3 "" H 3800 3750 50  0001 C CNN
+F 3 "https://ca.mouser.com/ProductDetail/Bourns/CHV1206-FX-1004ELF/?qs=%2fha2pyFadugSy6dYV9l6fxbWdTbmdsWSmCbzMVjyPUH0nr4JhkrW7wEz2YoAFni8" H 3800 3750 50  0001 C CNN
+F 4 "CHV1206-FX-1004ELF " V 3800 3750 50  0001 C CNN "Mfg.#"
 	1    3800 3750
 	0    1    1    0
@@
 F 1 "1M" V 4084 3750 50  0000 C CNN
 F 2 "Resistors_SMD:R_1206" V 4130 3750 50  0001 C CNN
-F 3 "" H 4200 3750 50  0001 C CNN
+F 3 "https://ca.mouser.com/ProductDetail/Bourns/CHV1206-FX-1004ELF/?qs=%2fha2pyFadugSy6dYV9l6fxbWdTbmdsWSmCbzMVjyPUH0nr4JhkrW7wEz2YoAFni8" H 4200 3750 50  0001 C CNN
+F 4 "CHV1206-FX-1004ELF " V 4200 3750 50  0001 C CNN "Mfg.#"
 	1    4200 3750
 	0    1    1    0
@@
 F 1 "1k" H 4430 3995 50  0000 R CNN
 F 2 "Resistors_SMD:R_0805_HandSoldering" V 4430 3950 50  0001 C CNN
-F 3 "" H 4500 3950 50  0001 C CNN
+F 3 "http://www.mouser.com/ds/2/447/Yageo_08112016_RC0805-1211991.pdf" H 4500 3950 50  0001 C CNN
+F 4 "RC0805JR-071KL" H 4500 3950 50  0001 C CNN "Mfg.#"
 	1    4500 3950
 	-1   0    0    1
@@
 F 1 "5V " V 4545 3329 50  0000 L CNN
 F 2 "Diodes_SMD:D_SOT-23_ANK" H 4500 3250 50  0001 C CNN
-F 3 "https://en.wikipedia.org/wiki/Zener_diode" H 4500 3250 50  0001 C CNN
+F 3 "http://www.mouser.com/ds/2/302/BZX84_SERIES-114620.pdf" H 4500 3250 50  0001 C CNN
+F 4 "BZX84-A5V1,215 " V 4500 3250 50  0001 C CNN "Mfg.#"
 	1    4500 3250
 	0    1    1    0
@@
 F 1 "2.2u" H 7315 3255 50  0000 L CNN
 F 2 "Capacitors_SMD:C_0805_HandSoldering" H 7238 3150 50  0001 C CNN
-F 3 "" H 7200 3300 50  0001 C CNN
+F 3 "http://www.mouser.com/ds/2/396/mlcc11_hq_e-541564.pdf" H 7200 3300 50  0001 C CNN
+F 4 "UMK212ABJ225KG-T " H 7200 3300 50  0001 C CNN "Mfg.#"
 	1    7200 3300
 	1    0    0    -1

Commit message: V0.2 pcb changes
Parts:
- added R17: 10, Resistors_SMD:R_0805_HandSoldering, symbol device:R
Connections:
- wire segments 46 -> 45
Changed lines of the file:
@@
 	4500 3750 4350 3750
-Wire Wire Line
-	4500 3750 5150 3750
-Connection ~ 4500 3750
-Connection ~ 5150 3750
 Wire Wire Line
 	4050 3750 3950 3750
@@
 Wire Wire Line
 	4500 3000 4350 3000
-Wire Wire Line
-	5150 3550 4800 3550
-Wire Wire Line
-	4500 3550 4500 3450
-Connection ~ 5150 3550
 Connection ~ 4500 3450
 Wire Wire Line
@@
 	4800 3000 4500 3000
 Wire Wire Line
-	4800 3450 4800 3550
-Connection ~ 4800 3550
-Wire Wire Line
-	4800 3550 4500 3550
+	4800 3450 4500 3450
 Wire Wire Line
 	7200 3550 7700 3550
 Wire Wire Line
 	7200 3050 7950 3050
+$Comp
+L device:R R17
+U 1 1 5A606745
+P 4800 3750
+F 0 "R17" V 5007 3750 50  0000 C CNN
+F 1 "10" V 4916 3750 50  0000 C CNN
+F 2 "Resistors_SMD:R_0805_HandSoldering" V 4730 3750 50  0001 C CNN
+F 3 "" H 4800 3750 50  0001 C CNN
+	1    4800 3750
+	0    -1   -1   0
+$EndComp
+Connection ~ 4500 3750
+Wire Wire Line
+	4500 3750 4650 3750
+Connection ~ 5150 3750
+Wire Wire Line
+	4950 3750 5150 3750
+Wire Wire Line
+	4800 3450 5150 3450
+Connection ~ 4800 3450
+Connection ~ 5150 3450
 $EndSCHEMATC

Commit message: Maintenance update
Parts:
- removed R31: 1k, Resistors_SMD:R_0805_HandSoldering, symbol device:R
- C37, C38, C39, C40, C9: symbol device:C -> ENNOID-Dual-Gate-Driver-rescue:C-device
- D9: symbol device:D_Zener -> ENNOID-Dual-Gate-Driver-rescue:D_Zener-device
- R17, R27, R28, R29, R30: symbol device:R -> ENNOID-Dual-Gate-Driver-rescue:R-device
Connections:
- wire segments 45 -> 44
Changed lines of the file:
@@
 $EndComp
 $Comp
-L device:C C37
+L ENNOID-Dual-Gate-Driver-rescue:C-device C37
 U 1 1 5A30FC69
 P 5150 3300
@@
 $EndComp
 $Comp
-L device:C C38
+L ENNOID-Dual-Gate-Driver-rescue:C-device C38
 U 1 1 5A30FE1D
 P 5150 3950
@@
 	5150 4200 5150 4100
 $Comp
-L device:R R28
+L ENNOID-Dual-Gate-Driver-rescue:R-device R28
 U 1 1 5A30FF82
 P 4200 3000
@@
 $EndComp
 $Comp
-L device:R R27
+L ENNOID-Dual-Gate-Driver-rescue:R-device R27
 U 1 1 5A30FFC5
 P 3800 3750
@@
 $EndComp
 $Comp
-L device:R R29
+L ENNOID-Dual-Gate-Driver-rescue:R-device R29
 U 1 1 5A30FFF9
 P 4200 3750
@@
 $EndComp
 $Comp
-L device:R R30
+L ENNOID-Dual-Gate-Driver-rescue:R-device R30
 U 1 1 5A310023
 P 4500 3950
@@
 	-1   0    0    1
 $EndComp
-$Comp
-L device:R R31
-U 1 1 5A3100D1
-P 4800 4200
-F 0 "R31" V 5007 4200 50  0000 C CNN
-F 1 "1k" V 4916 4200 50  0000 C CNN
-F 2 "Resistors_SMD:R_0805_HandSoldering" V 4730 4200 50  0001 C CNN
-F 3 "" H 4800 4200 50  0001 C CNN
-	1    4800 4200
-	0    -1   -1   0
-$EndComp
-Wire Wire Line
-	5150 4200 4950 4200
-Wire Wire Line
-	4650 4200 4500 4200
 Wire Wire Line
 	4500 4200 4500 4100
@@
 Connection ~ 5150 3000
 $Comp
-L device:D_Zener D9
+L ENNOID-Dual-Gate-Driver-rescue:D_Zener-device D9
 U 1 1 5A3109F4
 P 4500 3250
@@
 	4500 3450 4500 3400
 $Comp
-L device:C C39
+L ENNOID-Dual-Gate-Driver-rescue:C-device C39
 U 1 1 5A311419
 P 6750 3300
@@
 $EndComp
 $Comp
-L device:C C40
+L ENNOID-Dual-Gate-Driver-rescue:C-device C40
 U 1 1 5A31145B
 P 7200 3300
@@
 	4050 3000 3800 3000
 $Comp
-L device:C C9
+L ENNOID-Dual-Gate-Driver-rescue:C-device C9
 U 1 1 5A4DF1BA
 P 4800 3300
@@
 	7200 3050 7950 3050
 $Comp
-L device:R R17
+L ENNOID-Dual-Gate-Driver-rescue:R-device R17
 U 1 1 5A606745
 P 4800 3750
@@
 Connection ~ 4800 3450
 Connection ~ 5150 3450
+Wire Wire Line
+	4500 4200 5150 4200
 $EndSCHEMATC
