File: V0.3/PCB/ENNOID Dual Gate Driver.kicad_pcb (KiCad board)
At the start: 2 copper layers, 60 x 98 mm, 142 parts, among them J1 Conn_02x08_Odd_Even, J2 Current, J3 TEMP, J4 PHASE, J5 Collector, J6 Gate_H, J7 G_L, J8 E, Q3 MJD3055T4G, Q4 MJD2955T4G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

Commit message: V0.3 started
Parts:
- removed D16, D22: PMEG4010, Diodes_SMD:D_SOD-323_HandSoldering
Connections:
- J1 pad 7: Net-(J1-Pad7) -> (no net)
- J1 pad 8: Net-(J1-Pad8) -> (no net)
- U4 pad 7: Net-(U4-Pad7) -> (no net)
- U5 pad 7: Net-(U5-Pad7) -> (no net)
Routing:
- net /GD_HIGH/+VCC: track 64.3 -> 58.5 mm
- net /GD_LOW/+VCC: track 62.8 -> 57.3 mm
- net /GD_HIGH/G: track 5.27 -> 3.78 mm
- net /GD_LOW/G: track 14.9 -> 13.5 mm
Changed lines of the file:
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@@
     (thickness 1.6)
     (drawings 31)
-    (tracks 946)
+    (tracks 938)
     (zones 0)
-    (modules 142)
-    (nets 63)
+    (modules 140)
+    (nets 59)
   )
   (page A4)
@@
   (net 57 "Net-(Q3-Pad1)")
   (net 58 "Net-(Q5-Pad1)")
-  (net 59 "Net-(J1-Pad8)")
-  (net 60 "Net-(J1-Pad7)")
-  (net 61 "Net-(U4-Pad7)")
-  (net 62 "Net-(U5-Pad7)")
   (net_class Default "This is the default net class."
     (clearance 0.2)
@@
     (add_net "Net-(D7-Pad2)")
     (add_net "Net-(F1-Pad1)")
-    (add_net "Net-(J1-Pad7)")
-    (add_net "Net-(J1-Pad8)")
     (add_net "Net-(Q3-Pad1)")
     (add_net "Net-(Q3-Pad3)")
@@
     (add_net "Net-(R26-Pad2)")
     (add_net "Net-(R27-Pad1)")
-    (add_net "Net-(U4-Pad7)")
-    (add_net "Net-(U5-Pad7)")
     (add_net PHASE)
     (add_net PWM_H)
@@
     (pad 9 thru_hole circle (at 10.16 0) (size 1.7 1.7) (drill 1) (layers *.Cu *.Mask)
       (net 22 TEMP))
-    (pad 8 thru_hole circle (at 7.62 -2.54) (size 1.7 1.7) (drill 1) (layers *.Cu *.Mask)
-      (net 59 "Net-(J1-Pad8)"))
-    (pad 7 thru_hole circle (at 7.62 0) (size 1.7 1.7) (drill 1) (layers *.Cu *.Mask)
-      (net 60 "Net-(J1-Pad7)"))
+    (pad 8 thru_hole circle (at 7.62 -2.54) (size 1.7 1.7) (drill 1) (layers *.Cu *.Mask))
+    (pad 7 thru_hole circle (at 7.62 0) (size 1.7 1.7) (drill 1) (layers *.Cu *.Mask))
     (pad 6 thru_hole circle (at 5.08 -2.54) (size 1.7 1.7) (drill 1) (layers *.Cu *.Mask)
       (net 34 FLT))
@@
     (pad 8 smd rect (at -4.65 4.445 270) (size 1.5 0.6) (layers F.Cu F.Paste F.Mask)
       (net 7 /GD_HIGH/-VEE))
-    (pad 7 smd rect (at -4.65 3.175 270) (size 1.5 0.6) (layers F.Cu F.Paste F.Mask)
-      (net 61 "Net-(U4-Pad7)"))
+    (pad 7 smd rect (at -4.65 3.175 270) (size 1.5 0.6) (layers F.Cu F.Paste F.Mask))
     (pad 6 smd rect (at -4.65 1.905 270) (size 1.5 0.6) (layers F.Cu F.Paste F.Mask)
       (net 46 "Net-(R11-Pad2)"))
@@
     (pad 8 smd rect (at -4.65 4.445 270) (size 1.5 0.6) (layers F.Cu F.Paste F.Mask)
       (net 11 /GD_LOW/-VEE))
-    (pad 7 smd rect (at -4.65 3.175 270) (size 1.5 0.6) (layers F.Cu F.Paste F.Mask)
-      (net 62 "Net-(U5-Pad7)"))
+    (pad 7 smd rect (at -4.65 3.175 270) (size 1.5 0.6) (layers F.Cu F.Paste F.Mask))
     (pad 6 smd rect (at -4.65 1.905 270) (size 1.5 0.6) (layers F.Cu F.Paste F.Mask)
       (net 48 "Net-(R25-Pad2)"))
@@
     )
   )
-  (module Diodes_SMD:D_SOD-323_HandSoldering (layer B.Cu)
-    (at 9.398 17.1704 90)
-    (descr SOD-323)
-    (tags SOD-323)
-    (attr smd)
-    (fp_text reference D16 (at 0 1.85 90) (layer B.SilkS)
-      (effects (font (size 1 1) (thickness 0.15)) (justify mirror))
-    )
-    (fp_text value PMEG4010 (at 0.1 -1.9 90) (layer B.Fab)
-      (effects (font (size 1 1) (thickness 0.15)) (justify mirror))
-    )
-    (fp_text user %R (at 0 1.85 90) (layer B.Fab)
-      (effects (font (size 1 1) (thickness 0.15)) (justify mirror))
-    )
-    (fp_line (start -1.9 0.85) (end -1.9 -0.85) (layer B.SilkS) (width 0.12))
-    (fp_line (start 0.2 0) (end 0.45 0) (layer B.Fab) (width 0.1))
-    (fp_line (start 0.2 -0.35) (end -0.3 0) (layer B.Fab) (width 0.1))
-    (fp_line (start 0.2 0.35) (end 0.2 -0.35) (layer B.Fab) (width 0.1))
-    (fp_line (start -0.3 0) (end 0.2 0.35) (layer B.Fab) (width 0.1))
-    (fp_line (start -0.3 0) (end -0.5 0) (layer B.Fab) (width 0.1))
-    (fp_line (start -0.3 0.35) (end -0.3 -0.35) (layer B.Fab) (width 0.1))
-    (fp_line (start -0.9 -0.7) (end -0.9 0.7) (layer B.Fab) (width 0.1))
-    (fp_line (start 0.9 -0.7) (end -0.9 -0.7) (layer B.Fab) (width 0.1))
-    (fp_line (start 0.9 0.7) (end 0.9 -0.7) (layer B.Fab) (width 0.1))
-    (fp_line (start -0.9 0.7) (end 0.9 0.7) (layer B.Fab) (width 0.1))
-    (fp_line (start -2 0.95) (end 2 0.95) (layer B.CrtYd) (width 0.05))
-    (fp_line (start 2 0.95) (end 2 -0.95) (layer B.CrtYd) (width 0.05))
-    (fp_line (start -2 -0.95) (end 2 -0.95) (layer B.CrtYd) (width 0.05))
-    (fp_line (start -2 0.95) (end -2 -0.95) (layer B.CrtYd) (width 0.05))
-    (fp_line (start -1.9 -0.85) (end 1.25 -0.85) (layer B.SilkS) (width 0.12))
-    (fp_line (start -1.9 0.85) (end 1.25 0.85) (layer B.SilkS) (width 0.12))
-    (pad 1 smd rect (at -1.25 0 90) (size 1 1) (layers B.Cu B.Paste B.Mask)
-      (net 6 /GD_HIGH/+VCC))
-    (pad 2 smd rect (at 1.25 0 90) (size 1 1) (layers B.Cu B.Paste B.Mask)
-      (net 12 /GD_HIGH/G))
-    (model ${KISYS3DMOD}/Diodes_SMD.3dshapes/D_SOD-323.wrl
-      (at (xyz 0 0 0))
-      (scale (xyz 1 1 1))
-      (rotate (xyz 0 0 0))
-    )
-  )
-  (module Diodes_SMD:D_SOD-323_HandSoldering (layer B.Cu)
-    (at 45.5676 17.2466 90)
-    (descr SOD-323)
-    (tags SOD-323)
-    (attr smd)
-    (fp_text reference D22 (at 0 1.85 90) (layer B.SilkS)
-      (effects (font (size 1 1) (thickness 0.15)) (justify mirror))
-    )
-    (fp_text value PMEG4010 (at 0.1 -1.9 90) (layer B.Fab)
-      (effects (font (size 1 1) (thickness 0.15)) (justify mirror))
-    )
-    (fp_line (start -1.9 0.85) (end 1.25 0.85) (layer B.SilkS) (width 0.12))
-    (fp_line (start -1.9 -0.85) (end 1.25 -0.85) (layer B.SilkS) (width 0.12))
-    (fp_line (start -2 0.95) (end -2 -0.95) (layer B.CrtYd) (width 0.05))
-    (fp_line (start -2 -0.95) (end 2 -0.95) (layer B.CrtYd) (width 0.05))
-    (fp_line (start 2 0.95) (end 2 -0.95) (layer B.CrtYd) (width 0.05))
-    (fp_line (start -2 0.95) (end 2 0.95) (layer B.CrtYd) (width 0.05))
-    (fp_line (start -0.9 0.7) (end 0.9 0.7) (layer B.Fab) (width 0.1))
-    (fp_line (start 0.9 0.7) (end 0.9 -0.7) (layer B.Fab) (width 0.1))
-    (fp_line (start 0.9 -0.7) (end -0.9 -0.7) (layer B.Fab) (width 0.1))
-    (fp_line (start -0.9 -0.7) (end -0.9 0.7) (layer B.Fab) (width 0.1))
-    (fp_line (start -0.3 0.35) (end -0.3 -0.35) (layer B.Fab) (width 0.1))
-    (fp_line (start -0.3 0) (end -0.5 0) (layer B.Fab) (width 0.1))
-    (fp_line (start -0.3 0) (end 0.2 0.35) (layer B.Fab) (width 0.1))
-    (fp_line (start 0.2 0.35) (end 0.2 -0.35) (layer B.Fab) (width 0.1))
-    (fp_line (start 0.2 -0.35) (end -0.3 0) (layer B.Fab) (width 0.1))
-    (fp_line (start 0.2 0) (end 0.45 0) (layer B.Fab) (width 0.1))
-    (fp_line (start -1.9 0.85) (end -1.9 -0.85) (layer B.SilkS) (width 0.12))
-    (fp_text user %R (at 0 1.85 90) (layer B.Fab)
-      (effects (font (size 1 1) (thickness 0.15)) (justify mirror))
-    )
-    (pad 2 smd rect (at 1.25 0 90) (size 1 1) (layers B.Cu B.Paste B.Mask)
-      (net 13 /GD_LOW/G))
-    (pad 1 smd rect (at -1.25 0 90) (size 1 1) (layers B.Cu B.Paste B.Mask)
-      (net 10 /GD_LOW/+VCC))
-    (model ${KISYS3DMOD}/Diodes_SMD.3dshapes/D_SOD-323.wrl
-      (at (xyz 0 0 0))
-      (scale (xyz 1 1 1))
-      (rotate (xyz 0 0 0))
-    )
-  )
   (gr_line (start 30.8 1.5) (end 27.8 1.5) (layer Edge.Cuts) (width 0.15))
   (gr_line (start 30.8 8.5) (end 30.8 1.5) (layer Edge.Cuts) (width 0.15))
@@
   (segment (start 3.2032 47.2276) (end 5.323 47.2276) (width 1) (layer B.Cu) (net 5))
   (segment (start 5.323 47.2276) (end 5.3594 47.264) (width 1) (layer B.Cu) (net 5))
-  (segment (start 9.398 18.4204) (end 9.398 24.154526) (width 0.25) (layer B.Cu) (net 6))
-  (segment (start 9.398 24.154526) (end 9.422146 24.178672) (width 0.25) (layer B.Cu) (net 6))
   (segment (start 9.1948 43.2054) (end 8.4836 42.4942) (width 1) (layer B.Cu) (net 6))
   (segment (start 5.3921 42.4942) (end 5.3594 42.5269) (width 1) (layer B.Cu) (net 6))
@@
   (segment (start 37.2032 57.3876) (end 41.137 57.3876) (width 2) (layer B.Cu) (net 9))
   (segment (start 41.137 57.3876) (end 41.1734 57.424) (width 2) (layer B.Cu) (net 9))
-  (segment (start 45.5676 18.4966) (end 45.5676 23.908) (width 0.25) (layer B.Cu) (net 10))
-  (segment (start 45.5676 23.908) (end 45.5234 23.9522) (width 0.25) (layer B.Cu) (net 10))
-  (segment (start 9.398 15.9204) (end 9.398 14.9982) (width 0.25) (layer B.Cu) (net 12))
-  (segment (start 9.398 14.9982) (end 9.7978 14.5984) (width 0.25) (layer B.Cu) (net 12))
   (via (at 16.7978 12.5984) (size 0.8) (drill 0.4) (layers F.Cu B.Cu) (net 12))
   (via (at 15.7978 12.5984) (size 0.8) (drill 0.4) (layers F.Cu B.Cu) (net 12))
@@
   (via (at 13.7978 12.5984) (size 0.8) (drill 0.4) (layers F.Cu B.Cu) (net 12))
   (via (at 16.7978 14.5984) (size 0.8) (drill 0.4) (layers F.Cu B.Cu) (net 12))
-  (segment (start 45.5676 15.9966) (end 45.5676 15.1252) (width 0.25) (layer B.Cu) (net 13))
-  (segment (start 45.5676 15.1252) (end 45.9674 14.7254) (width 0.25) (layer B.Cu) (net 13))
   (segment (start 40.8634 0.5334) (end 35.0774 0.5334) (width 1) (layer B.Cu) (net 13))
   (segment (start 43.5 3.17) (end 40.8634 0.5334) (width 1) (layer B.Cu) (net 13))
