File: V0.3/PCB/ENNOID Dual Gate Driver.sch (KiCad schematic (older format))
At the start: 24 parts, among them J1 Conn_02x08_Odd_Even, J2 Current, J3 TEMP, J4 PHASE, J5 Collector, J6 Gate_H, J7 G_L, J8 E, U1 MC7805

Commit message: V0.2 completed
Parts:
- added D?: GSOT03C, TO_SOT_Packages_SMD:SOT-23, symbol device:D_Schottky_x2_ACom_KKA
- added R?: 4.7k, Resistors_SMD:R_0805_HandSoldering, symbol device:R
- added R?: 1k, Resistors_SMD:R_0805_HandSoldering, symbol device:R
- added U? (x2): 74LVC1G86, symbol Logic_74xgxx:74LVC1G86
- added U?: 74LVC2G08, symbol Logic_74xgxx:74LVC2G08
Connections:
- wire segments 120 -> 142
