File: V0.3/PCB/GD.sch (KiCad schematic (older format))
At the start: 44 parts, among them Q3 MJD3055T4G, Q4 MJD2955T4G, U4 ISO5852SDWR

Commit message: V0.3 started
Parts:
- removed D16: PMEG4010, Diodes_SMD:D_SOD-323_HandSoldering, symbol device:D_Schottky
- removed Q3: MJD3055T4G, TO_SOT_Packages_SMD:TO-252-2, symbol device:Q_NPN_Darlington_BCEC
- removed Q4: MJD2955T4G, TO_SOT_Packages_SMD:TO-252-2, symbol device:Q_PNP_Darlington_BCEC
- removed R12, R13: 12, Resistors_SMD:R_0805_HandSoldering, symbol device:R
- removed U4: ISO5852SDWR, Housings_SOIC:SOIC-16W_7.5x10.3mm_Pitch1.27mm, symbol ENNOID:ISO5852SDWR
Connections:
- wire segments 159 -> 150
- no-connect marks 3 -> 1

Commit message: V0.2 completed
Parts:
- removed C17: 15n, Capacitors_SMD:C_0805_HandSoldering, symbol device:C
- removed C18, C19: 100n, Capacitors_SMD:C_0805_HandSoldering, symbol device:C
- removed C20, C21: 1u, Capacitors_SMD:C_0805_HandSoldering, symbol device:C
- removed C23: 10u, Capacitors_SMD:C_1206_HandSoldering, symbol device:C
- removed D2: GSOT03C, TO_SOT_Packages_SMD:SOT-23, symbol device:D_Schottky_x2_ACom_KKA
- removed R11: 12, Resistors_SMD:R_0805_HandSoldering, symbol device:R
- removed R3: 4.7k, Resistors_SMD:R_0805_HandSoldering, symbol device:R
- removed R4: 1k, Resistors_SMD:R_0805_HandSoldering, symbol device:R
- removed R9: 10k, Resistors_SMD:R_0805_HandSoldering, symbol device:R
- added C?: 10n, Capacitors_SMD:C_0805_HandSoldering, symbol device:C
- added C?: 33p, Capacitors_SMD:C_0805_HandSoldering, symbol device:C
- added U?: SID11X2K, Housing_eSOP, symbol ENNOID:SID11X2K
Connections:
- net labels removed: PWM-, RDY
- wire segments 150 -> 111
- no-connect marks 1 -> 0
