File: V0.3/PCB/GD.sch (KiCad schematic (older format))
At the start: 44 parts, among them Q3 MJD3055T4G, Q4 MJD2955T4G, U4 ISO5852SDWR

Commit message: Maintenance update
Parts:
- removed D21: es2j-ltp, Diodes_SMD:D_SMA_Handsoldering, symbol Device:D
- removed D8: smcj440ca, Diodes_SMD:D_SMC, symbol ENNOID-Dual-Gate-Driver-rescue:D_TVS-device-ENNOID-Dual-Gate-Driver-rescue-ENNO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
- added D?: diode, Diodes_THT:D_DO-41_SOD81_P12.70mm_Horizontal, symbol ENNOID-Dual-Gate-Driver-rescue:D-device-ENNOID-Dual-Gate-Driver-rescue
- added R? (x2): r, Resistors_SMD:R_2512, symbol ENNOID-Dual-Gate-Driver-rescue:R-device-ENNOID-Dual-Gate-Driver-rescue
- C14, C17, C18, C19, C20, C21, C22, C23, C24, C25, C26, C28, C29, C30, C31, C32, C33, C34: symbol ENNOID-Dual-Gate-Driver-rescue:C-device-ENNOID-Dual-Gate-Driver-rescue-ENNOID-Dual-Gate-Driver-rescue-ENNOID-Dual-Gate-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 -> ENNOID-Dual-Gate-Driver-rescue:C-device-ENNOID-Dual-Gate-Driver-rescue
- D10, D16: symbol ENNOID-Dual-Gate-Driver-rescue:D_Schottky-device-ENNOID-Dual-Gate-Driver-rescue-ENNOID-Dual-Gate-Driver-rescue-ENNOID-D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 -> ENNOID-Dual-Gate-Driver-rescue:D_Schottky-device-ENNOID-Dual-Gate-Driver-rescue
- D11: symbol ENNOID-Dual-Gate-Driver-rescue:D_TVS-device-ENNOID-Dual-Gate-Driver-rescue-ENNOID-Dual-Gate-Driver-rescue-ENNOID-Dual-G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 -> ENNOID-Dual-Gate-Driver-rescue:D_TVS-device-ENNOID-Dual-Gate-Driver-rescue
- D2: symbol ENNOID-Dual-Gate-Driver-rescue:D_Schottky_x2_ACom_KKA-device-ENNOID-Dual-Gate-Driver-rescue-ENNOID-Dual-Gate-Driver-res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 -> ENNOID-Dual-Gate-Driver-rescue:D_Schottky_x2_ACom_KKA-device-ENNOID-Dual-Gate-Driver-rescue
- D3, D4: symbol ENNOID-Dual-Gate-Driver-rescue:D-device-ENNOID-Dual-Gate-Driver-rescue-ENNOID-Dual-Gate-Driver-rescue-ENNOID-Dual-Gate-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 -> ENNOID-Dual-Gate-Driver-rescue:D-device-ENNOID-Dual-Gate-Driver-rescue
- D6: symbol ENNOID-Dual-Gate-Driver-rescue:D_Zener-device-ENNOID-Dual-Gate-Driver-rescue-ENNOID-Dual-Gate-Driver-rescue-ENNOID-Dual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 -> ENNOID-Dual-Gate-Driver-rescue:D_Zener-device-ENNOID-Dual-Gate-Driver-rescue
- Q3: symbol ENNOID-Dual-Gate-Driver-rescue:Q_NPN_Darlington_BCEC-device-ENNOID-Dual-Gate-Driver-rescue-ENNOID-Dual-Gate-Driver-resc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 -> ENNOID-Dual-Gate-Driver-rescue:Q_NPN_Darlington_BCEC-device-ENNOID-Dual-Gate-Driver-rescue
- Q4: symbol ENNOID-Dual-Gate-Driver-rescue:Q_PNP_Darlington_BCEC-device-ENNOID-Dual-Gate-Driver-rescue-ENNOID-Dual-Gate-Driver-resc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 -> ENNOID-Dual-Gate-Driver-rescue:Q_PNP_Darlington_BCEC-device-ENNOID-Dual-Gate-Driver-rescue
- R10, R11, R12, R13, R14, R15, R22, R23, R24, R3, R4, R7, R8, R9: symbol ENNOID-Dual-Gate-Driver-rescue:R-device-ENNOID-Dual-Gate-Driver-rescue-ENNOID-Dual-Gate-Driver-rescue-ENNOID-Dual-Gate-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 -> ENNOID-Dual-Gate-Driver-rescue:R-device-ENNOID-Dual-Gate-Driver-rescue
Connections:
- net labels added: bus
- net labels removed: GND_ISO
- wire segments 161 -> 163
Other:
- note added: "+Vle\n"
- note added: "-Vle\n"
- note added: "Adjust resistors (depend of circuit)\n"
- note added: "TM4 (reflex) active clamping"

Commit message: V0.3 - New voltage clamping technique
Added TM4 reflex active clampiing
Parts:
- C14, C17, C18, C19, C20, C21, C22, C23, C24, C25, C26, C28, C29, C30, C31, C32, C33, C34: symbol ENNOID-Dual-Gate-Driver-rescue:C-device-ENNOID-Dual-Gate-Driver-rescue -> ENNOID-Dual-Gate-Driver-rescue:C-device-ENNOID-Dual-Gate-Driver-rescue-ENNOID-Dual-Gate-Driver-rescue
- D10, D16: symbol ENNOID-Dual-Gate-Driver-rescue:D_Schottky-device-ENNOID-Dual-Gate-Driver-rescue -> ENNOID-Dual-Gate-Driver-rescue:D_Schottky-device-ENNOID-Dual-Gate-Driver-rescue-ENNOID-Dual-Gate-Driver-rescue
- D11: footprint Diodes_SMD:D_SMA_Handsoldering -> Diodes_SMD:D_SMA; symbol ENNOID-Dual-Gate-Driver-rescue:D_TVS-device-ENNOID-Dual-Gate-Driver-rescue -> ENNOID-Dual-Gate-Driver-rescue:D_TVS-device-ENNOID-Dual-Gate-Driver-rescue-ENNOID-Dual-Gate-Driver-rescue
- D2: symbol ENNOID-Dual-Gate-Driver-rescue:D_Schottky_x2_ACom_KKA-device-ENNOID-Dual-Gate-Driver-rescue -> ENNOID-Dual-Gate-Driver-rescue:D_Schottky_x2_ACom_KKA-device-ENNOID-Dual-Gate-Driver-rescue-ENNOID-Dual-Gate-Driver-res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
- D3, D4: symbol ENNOID-Dual-Gate-Driver-rescue:D-device-ENNOID-Dual-Gate-Driver-rescue -> ENNOID-Dual-Gate-Driver-rescue:D-device-ENNOID-Dual-Gate-Driver-rescue-ENNOID-Dual-Gate-Driver-rescue
- D5: renamed from D?; footprint Diodes_THT:D_DO-41_SOD81_P12.70mm_Horizontal -> Diodes_SMD:D_SMA; symbol ENNOID-Dual-Gate-Driver-rescue:D-device-ENNOID-Dual-Gate-Driver-rescue -> ENNOID-Dual-Gate-Driver-rescue:D-device-ENNOID-Dual-Gate-Driver-rescue-ENNOID-Dual-Gate-Driver-rescue
- D6: symbol ENNOID-Dual-Gate-Driver-rescue:D_Zener-device-ENNOID-Dual-Gate-Driver-rescue -> ENNOID-Dual-Gate-Driver-rescue:D_Zener-device-ENNOID-Dual-Gate-Driver-rescue-ENNOID-Dual-Gate-Driver-rescue
- Q3: symbol ENNOID-Dual-Gate-Driver-rescue:Q_NPN_Darlington_BCEC-device-ENNOID-Dual-Gate-Driver-rescue -> ENNOID-Dual-Gate-Driver-rescue:Q_NPN_Darlington_BCEC-device-ENNOID-Dual-Gate-Driver-rescue-ENNOID-Dual-Gate-Driver-resc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
- Q4: symbol ENNOID-Dual-Gate-Driver-rescue:Q_PNP_Darlington_BCEC-device-ENNOID-Dual-Gate-Driver-rescue -> ENNOID-Dual-Gate-Driver-rescue:Q_PNP_Darlington_BCEC-device-ENNOID-Dual-Gate-Driver-rescue-ENNOID-Dual-Gate-Driver-resc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
- R10, R11, R12, R13, R14, R15, R22, R23, R24, R3, R4, R7, R8, R9: symbol ENNOID-Dual-Gate-Driver-rescue:R-device-ENNOID-Dual-Gate-Driver-rescue -> ENNOID-Dual-Gate-Driver-rescue:R-device-ENNOID-Dual-Gate-Driver-rescue-ENNOID-Dual-Gate-Driver-rescue
- R19, R31: renamed from R?; footprint Resistors_SMD:R_2512 -> Resistors_SMD:R_1210; symbol ENNOID-Dual-Gate-Driver-rescue:R-device-ENNOID-Dual-Gate-Driver-rescue -> ENNOID-Dual-Gate-Driver-rescue:R-device-ENNOID-Dual-Gate-Driver-rescue-ENNOID-Dual-Gate-Driver-rescue
Connections:
- net labels added: BUS, GND_ISO
- net labels removed: bus
- wire segments 163 -> 166

Commit message: readme
Parts:
- C14, C17, C18, C19, C20, C21, C22, C23, C24, C25, C26, C28, C29, C30, C31, C32, C33, C34: symbol ENNOID-Dual-Gate-Driver-rescue:C-device-ENNOID-Dual-Gate-Driver-rescue-ENNOID-Dual-Gate-Driver-rescue -> ENNOID-Dual-Gate-Driver-rescue:C-device-ENNOID-Dual-Gate-Driver-rescue-ENNOID-Dual-Gate-Driver-rescue-ENNOID-Dual-Gate-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
- D10, D16: symbol ENNOID-Dual-Gate-Driver-rescue:D_Schottky-device-ENNOID-Dual-Gate-Driver-rescue-ENNOID-Dual-Gate-Driver-rescue -> ENNOID-Dual-Gate-Driver-rescue:D_Schottky-device-ENNOID-Dual-Gate-Driver-rescue-ENNOID-Dual-Gate-Driver-rescue-ENNOID-D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
- D11: symbol ENNOID-Dual-Gate-Driver-rescue:D_TVS-device-ENNOID-Dual-Gate-Driver-rescue-ENNOID-Dual-Gate-Driver-rescue -> ENNOID-Dual-Gate-Driver-rescue:D_TVS-device-ENNOID-Dual-Gate-Driver-rescue-ENNOID-Dual-Gate-Driver-rescue-ENNOID-Dual-G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
- D2: symbol ENNOID-Dual-Gate-Driver-rescue:D_Schottky_x2_ACom_KKA-device-ENNOID-Dual-Gate-Driver-rescue-ENNOID-Dual-Gate-Driver-rescue -> ENNOID-Dual-Gate-Driver-rescue:D_Schottky_x2_ACom_KKA-device-ENNOID-Dual-Gate-Driver-rescue-ENNOID-Dual-Gate-Driver-rescue-ENNOID-Dual-Gate-Driver-rescue
- D3, D4, D5: symbol ENNOID-Dual-Gate-Driver-rescue:D-device-ENNOID-Dual-Gate-Driver-rescue-ENNOID-Dual-Gate-Driver-rescue -> ENNOID-Dual-Gate-Driver-rescue:D-device-ENNOID-Dual-Gate-Driver-rescue-ENNOID-Dual-Gate-Driver-rescue-ENNOID-Dual-Gate-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
- D6: symbol ENNOID-Dual-Gate-Driver-rescue:D_Zener-device-ENNOID-Dual-Gate-Driver-rescue-ENNOID-Dual-Gate-Driver-rescue -> ENNOID-Dual-Gate-Driver-rescue:D_Zener-device-ENNOID-Dual-Gate-Driver-rescue-ENNOID-Dual-Gate-Driver-rescue-ENNOID-Dual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
- Q3: symbol ENNOID-Dual-Gate-Driver-rescue:Q_NPN_Darlington_BCEC-device-ENNOID-Dual-Gate-Driver-rescue-ENNOID-Dual-Gate-Driver-rescue -> ENNOID-Dual-Gate-Driver-rescue:Q_NPN_Darlington_BCEC-device-ENNOID-Dual-Gate-Driver-rescue-ENNOID-Dual-Gate-Driver-rescue-ENNOID-Dual-Gate-Driver-rescue
- Q4: symbol ENNOID-Dual-Gate-Driver-rescue:Q_PNP_Darlington_BCEC-device-ENNOID-Dual-Gate-Driver-rescue-ENNOID-Dual-Gate-Driver-rescue -> ENNOID-Dual-Gate-Driver-rescue:Q_PNP_Darlington_BCEC-device-ENNOID-Dual-Gate-Driver-rescue-ENNOID-Dual-Gate-Driver-rescue-ENNOID-Dual-Gate-Driver-rescue
- R10, R11, R12, R13, R14, R15, R19, R22, R23, R24, R3, R31, R4, R7, R8, R9: symbol ENNOID-Dual-Gate-Driver-rescue:R-device-ENNOID-Dual-Gate-Driver-rescue-ENNOID-Dual-Gate-Driver-rescue -> ENNOID-Dual-Gate-Driver-rescue:R-device-ENNOID-Dual-Gate-Driver-rescue-ENNOID-Dual-Gate-Driver-rescue-ENNOID-Dual-Gate-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
