File: VBUS-Sense/PCB/VBUS-Sense.sch (KiCad schematic (older format))
At the start: 0 parts

Commit message: VBUS sensor & voltage sense circuit changes
Parts:
- added J1, J2: Conn_01x01, Mounting_Holes:MountingHole_3.2mm_M3_ISO14580_Pad, symbol Connector:Conn_01x01
- added J3: Conn_01x04, Connectors_Molex:Molex_KK-6410-04_04x2.54mm_Straight, symbol Connector:Conn_01x04
Connections:
- net labels added: +5V, GND
- wire segments 0 -> 16
Changed lines of the file:
@@
 $Descr A4 11693 8268
 encoding utf-8
-Sheet 1 2
+Sheet 1 3
 Title ""
 Date ""
@@
 $EndDescr
 $Sheet
-S 3100 2500 2100 1300
+S 3200 2500 2100 1300
 U 5A4D4667
 F0 "V_PHASE" 50
 F1 "V_PHASE.sch" 50
-F2 "PHASE" I L 3100 2700 50
-F3 "E" I L 3100 2950 50
-F4 "+5V" I L 3100 3250 50
-F5 "Vout+" O R 5200 2850 50
-F6 "Vout-" O R 5200 3200 50
-F7 "GND" I R 5200 3500 50
-F8 "+VCC" I R 5200 2650 50
+F2 "+5V" I R 5300 2700 50
+F3 "Vout+" O R 5300 2800 50
+F4 "Vout-" O R 5300 2900 50
+F5 "GND" I R 5300 3000 50
+F6 "VBUS+" I L 3200 2600 50
+F7 "VBUS-" I L 3200 3050 50
+F8 "+VCC" I L 3200 2900 50
 $EndSheet
+$Comp
+L Connector:Conn_01x04 J3
+U 1 1 5A4FB1AF
+P 5750 2800
+F 0 "J3" H 5830 2792 50  0000 L CNN
+F 1 "Conn_01x04" H 5830 2701 50  0000 L CNN
+F 2 "Connectors_Molex:Molex_KK-6410-04_04x2.54mm_Straight" H 5750 2800 50  0001 C CNN
+F 3 "~" H 5750 2800 50  0001 C CNN
+	1    5750 2800
+	1    0    0    -1
+$EndComp
+Wire Wire Line
+	5300 2700 5500 2700
+Wire Wire Line
+	5550 2800 5300 2800
+Wire Wire Line
+	5550 2900 5300 2900
+Wire Wire Line
+	5550 3000 5450 3000
+$Comp
+L power:GND #PWR03
+U 1 1 5A50046C
+P 5450 3000
+F 0 "#PWR03" H 5450 2750 50  0001 C CNN
+F 1 "GND" H 5455 2827 50  0000 C CNN
+F 2 "" H 5450 3000 50  0001 C CNN
+F 3 "" H 5450 3000 50  0001 C CNN
+	1    5450 3000
+	1    0    0    -1
+$EndComp
+Connection ~ 5450 3000
+Wire Wire Line
+	5450 3000 5300 3000
+$Comp
+L power:+5V #PWR04
+U 1 1 5A500584
+P 5500 2700
+F 0 "#PWR04" H 5500 2550 50  0001 C CNN
+F 1 "+5V" H 5515 2873 50  0000 C CNN
+F 2 "" H 5500 2700 50  0001 C CNN
+F 3 "" H 5500 2700 50  0001 C CNN
+	1    5500 2700
+	1    0    0    -1
+$EndComp
+Connection ~ 5500 2700
+Wire Wire Line
+	5500 2700 5550 2700
+Wire Wire Line
+	2600 2900 3200 2900
+$Comp
+L Connector:Conn_01x01 J1
+U 1 1 5A502646
+P 1650 2600
+F 0 "J1" H 1570 2375 50  0000 C CNN
+F 1 "Conn_01x01" H 1570 2466 50  0000 C CNN
+F 2 "Mounting_Holes:MountingHole_3.2mm_M3_ISO14580_Pad" H 1650 2600 50  0001 C CNN
+F 3 "~" H 1650 2600 50  0001 C CNN
+	1    1650 2600
+	-1   0    0    1
+$EndComp
+Wire Wire Line
+	1850 2600 3200 2600
+$Comp
+L Connector:Conn_01x01 J2
+U 1 1 5A5032A8
+P 1650 3050
+F 0 "J2" H 1570 2825 50  0000 C CNN
+F 1 "Conn_01x01" H 1570 2916 50  0000 C CNN
+F 2 "Mounting_Holes:MountingHole_3.2mm_M3_ISO14580_Pad" H 1650 3050 50  0001 C CNN
+F 3 "~" H 1650 3050 50  0001 C CNN
+	1    1650 3050
+	-1   0    0    1
+$EndComp
+Wire Wire Line
+	1850 3050 2900 3050
+$Sheet
+S 3300 1100 1650 700
+U 5A511F6B
+F0 "isolated_5v" 50
+F1 "isolated_5v.sch" 50
+F2 "+5V" I R 4950 1200 50
+F3 "GND" I R 4950 1600 50
+F4 "+VCC" I L 3300 1250 50
+F5 "VBUS-" I L 3300 1650 50
+$EndSheet
+Wire Wire Line
+	3300 1250 2600 1250
+Wire Wire Line
+	2600 1250 2600 2900
+Wire Wire Line
+	2900 3050 2900 1650
+Wire Wire Line
+	2900 1650 3300 1650
+Connection ~ 2900 3050
+Wire Wire Line
+	2900 3050 3200 3050
+$Comp
+L power:+5V #PWR01
+U 1 1 5A511DAF
+P 5150 1200
+F 0 "#PWR01" H 5150 1050 50  0001 C CNN
+F 1 "+5V" H 5165 1373 50  0000 C CNN
+F 2 "" H 5150 1200 50  0001 C CNN
+F 3 "" H 5150 1200 50  0001 C CNN
+	1    5150 1200
+	1    0    0    -1
+$EndComp
+Wire Wire Line
+	4950 1200 5150 1200
+$Comp
+L power:GND #PWR02
+U 1 1 5A511F9D
+P 5150 1600
+F 0 "#PWR02" H 5150 1350 50  0001 C CNN
+F 1 "GND" H 5155 1427 50  0000 C CNN
+F 2 "" H 5150 1600 50  0001 C CNN
+F 3 "" H 5150 1600 50  0001 C CNN
+	1    5150 1600
+	1    0    0    -1
+$EndComp
+Wire Wire Line
+	4950 1600 5150 1600
 $EndSCHEMATC

Commit message: V0.2 pcb changes
Parts:
- added Q?: Q_NMOS_GDS, symbol device:Q_NMOS_GDS
- added R? (x4): 20k, Resistors_SMD:R_2512_HandSoldering, symbol device:R
Connections:
- wire segments 16 -> 28

Commit message: V0.2 PCB
Parts:
- Q1: renamed from Q?; footprint (none) -> TO_SOT_Packages_SMD:TO-252-2
- gave numbers to parts that had none: 4
Changed lines of the file:
@@
 Wire Wire Line
 	8100 3800 8150 3800
-Wire Wire Line
-	5200 4000 5800 4000
 $Comp
 L Connector:Conn_01x01 J1
@@
 Wire Wire Line
 	2150 4150 4450 4150
-$Sheet
-S 5800 2200 2100 850
-U 5A511F6B
-F0 "isolated_5v" 50
-F1 "isolated_5v.sch" 50
-F2 "+5V" I R 7900 2300 50
-F3 "GND" I R 7900 2700 50
-F4 "+VCC" I L 5800 2350 50
-F5 "VBUS-" I L 5800 2750 50
-$EndSheet
-Wire Wire Line
-	5800 2350 5200 2350
-Wire Wire Line
-	5200 2350 5200 3400
-Wire Wire Line
-	5500 4150 5500 2750
-Wire Wire Line
-	5500 2750 5800 2750
-Connection ~ 5500 4150
-Wire Wire Line
-	5500 4150 5800 4150
 $Comp
 L power:+5V #PWR01
 U 1 1 5A511DAF
-P 8100 2300
-F 0 "#PWR01" H 8100 2150 50  0001 C CNN
-F 1 "+5V" H 8115 2473 50  0000 C CNN
-F 2 "" H 8100 2300 50  0001 C CNN
-F 3 "" H 8100 2300 50  0001 C CNN
-	1    8100 2300
+P 8100 2500
+F 0 "#PWR01" H 8100 2350 50  0001 C CNN
+F 1 "+5V" H 8115 2673 50  0000 C CNN
+F 2 "" H 8100 2500 50  0001 C CNN
+F 3 "" H 8100 2500 50  0001 C CNN
+	1    8100 2500
 	1    0    0    -1
 $EndComp
 Wire Wire Line
-	7900 2300 8100 2300
+	7900 2500 8100 2500
 $Comp
 L power:GND #PWR02
@@
 	7900 2700 8100 2700
 $Comp
-L device:R R?
+L device:R R1
 U 1 1 5A5F09F3
 P 2650 3150
-F 0 "R?" V 2443 3150 50  0000 C CNN
+F 0 "R1" V 2443 3150 50  0000 C CNN
 F 1 "20k" V 2534 3150 50  0000 C CNN
 F 2 "Resistors_SMD:R_2512_HandSoldering" V 2580 3150 50  0001 C CNN
@@
 $EndComp
 $Comp
-L device:Q_NMOS_GDS Q?
+L device:Q_NMOS_GDS Q1
 U 1 1 5A5F1396
 P 4550 3400
-F 0 "Q?" H 4756 3446 50  0000 L CNN
+F 0 "Q1" H 4756 3446 50  0000 L CNN
 F 1 "Q_NMOS_GDS" H 4756 3355 50  0000 L CNN
-F 2 "" H 4750 3500 50  0001 C CNN
+F 2 "TO_SOT_Packages_SMD:TO-252-2" H 4750 3500 50  0001 C CNN
 F 3 "" H 4550 3400 50  0001 C CNN
 	1    4550 3400
@@
 $EndComp
 Wire Wire Line
-	4750 3400 5200 3400
-Connection ~ 5200 3400
-Wire Wire Line
-	5200 3400 5200 4000
-Wire Wire Line
 	4450 3600 4450 4150
 Connection ~ 4450 4150
-Wire Wire Line
-	4450 4150 5500 4150
 Wire Wire Line
 	4000 3150 4450 3150
@@
 	2400 3700 5800 3700
 $Comp
-L device:R R?
+L device:R R2
 U 1 1 5A5F51B6
 P 3050 3150
-F 0 "R?" V 2843 3150 50  0000 C CNN
+F 0 "R2" V 2843 3150 50  0000 C CNN
 F 1 "20k" V 2934 3150 50  0000 C CNN
 F 2 "Resistors_SMD:R_2512_HandSoldering" V 2980 3150 50  0001 C CNN
@@
 $EndComp
 $Comp
-L device:R R?
+L device:R R3
 U 1 1 5A5F5226
 P 3450 3150
-F 0 "R?" V 3243 3150 50  0000 C CNN
+F 0 "R3" V 3243 3150 50  0000 C CNN
 F 1 "20k" V 3334 3150 50  0000 C CNN
 F 2 "Resistors_SMD:R_2512_HandSoldering" V 3380 3150 50  0001 C CNN
@@
 $EndComp
 $Comp
-L device:R R?
+L device:R R4
 U 1 1 5A5F5294
 P 3850 3150
-F 0 "R?" V 3643 3150 50  0000 C CNN
+F 0 "R4" V 3643 3150 50  0000 C CNN
 F 1 "20k" V 3734 3150 50  0000 C CNN
 F 2 "Resistors_SMD:R_2512_HandSoldering" V 3780 3150 50  0001 C CNN
@@
 Wire Notes Line
 	6900 600  6900 650
+$Sheet
+S 5800 2400 2100 750
+U 5A628F9C
+F0 "ISO_PSU" 50
+F1 "ISO_PSU.sch" 50
+F2 "+5V" I R 7900 2500 50
+F3 "GND" I R 7900 2900 50
+F4 "+VCC" O L 5800 2950 50
+F5 "-VEE" O L 5800 2500 50
+F6 "COM" I L 5800 2750 50
+$EndSheet
+Wire Wire Line
+	4450 4150 5450 4150
+Wire Wire Line
+	5800 2950 5600 2950
+Wire Wire Line
+	5600 2950 5600 4000
+Wire Wire Line
+	5600 4000 5800 4000
+Wire Wire Line
+	5800 2750 5450 2750
+Wire Wire Line
+	5450 2750 5450 4150
+Connection ~ 5450 4150
+Wire Wire Line
+	5450 4150 5800 4150
+Wire Wire Line
+	5800 2500 4750 2500
+Wire Wire Line
+	4750 2500 4750 3400
 $EndSCHEMATC

Commit message: VBUS update
Parts:
- removed J1, J2: Conn_01x01, Mounting_Holes:MountingHole_3.2mm_M3_ISO14580_Pad, symbol Connector:Conn_01x01
- added J1: Conn_01x02 E-STOP, Connectors_Molex:Molex_KK-6410-02_02x2.54mm_Straight, symbol Connector_Generic:Conn_01x02
- added MK1: VBUS-, Pin_Headers:Pin_Header_Straight_1x01_Pitch2.54mm, symbol Mechanical:Mounting_Hole_PAD
- added MK2: VBUS+, Pin_Headers:Pin_Header_Straight_1x01_Pitch2.54mm, symbol Mechanical:Mounting_Hole_PAD
- added MK3: Gate, Mounting_Holes:MountingHole_4.3mm_M4_Pad_Via, symbol Mechanical:Mounting_Hole_PAD
- added MK4: BAT-, Mounting_Holes:MountingHole_4.3mm_M4_Pad_Via, symbol Mechanical:Mounting_Hole_PAD
- added R5: 20k, Resistors_SMD:R_0805_HandSoldering, symbol VBUS-Sense-rescue:R-device
- added R6: 100, Resistors_SMD:R_0805_HandSoldering, symbol VBUS-Sense-rescue:R-device
- J3: symbol Connector:Conn_01x04 -> VBUS-Sense-rescue:Conn_01x04-Connector
- Q1: value Q_NMOS_GDS -> Depletion mode FET ex: CPC3982; footprint TO_SOT_Packages_SMD:TO-252-2 -> TO_SOT_Packages_SMD:SOT-23W; symbol device:Q_NMOS_GDS -> VBUS-Sense-rescue:Q_NMOS_GDS-device
- R1, R2, R3, R4: symbol device:R -> VBUS-Sense-rescue:R-device
Connections:
- wire segments 28 -> 48
Other:
- note added: "Disharge circuit"
- note added: "This board has 4 functions\n- Measuring the voltage of the DC bus (VBUS)\n- Discharging the DC Bus when power is turned off\n- Precharging the DC bus through an external single IGBT module (Inrush_Limiter)\n- Driving an external Solid state contactor for E-STOP"
Changed lines of the file:
@@
 $Descr A4 11693 8268
 encoding utf-8
-Sheet 1 3
+Sheet 1 4
 Title ""
 Date ""
@@
 $EndDescr
 $Sheet
-S 5800 3600 2100 1300
+S 5800 3600 2100 900
 U 5A4D4667
-F0 "V_PHASE" 50
+F0 "V_BUS" 50
 F1 "V_PHASE.sch" 50
 F2 "+5V" I R 7900 3800 50
@@
 $EndSheet
 $Comp
-L Connector:Conn_01x04 J3
+L VBUS-Sense-rescue:Conn_01x04-Connector J3
 U 1 1 5A4FB1AF
 P 8350 3900
@@
 	8100 3800 8150 3800
 $Comp
-L Connector:Conn_01x01 J1
-U 1 1 5A502646
-P 1950 3700
-F 0 "J1" H 1870 3475 50  0000 C CNN
-F 1 "Conn_01x01" H 1870 3566 50  0000 C CNN
-F 2 "Mounting_Holes:MountingHole_3.2mm_M3_ISO14580_Pad" H 1950 3700 50  0001 C CNN
-F 3 "~" H 1950 3700 50  0001 C CNN
-	1    1950 3700
-	-1   0    0    1
-$EndComp
-$Comp
-L Connector:Conn_01x01 J2
-U 1 1 5A5032A8
-P 1950 4150
-F 0 "J2" H 1870 3925 50  0000 C CNN
-F 1 "Conn_01x01" H 1870 4016 50  0000 C CNN
-F 2 "Mounting_Holes:MountingHole_3.2mm_M3_ISO14580_Pad" H 1950 4150 50  0001 C CNN
-F 3 "~" H 1950 4150 50  0001 C CNN
-	1    1950 4150
-	-1   0    0    1
-$EndComp
-Wire Wire Line
-	2150 4150 4450 4150
-$Comp
 L power:+5V #PWR01
 U 1 1 5A511DAF
@@
 L power:GND #PWR02
 U 1 1 5A511F9D
-P 8100 2700
-F 0 "#PWR02" H 8100 2450 50  0001 C CNN
-F 1 "GND" H 8105 2527 50  0000 C CNN
-F 2 "" H 8100 2700 50  0001 C CNN
-F 3 "" H 8100 2700 50  0001 C CNN
-	1    8100 2700
-	1    0    0    -1
-$EndComp
-Wire Wire Line
-	7900 2700 8100 2700
-$Comp
-L device:R R1
+P 8100 2900
+F 0 "#PWR02" H 8100 2650 50  0001 C CNN
+F 1 "GND" H 8105 2727 50  0000 C CNN
+F 2 "" H 8100 2900 50  0001 C CNN
+F 3 "" H 8100 2900 50  0001 C CNN
+	1    8100 2900
+	1    0    0    -1
+$EndComp
+Wire Wire Line
+	7900 2900 8100 2900
+$Comp
+L VBUS-Sense-rescue:R-device R1
 U 1 1 5A5F09F3
 P 2650 3150
@@
 	0    1    1    0
 $EndComp
-$Comp
-L device:Q_NMOS_GDS Q1
-U 1 1 5A5F1396
-P 4550 3400
-F 0 "Q1" H 4756 3446 50  0000 L CNN
-F 1 "Q_NMOS_GDS" H 4756 3355 50  0000 L CNN
-F 2 "TO_SOT_Packages_SMD:TO-252-2" H 4750 3500 50  0001 C CNN
-F 3 "" H 4550 3400 50  0001 C CNN
-	1    4550 3400
-	-1   0    0    -1
-$EndComp
 Wire Wire Line
 	4450 3600 4450 4150
-Connection ~ 4450 4150
-Wire Wire Line
-	4000 3150 4450 3150
 Wire Wire Line
 	4450 3150 4450 3200
@@
 Wire Wire Line
 	2400 3150 2500 3150
-Wire Wire Line
-	2150 3700 2400 3700
 Connection ~ 2400 3700
 Wire Wire Line
 	2400 3700 5800 3700
 $Comp
-L device:R R2
+L VBUS-Sense-rescue:R-device R2
 U 1 1 5A5F51B6
 P 3050 3150
@@
 $EndComp
 $Comp
-L device:R R3
+L VBUS-Sense-rescue:R-device R3
 U 1 1 5A5F5226
 P 3450 3150
@@
 $EndComp
 $Comp
-L device:R R4
+L VBUS-Sense-rescue:R-device R4
 U 1 1 5A5F5294
 P 3850 3150
@@
 $EndSheet
 Wire Wire Line
-	4450 4150 5450 4150
+	4450 4150 4850 4150
 Wire Wire Line
 	5800 2950 5600 2950
@@
 	5800 2750 5450 2750
 Wire Wire Line
+	5450 4150 5800 4150
+$Sheet
+S 5800 750  2100 1350
+U 5A652E46
+F0 "Inrush_Limiter" 50
+F1 "Inrush_Limiter.sch" 50
+F2 "VBUS-" I L 5800 1450 50
+F3 "GATE" I L 5800 1200 50
+F4 "+VBUS" I L 5800 1750 50
+F5 "VBAT-" I L 5800 950 50
+F6 "ON/OFF" I R 7900 1000 50
+F7 "GND" I R 7900 1550 50
+F8 "+VCC" I L 5800 1950 50
+$EndSheet
+$Comp
+L Mechanical:Mounting_Hole_PAD MK3
+U 1 1 5A653073
+P 2850 1200
+F 0 "MK3" V 3087 1205 50  0000 C CNN
+F 1 "Gate" V 2996 1205 50  0000 C CNN
+F 2 "Mounting_Holes:MountingHole_4.3mm_M4_Pad_Via" H 2850 1200 50  0001 C CNN
+F 3 "" H 2850 1200 50  0001 C CNN
+	1    2850 1200
+	0    -1   -1   0
+$EndComp
+$Comp
+L Mechanical:Mounting_Hole_PAD MK1
+U 1 1 5A653119
+P 1000 1450
+F 0 "MK1" V 1237 1455 50  0000 C CNN
+F 1 "VBUS-" V 1146 1455 50  0000 C CNN
+F 2 "Pin_Headers:Pin_Header_Straight_1x01_Pitch2.54mm" H 1000 1450 50  0001 C CNN
+F 3 "" H 1000 1450 50  0001 C CNN
+	1    1000 1450
+	0    -1   -1   0
+$EndComp
+$Comp
+L Mechanical:Mounting_Hole_PAD MK2
+U 1 1 5A657E0D
+P 1650 3700
+F 0 "MK2" V 1887 3705 50  0000 C CNN
+F 1 "VBUS+" V 1796 3705 50  0000 C CNN
+F 2 "Pin_Headers:Pin_Header_Straight_1x01_Pitch2.54mm" H 1650 3700 50  0001 C CNN
+F 3 "" H 1650 3700 50  0001 C CNN
+	1    1650 3700
+	0    -1   -1   0
+$EndComp
+Wire Wire Line
+	2950 1200 5800 1200
+$Comp
+L VBUS-Sense-rescue:Q_NMOS_GDS-device Q1
+U 1 1 5A5F1396
+P 4550 3400
+F 0 "Q1" H 4756 3446 50  0000 L CNN
+F 1 "Depletion mode FET ex: CPC3982" H 4756 3355 50  0000 L CNN
+F 2 "TO_SOT_Packages_SMD:SOT-23W" H 4750 3500 50  0001 C CNN
+F 3 "" H 4550 3400 50  0001 C CNN
+	1    4550 3400
+	-1   0    0    -1
+$EndComp
+Wire Wire Line
+	4750 3400 4850 3400
+Wire Wire Line
+	5150 3400 5150 2500
+$Comp
+L VBUS-Sense-rescue:R-device R5
+U 1 1 5A66B839
+P 4850 3700
+F 0 "R5" V 4643 3700 50  0000 C CNN
+F 1 "20k" V 4734 3700 50  0000 C CNN
+F 2 "Resistors_SMD:R_0805_HandSoldering" V 4780 3700 50  0001 C CNN
+F 3 "" H 4850 3700 50  0001 C CNN
+	1    4850 3700
+	-1   0    0    1
+$EndComp
+Wire Wire Line
+	4850 3550 4850 3400
+Connection ~ 4850 3400
+Wire Wire Line
+	4850 3400 5150 3400
+Wire Wire Line
+	4850 3850 4850 4150
+Connection ~ 4850 4150
+Wire Wire Line
+	4850 4150 5450 4150
+Text Notes 800  6400 0    118  ~ 24
+This board has 4 functions\n- Measuring the voltage of the DC bus (VBUS)\n- Discharging the DC Bus when power is turned off\n- Precharging the DC bus through an external single IGBT module (Inrush_Limiter)\n- Driving an external Solid state contactor for E-STOP
+Wire Notes Line
+	2300 2800 5100 2800
+Wire Notes Line
+	5100 2800 5100 4000
+Wire Notes Line
+	5100 4000 2300 4000
+Wire Notes Line
+	2300 4000 2300 2800
+Text Notes 4250 3000 0    50   ~ 0
+Disharge circuit
+$Comp
+L VBUS-Sense-rescue:R-device R6
+U 1 1 5A678EEC
+P 5350 2500
+F 0 "R6" V 5143 2500 50  0000 C CNN
+F 1 "100" V 5234 2500 50  0000 C CNN
+F 2 "Resistors_SMD:R_0805_HandSoldering" V 5280 2500 50  0001 C CNN
+F 3 "" H 5350 2500 50  0001 C CNN
+	1    5350 2500
+	0    -1   -1   0
+$EndComp
+Wire Wire Line
+	5150 2500 5200 2500
+Wire Wire Line
+	5500 2500 5800 2500
+$Comp
+L Mechanical:Mounting_Hole_PAD MK4
+U 1 1 5A684EEC
+P 3450 950
+F 0 "MK4" V 3687 955 50  0000 C CNN
+F 1 "BAT-" V 3596 955 50  0000 C CNN
+F 2 "Mounting_Holes:MountingHole_4.3mm_M4_Pad_Via" H 3450 950 50  0001 C CNN
+F 3 "" H 3450 950 50  0001 C CNN
+	1    3450 950
+	0    -1   -1   0
+$EndComp
+Wire Wire Line
+	3550 950  5800 950
+Connection ~ 4450 4150
+Connection ~ 5450 4150
+Wire Wire Line
 	5450 2750 5450 4150
-Connection ~ 5450 4150
-Wire Wire Line
-	5450 4150 5800 4150
-Wire Wire Line
-	5800 2500 4750 2500
-Wire Wire Line
-	4750 2500 4750 3400
+Wire Wire Line
+	1100 1450 1250 1450
+Wire Wire Line
+	1250 1450 1250 4150
+Wire Wire Line
+	1250 4150 4450 4150
+Wire Wire Line
+	1750 3700 2000 3700
+Connection ~ 1250 1450
+Wire Wire Line
+	1250 1450 5800 1450
+Wire Wire Line
+	5800 1750 2000 1750
+Wire Wire Line
+	2000 1750 2000 3700
+Wire Wire Line
+	2000 3700 2400 3700
+Connection ~ 2000 3700
+$Comp
+L Connector_Generic:Conn_01x02 J1
+U 1 1 5A68F4CF
+P 8850 1300
+F 0 "J1" H 8930 1292 50  0000 L CNN
+F 1 "Conn_01x02 E-STOP" H 8930 1201 50  0000 L CNN
+F 2 "Connectors_Molex:Molex_KK-6410-02_02x2.54mm_Straight" H 8850 1300 50  0001 C CNN
+F 3 "~" H 8850 1300 50  0001 C CNN
+	1    8850 1300
+	1    0    0    -1
+$EndComp
+Wire Wire Line
+	8650 1300 8650 1000
+Wire Wire Line
+	8650 1000 7900 1000
+Wire Wire Line
+	8650 1400 8650 1550
+Wire Wire Line
+	8650 1550 7900 1550
+Wire Wire Line
+	4000 3150 4450 3150
+Wire Wire Line
+	5800 1950 5600 1950
+Wire Wire Line
+	5600 1950 5600 2950
+Connection ~ 5600 2950
 $EndSCHEMATC

Commit message: VBUS-SENSE changes
Parts:
- added C5: 100n, Capacitors_SMD:C_0805_HandSoldering, symbol Device:C
Connections:
- wire segments 48 -> 51
Other:
- moved on the sheet: Q1, R5
Changed lines of the file:
@@
 encoding utf-8
 Sheet 1 4
-Title ""
+Title "VBUS-SENSE"
 Date ""
-Rev ""
-Comp ""
+Rev "0.1"
+Comp "ENNOID"
 Comment1 ""
 Comment2 ""
@@
 $EndComp
 Wire Wire Line
-	4450 3600 4450 4150
-Wire Wire Line
-	4450 3150 4450 3200
+	4300 3600 4300 4150
+Wire Wire Line
+	4300 3150 4300 3200
 Wire Wire Line
 	3700 3150 3600 3150
@@
 $EndSheet
 Wire Wire Line
-	4450 4150 4850 4150
+	4300 4150 4650 4150
 Wire Wire Line
 	5800 2950 5600 2950
@@
 L VBUS-Sense-rescue:Q_NMOS_GDS-device Q1
 U 1 1 5A5F1396
-P 4550 3400
-F 0 "Q1" H 4756 3446 50  0000 L CNN
-F 1 "Depletion mode FET ex: CPC3982" H 4756 3355 50  0000 L CNN
-F 2 "TO_SOT_Packages_SMD:SOT-23W" H 4750 3500 50  0001 C CNN
-F 3 "" H 4550 3400 50  0001 C CNN
-	1    4550 3400
+P 4400 3400
+F 0 "Q1" H 4606 3446 50  0000 L CNN
+F 1 "Depletion mode FET ex: CPC3982" H 4606 3355 50  0000 L CNN
+F 2 "TO_SOT_Packages_SMD:SOT-23W" H 4600 3500 50  0001 C CNN
+F 3 "" H 4400 3400 50  0001 C CNN
+	1    4400 3400
 	-1   0    0    -1
 $EndComp
 Wire Wire Line
-	4750 3400 4850 3400
-Wire Wire Line
-	5150 3400 5150 2500
+	4600 3400 4650 3400
+Wire Wire Line
+	5050 3400 5050 2500
 $Comp
 L VBUS-Sense-rescue:R-device R5
 U 1 1 5A66B839
-P 4850 3700
-F 0 "R5" V 4643 3700 50  0000 C CNN
-F 1 "20k" V 4734 3700 50  0000 C CNN
-F 2 "Resistors_SMD:R_0805_HandSoldering" V 4780 3700 50  0001 C CNN
-F 3 "" H 4850 3700 50  0001 C CNN
-	1    4850 3700
+P 4650 3700
+F 0 "R5" V 4443 3700 50  0000 C CNN
+F 1 "20k" V 4534 3700 50  0000 C CNN
+F 2 "Resistors_SMD:R_0805_HandSoldering" V 4580 3700 50  0001 C CNN
+F 3 "" H 4650 3700 50  0001 C CNN
+	1    4650 3700
 	-1   0    0    1
 $EndComp
 Wire Wire Line
-	4850 3550 4850 3400
-Connection ~ 4850 3400
-Wire Wire Line
-	4850 3400 5150 3400
-Wire Wire Line
-	4850 3850 4850 4150
-Connection ~ 4850 4150
-Wire Wire Line
-	4850 4150 5450 4150
+	4650 3550 4650 3400
+Connection ~ 4650 3400
+Wire Wire Line
+	4650 3400 5050 3400
+Wire Wire Line
+	4650 3850 4650 4150
+Connection ~ 4650 4150
+Wire Wire Line
+	4650 4150 5050 4150
 Text Notes 800  6400 0    118  ~ 24
 This board has 4 functions\n- Measuring the voltage of the DC bus (VBUS)\n- Discharging the DC Bus when power is turned off\n- Precharging the DC bus through an external single IGBT module (Inrush_Limiter)\n- Driving an external Solid state contactor for E-STOP
 Wire Notes Line
-	2300 2800 5100 2800
-Wire Notes Line
-	5100 2800 5100 4000
-Wire Notes Line
-	5100 4000 2300 4000
+	2300 2800 5400 2800
+Wire Notes Line
+	5400 2800 5400 4000
+Wire Notes Line
+	5400 4000 2300 4000
 Wire Notes Line
 	2300 4000 2300 2800
@@
 $EndComp
 Wire Wire Line
-	5150 2500 5200 2500
+	5050 2500 5200 2500
 Wire Wire Line
 	5500 2500 5800 2500
@@
 Wire Wire Line
 	3550 950  5800 950
-Connection ~ 4450 4150
+Connection ~ 4300 4150
 Connection ~ 5450 4150
 Wire Wire Line
@@
 	1250 1450 1250 4150
 Wire Wire Line
-	1250 4150 4450 4150
+	1250 4150 4300 4150
 Wire Wire Line
 	1750 3700 2000 3700
@@
 	8650 1550 7900 1550
 Wire Wire Line
-	4000 3150 4450 3150
+	4000 3150 4300 3150
 Wire Wire Line
 	5800 1950 5600 1950
@@
 	5600 1950 5600 2950
 Connection ~ 5600 2950
+$Comp
+L Device:C C5
+U 1 1 5A6BE82E
+P 5050 3700
+F 0 "C5" H 5165 3746 50  0000 L CNN
+F 1 "100n" H 5165 3655 50  0000 L CNN
+F 2 "Capacitors_SMD:C_0805_HandSoldering" H 5088 3550 50  0001 C CNN
+F 3 "" H 5050 3700 50  0001 C CNN
+	1    5050 3700
+	1    0    0    -1
+$EndComp
+Wire Wire Line
+	5050 3550 5050 3400
+Connection ~ 5050 3400
+Wire Wire Line
+	5050 3850 5050 4150
+Connection ~ 5050 4150
+Wire Wire Line
+	5050 4150 5450 4150
 $EndSCHEMATC
