File: VBUS-Sense/PCB/VBUS-Sense.sch (KiCad schematic (older format))
At the start: 14 parts, among them J1 Conn_01x02 E-STOP, J3 Conn_01x04, Q1 Depletion mode FET ex: CPC3982

Commit message: VBUS-sense
Parts:
- added C?: DC Link Cap, Capacitors_SMD:C_0805_HandSoldering, symbol Device:C
- added Q?: IGBT, symbol Device:Q_NIGBT_CEG
Connections:
- no-connect marks 0 -> 5
Other:
- note added: "1200V 600A IGBT module"
- note added: "GATE"
- note added: "Switch turn on when power is down"
- note added: "This board has 4 functions\n- Measuring the voltage of the DC bus (VBUS)\n- Discharging the DC Bus when power is turned off\n- Precharging the DC bus through an external single IGBT module (Inrush_Limiter)\n- Driving the same IGBT module for DC link current & E-STOP (replacing contactor)"
- note added: "VBAT-"
- note added: "VBUS-\n"
- note removed: "This board has 4 functions\n- Measuring the voltage of the DC bus (VBUS)\n- Discharging the DC Bus when power is turned off\n- Precharging the DC bus through an external single IGBT module (Inrush_Limiter)\n- Driving an external Solid state contactor for E-STOP (IGBT module)"
Changed lines of the file:
@@
 	4650 4150 5050 4150
 Text Notes 800  6400 0    118  ~ 24
-This board has 4 functions\n- Measuring the voltage of the DC bus (VBUS)\n- Discharging the DC Bus when power is turned off\n- Precharging the DC bus through an external single IGBT module (Inrush_Limiter)\n- Driving an external Solid state contactor for E-STOP (IGBT module)
+This board has 4 functions\n- Measuring the voltage of the DC bus (VBUS)\n- Discharging the DC Bus when power is turned off\n- Precharging the DC bus through an external single IGBT module (Inrush_Limiter)\n- Driving the same IGBT module for DC link current & E-STOP (replacing contactor)
 Wire Notes Line
 	2300 2800 5400 2800
@@
 Wire Wire Line
 	5050 4150 5450 4150
+Text Notes 2700 3850 0    50   ~ 0
+Switch turn on when power is down
+$Comp
+L Device:Q_NIGBT_CEG Q?
+U 1 1 5A6C71DF
+P 9150 5350
+F 0 "Q?" H 9341 5396 50  0000 L CNN
+F 1 "IGBT" H 9341 5305 50  0000 L CNN
+F 2 "" H 9350 5450 50  0001 C CNN
+F 3 "" H 9150 5350 50  0001 C CNN
+	1    9150 5350
+	1    0    0    -1
+$EndComp
+NoConn ~ 9250 5150
+NoConn ~ 8950 5350
+NoConn ~ 9250 5550
+Text Notes 9300 5050 0    50   ~ 0
+VBUS-\n
+Text Notes 9250 5700 0    50   ~ 0
+VBAT-
+Text Notes 8700 5400 0    50   ~ 0
+GATE
+Wire Notes Line
+	8700 4750 8700 5800
+Wire Notes Line
+	8700 5800 10600 5800
+Wire Notes Line
+	10600 5800 10600 4750
+Wire Notes Line
+	10600 4750 8700 4750
+$Comp
+L Device:C C?
+U 1 1 5A6C71F0
+P 9700 5400
+F 0 "C?" H 9815 5446 50  0000 L CNN
+F 1 "DC Link Cap" H 9815 5355 50  0000 L CNN
+F 2 "Capacitors_SMD:C_0805_HandSoldering" H 9738 5250 50  0001 C CNN
+F 3 "" H 9700 5400 50  0001 C CNN
+	1    9700 5400
+	1    0    0    -1
+$EndComp
+NoConn ~ 9700 5250
+NoConn ~ 9700 5550
+Text Notes 9250 4900 0    50   ~ 0
+1200V 600A IGBT module
 $EndSCHEMATC

Commit message: VBUS sense
Connections:
- wire segments 51 -> 58
Other:
- note added: "VBAT+"
- note added: "VBUS+\n"
Changed lines of the file:
@@
 Wire Wire Line
 	4650 4150 5050 4150
-Text Notes 800  6400 0    118  ~ 24
+Text Notes 550  6450 0    118  ~ 24
 This board has 4 functions\n- Measuring the voltage of the DC bus (VBUS)\n- Discharging the DC Bus when power is turned off\n- Precharging the DC bus through an external single IGBT module (Inrush_Limiter)\n- Driving the same IGBT module for DC link current & E-STOP (replacing contactor)
 Wire Notes Line
@@
 L Device:Q_NIGBT_CEG Q?
 U 1 1 5A6C71DF
-P 9150 5350
-F 0 "Q?" H 9341 5396 50  0000 L CNN
-F 1 "IGBT" H 9341 5305 50  0000 L CNN
-F 2 "" H 9350 5450 50  0001 C CNN
-F 3 "" H 9150 5350 50  0001 C CNN
-	1    9150 5350
+P 9400 5950
+F 0 "Q?" H 9591 5996 50  0000 L CNN
+F 1 "IGBT" H 9591 5905 50  0000 L CNN
+F 2 "" H 9600 6050 50  0001 C CNN
+F 3 "" H 9400 5950 50  0001 C CNN
+	1    9400 5950
 	1    0    0    -1
 $EndComp
-NoConn ~ 9250 5150
-NoConn ~ 8950 5350
-NoConn ~ 9250 5550
-Text Notes 9300 5050 0    50   ~ 0
+NoConn ~ 9200 5950
+Text Notes 10150 5800 0    50   ~ 0
 VBUS-\n
-Text Notes 9250 5700 0    50   ~ 0
+Text Notes 8750 6350 0    50   ~ 0
 VBAT-
-Text Notes 8700 5400 0    50   ~ 0
+Text Notes 8950 6000 0    50   ~ 0
 GATE
 Wire Notes Line
-	8700 4750 8700 5800
+	8650 4850 8650 6400
 Wire Notes Line
-	8700 5800 10600 5800
+	8650 6400 10850 6400
 Wire Notes Line
-	10600 5800 10600 4750
+	10850 6400 10850 4850
 Wire Notes Line
-	10600 4750 8700 4750
+	10850 4850 8650 4850
+Text Notes 9700 6150 0    50   ~ 0
+1200V 600A IGBT module
+Text Notes 10300 5350 0    50   ~ 0
+VBUS+\n
 $Comp
 L Device:C C?
 U 1 1 5A6C71F0
-P 9700 5400
-F 0 "C?" H 9815 5446 50  0000 L CNN
-F 1 "DC Link Cap" H 9815 5355 50  0000 L CNN
-F 2 "Capacitors_SMD:C_0805_HandSoldering" H 9738 5250 50  0001 C CNN
-F 3 "" H 9700 5400 50  0001 C CNN
-	1    9700 5400
+P 9850 5500
+F 0 "C?" H 9965 5546 50  0000 L CNN
+F 1 "DC Link Cap" H 9965 5455 50  0000 L CNN
+F 2 "Capacitors_SMD:C_0805_HandSoldering" H 9888 5350 50  0001 C CNN
+F 3 "" H 9850 5500 50  0001 C CNN
+	1    9850 5500
 	1    0    0    -1
 $EndComp
-NoConn ~ 9700 5250
-NoConn ~ 9700 5550
-Text Notes 9250 4900 0    50   ~ 0
-1200V 600A IGBT module
+Wire Wire Line
+	9500 5750 9850 5750
+Wire Wire Line
+	9850 5350 10100 5350
+NoConn ~ 10100 5350
+NoConn ~ 10100 5750
+NoConn ~ 9050 5350
+NoConn ~ 9050 6350
+Wire Wire Line
+	9500 6150 9500 6350
+Wire Wire Line
+	9500 6350 9050 6350
+Connection ~ 9850 5350
+Wire Wire Line
+	9050 5350 9850 5350
+Wire Wire Line
+	9850 5650 9850 5750
+Connection ~ 9850 5750
+Wire Wire Line
+	9850 5750 10100 5750
+Text Notes 8750 5350 0    50   ~ 0
+VBAT+
 $EndSCHEMATC

Commit message: VBUS-sense
Parts:
- MK4: value BAT- -> VBAT-
Other:
- note added: "external circuit\n"
Changed lines of the file:
@@
 P 3450 950
 F 0 "MK4" V 3687 955 50  0000 C CNN
-F 1 "BAT-" V 3596 955 50  0000 C CNN
+F 1 "VBAT-" V 3596 955 50  0000 C CNN
 F 2 "Mounting_Holes:MountingHole_4.3mm_M4_Pad_Via" H 3450 950 50  0001 C CNN
 F 3 "" H 3450 950 50  0001 C CNN
@@
 Text Notes 8750 5350 0    50   ~ 0
 VBAT+
+Text Notes 9050 5000 0    50   ~ 0
+external circuit\n
 $EndSCHEMATC

Commit message: VBUS-Sense
Parts:
- J1: value Conn_01x02 E-STOP -> Conn_01x02 to external 12V power switch or VESC GPIO
- J3: value Conn_01x04 -> Conn_01x04 to vesc board
Changed lines of the file:
@@
 P 8350 3900
 F 0 "J3" H 8430 3892 50  0000 L CNN
-F 1 "Conn_01x04" H 8430 3801 50  0000 L CNN
+F 1 "Conn_01x04 to vesc board" H 8430 3801 50  0000 L CNN
 F 2 "Connectors_Molex:Molex_KK-6410-04_04x2.54mm_Straight" H 8350 3900 50  0001 C CNN
 F 3 "~" H 8350 3900 50  0001 C CNN
@@
 P 8850 1300
 F 0 "J1" H 8930 1292 50  0000 L CNN
-F 1 "Conn_01x02 E-STOP" H 8930 1201 50  0000 L CNN
+F 1 "Conn_01x02 to external 12V power switch or VESC GPIO" H 8930 1201 50  0000 L CNN
 F 2 "Connectors_Molex:Molex_KK-6410-02_02x2.54mm_Straight" H 8850 1300 50  0001 C CNN
 F 3 "~" H 8850 1300 50  0001 C CNN

Commit message: VBUS-sense
Other:
- note added: "FET turn on when power is down"
- note removed: "Switch turn on when power is down"
Changed lines of the file:
@@
 	5050 4150 5450 4150
 Text Notes 2700 3850 0    50   ~ 0
-Switch turn on when power is down
+FET turn on when power is down
 $Comp
 L Device:Q_NIGBT_CEG Q?

Commit message: Maintenance update
Parts:
- added BZ1: Buzzer, Buzzers_Beepers:MagneticBuzzer_ProSignal_ABT-410-RC, symbol Device:Buzzer
- C6: renamed from C?; footprint Capacitors_SMD:C_0805_HandSoldering -> (none)
- R1, R2, R3, R4: value 20k -> 7.5K
- gave numbers to parts that had none: 1
Connections:
- wire segments 58 -> 57
Other:
- note added: "FET turns on when power is down"
- note removed: "FET turn on when power is down"
- moved on the sheet: R1, R2, R3, R4

Commit message: Maintenance update
Parts:
- removed C6: DC Link Cap, symbol Device:C
- removed Q3: IGBT, symbol Device:Q_NIGBT_CEG
- added LOGO1: Logo_ENNOID, ENNOID:ENNOID-LOGO, symbol ENNOID:Logo_ENNOID
Connections:
- net labels added: DC Link Cap, IGBT
Changed lines of the file:
@@
 FET turns on when power is down
 $Comp
-L Device:Q_NIGBT_CEG Q3
+L Device:Q_NIGBT_CEG #Q3
 U 1 1 5A6C71DF
 P 1500 7100
-F 0 "Q3" H 1691 7146 50  0000 L CNN
+F 0 "#Q3" H 1691 7146 50  0001 L CNN
 F 1 "IGBT" H 1691 7055 50  0000 L CNN
-F 2 "" H 1700 7200 50  0001 C CNN
+F 2 "#" H 1700 7200 50  0001 C CNN
 F 3 "" H 1500 7100 50  0001 C CNN
 	1    1500 7100
@@
 VBUS+\n
 $Comp
-L Device:C C6
+L Device:C #C6
 U 1 1 5A6C71F0
 P 1950 6650
-F 0 "C6" H 2065 6696 50  0000 L CNN
+F 0 "#C6" H 2065 6696 50  0001 L CNN
 F 1 "DC Link Cap" H 2065 6605 50  0000 L CNN
-F 2 "" H 1988 6500 50  0001 C CNN
+F 2 "#" H 1988 6500 50  0001 C CNN
 F 3 "" H 1950 6650 50  0001 C CNN
 	1    1950 6650
@@
 Wire Wire Line
 	8100 4100 8150 4100
+$Comp
+L ENNOID:Logo_ENNOID LOGO1
+U 1 1 5A7768EF
+P 10350 6000
+F 0 "LOGO1" H 10350 6500 50  0001 C CNN
+F 1 "Logo_ENNOID" H 10350 5600 50  0001 C CNN
+F 2 "ENNOID:ENNOID-LOGO" H 10350 6000 50  0001 C CNN
+F 3 "" H 10350 6000 50  0001 C CNN
+	1    10350 6000
+	1    0    0    -1
+$EndComp
 $EndSCHEMATC

Commit message: Maintenance update
Other:
- note added: "This board has 4 functions\n- Measuring the voltage of the DC bus (VBUS)\n- Discharging the DC Bus when power is turned off\n- Precharging the DC bus through an external single IGBT module (Inrush_Limiter)\n- Driving an IGBT module for DC link current & E-STOP (replacing contactor)"
- note removed: "This board has 4 functions\n- Measuring the voltage of the DC bus (VBUS)\n- Discharging the DC Bus when power is turned off\n- Precharging the DC bus through an external single IGBT module (Inrush_Limiter)\n- Driving the same IGBT module for DC link current & E-STOP (replacing contactor)"
Changed lines of the file:
@@
 	4650 4150 5050 4150
 Text Notes 900  5650 0    118  ~ 24
-This board has 4 functions\n- Measuring the voltage of the DC bus (VBUS)\n- Discharging the DC Bus when power is turned off\n- Precharging the DC bus through an external single IGBT module (Inrush_Limiter)\n- Driving the same IGBT module for DC link current & E-STOP (replacing contactor)
+This board has 4 functions\n- Measuring the voltage of the DC bus (VBUS)\n- Discharging the DC Bus when power is turned off\n- Precharging the DC bus through an external single IGBT module (Inrush_Limiter)\n- Driving an IGBT module for DC link current & E-STOP (replacing contactor)
 Wire Notes Line
 	1950 2800 5400 2800
