File: VBUS-Sense/PCB/Inrush_Limiter.sch (KiCad schematic (older format))
At the start: 17 parts, among them Q2 BC546, U3 LTV-356T

Commit message: VBUS-SENSE changes
Parts:
- removed Q2: BC546, TO_SOT_Packages_THT:TO-92_Inline_Wide, symbol Transistor_BJT:BC546
- added Q2: 2N7000, TO_SOT_Packages_THT:TO-92_Inline_Wide, symbol Transistor_FET:2N7000
- C4: value DNP -> 100n
Changed lines of the file:
@@
 encoding utf-8
 Sheet 4 4
-Title ""
+Title "VBUS-SENSE"
 Date ""
-Rev ""
-Comp ""
+Rev "0.1"
+Comp "ENNOID"
 Comment1 ""
 Comment2 ""
@@
 	7600 2350 8850 2350
 $Comp
-L Transistor_BJT:BC546 Q2
-U 1 1 5A6EE6ED
-P 4950 3500
-F 0 "Q2" H 5141 3546 50  0000 L CNN
-F 1 "BC546" H 5141 3455 50  0000 L CNN
-F 2 "TO_SOT_Packages_THT:TO-92_Inline_Wide" H 5150 3425 50  0001 L CIN
-F 3 "http://www.fairchildsemi.com/ds/BC/BC547.pdf" H 4950 3500 50  0001 L CNN
-	1    4950 3500
-	1    0    0    -1
-$EndComp
-$Comp
 L Device:C C4
 U 1 1 5A6EEADE
 P 4000 3900
 F 0 "C4" H 4115 3946 50  0000 L CNN
-F 1 "DNP" H 4115 3855 50  0000 L CNN
+F 1 "100n" H 4115 3855 50  0000 L CNN
 F 2 "Capacitors_SMD:C_0805_HandSoldering" H 4038 3750 50  0001 C CNN
 F 3 "" H 4000 3900 50  0001 C CNN
@@
 Wire Wire Line
 	6300 2900 6300 3050
+$Comp
+L Transistor_FET:2N7000 Q2
+U 1 1 5A6CB3EA
+P 4950 3500
+F 0 "Q2" H 5155 3546 50  0000 L CNN
+F 1 "2N7000" H 5155 3455 50  0000 L CNN
+F 2 "TO_SOT_Packages_THT:TO-92_Inline_Wide" H 5150 3425 50  0001 L CIN
+F 3 "https://www.fairchildsemi.com/datasheets/2N/2N7000.pdf" H 4950 3500 50  0001 L CNN
+	1    4950 3500
+	1    0    0    -1
+$EndComp
 $EndSCHEMATC

Commit message: VBUS-sense
Other:
- note added: "Bring Gate to VBAT- \nfor shutting down the\nmain IGBT (E-STOP)\n\nconnected to external kill switch\n"
- note added: "automatic soft turn on of the external igbt"
- note removed: "Bring Gate to VBAT- \nfor shutting down the\nmain IGBT (E-STOP)\n"
Changed lines of the file:
@@
 	-1   0    0    1
 $EndComp
-Text Notes 4650 2200 0    50   ~ 0
-Bring Gate to VBAT-  \nfor shutting down the\nmain IGBT (E-STOP)\n
+Text Notes 1550 2300 0    50   ~ 0
+Bring Gate to VBAT-  \nfor shutting down the\nmain IGBT (E-STOP)\n\nconnected to external kill switch\n
 Wire Notes Line
 	7500 1000 5700 1000
@@
 	1    0    0    -1
 $EndComp
+Text Notes 6000 800  0    50   ~ 0
+automatic soft turn on of the external igbt
 $EndSCHEMATC

Commit message: Maintenance update
Parts:
- removed D4: D_Zener 12V, Diodes_SMD:D_SMA, symbol Device:D_Zener
- added C7: 100n, Capacitors_SMD:C_0805_HandSoldering, symbol Device:C
- added Q4: 2N7000, Package_TO_SOT_THT:TO-92_Inline, symbol Transistor_FET:2N7000
- added R16, R17: 1k, Resistors_SMD:R_0805_HandSoldering, symbol Device:R
- added R18: 200k, Resistors_SMD:R_1206, symbol Device:R
- C3: footprint Capacitors_SMD:C_0805_HandSoldering -> Capacitors_SMD:C_2225_HandSoldering
- Q2: footprint TO_SOT_Packages_THT:TO-92_Inline_Wide -> Package_TO_SOT_THT:TO-92_Inline
- R7: value 1k -> 1M
- R8: value 10k -> 1k
Connections:
- net labels added: +5V
- net labels removed: +VCC
- wire segments 49 -> 58
Other:
- note added: "Bring Gate to VBAT- \nfor shutting down the\nmain IGBT (E-STOP)\n"
- note added: "Full VBUS voltage \ncapacitor required"
- note removed: "Bring Gate to VBAT- \nfor shutting down the\nmain IGBT (E-STOP)\n\nconnected to external kill switch\n"

Commit message: Maintenance update
Parts:
- C3: footprint Capacitors_SMD:C_2225_HandSoldering -> Capacitors_SMD:C_1812_HandSoldering
Changed lines of the file:
@@
 F 0 "C3" H 6915 2546 50  0000 L CNN
 F 1 "0.15u" H 6915 2455 50  0000 L CNN
-F 2 "Capacitors_SMD:C_2225_HandSoldering" H 6838 2350 50  0001 C CNN
+F 2 "Capacitors_SMD:C_1812_HandSoldering" H 6838 2350 50  0001 C CNN
 F 3 "" H 6800 2500 50  0001 C CNN
 	1    6800 2500
