File: VBUS-Sense/PCB/V_PHASE.sch (KiCad schematic (older format))
At the start: 12 parts

Commit message: VBUS sensor & voltage sense circuit changes
Parts:
- U1: renamed from U?; footprint Housings_SOIC:SOIC-8_3.9x4.9mm_Pitch1.27mm -> Housings_SOIC:SSO-8_6.8x5.9mm_Pitch1.27mm_Clearance8mm
Connections:
- net labels added: VBUS+, VBUS-
- net labels removed: E, PHASE
Changed lines of the file:
@@
 $Descr A4 11693 8268
 encoding utf-8
-Sheet 2 2
+Sheet 2 3
 Title ""
 Date ""
@@
 	6650 3850 6300 3850
 Text HLabel 3500 3750 0    60   Input ~ 0
-PHASE
+VBUS+
 Wire Wire Line
 	3500 3750 3650 3750
 Text HLabel 2550 4200 0    60   Input ~ 0
-E
+VBUS-
 Connection ~ 4500 4200
 Wire Wire Line
@@
 	4800 3550 4500 3550
 $Comp
-L ENNOID:AMC1301 U?
+L ENNOID:AMC1301 U1
 U 1 1 5A4D5C88
 P 5900 3650
-F 0 "U?" H 5900 4117 50  0000 C CNN
+F 0 "U1" H 5900 4117 50  0000 C CNN
 F 1 "AMC1301" H 5900 4026 50  0000 C CNN
-F 2 "Housings_SOIC:SOIC-8_3.9x4.9mm_Pitch1.27mm" H 5900 3300 50  0001 C CIN
+F 2 "Housings_SOIC:SSO-8_6.8x5.9mm_Pitch1.27mm_Clearance8mm" H 5900 3300 50  0001 C CIN
 F 3 "" H 5900 3650 50  0001 C CNN
 	1    5900 3650

Commit message: Vsense
Parts:
- R27, R29: footprint Resistors_SMD:R_0805_HandSoldering -> Resistors_SMD:R_1206
Changed lines of the file:
@@
 F 0 "R27" V 3593 3750 50  0000 C CNN
 F 1 "1M" V 3684 3750 50  0000 C CNN
-F 2 "Resistors_SMD:R_0805_HandSoldering" V 3730 3750 50  0001 C CNN
+F 2 "Resistors_SMD:R_1206" V 3730 3750 50  0001 C CNN
 F 3 "" H 3800 3750 50  0001 C CNN
 	1    3800 3750
@@
 F 0 "R29" V 3993 3750 50  0000 C CNN
 F 1 "1M" V 4084 3750 50  0000 C CNN
-F 2 "Resistors_SMD:R_0805_HandSoldering" V 4130 3750 50  0001 C CNN
+F 2 "Resistors_SMD:R_1206" V 4130 3750 50  0001 C CNN
 F 3 "" H 4200 3750 50  0001 C CNN
 	1    4200 3750

Commit message: VBUS update
Parts:
- removed R31: 1k, Resistors_SMD:R_0805_HandSoldering, symbol device:R
- C37, C38, C39, C40, C9: symbol device:C -> VBUS-Sense-rescue:C-device
- D9: symbol device:D_Zener -> VBUS-Sense-rescue:D_Zener-device
- R27, R28, R29, R30: symbol device:R -> VBUS-Sense-rescue:R-device
Connections:
- wire segments 49 -> 48
Changed lines of the file:
@@
 $Descr A4 11693 8268
 encoding utf-8
-Sheet 2 3
+Sheet 2 4
 Title ""
 Date ""
@@
 $EndBitmap
 $Comp
-L device:C C37
+L VBUS-Sense-rescue:C-device C37
 U 1 1 5A30FC69
 P 5150 3300
@@
 $EndComp
 $Comp
-L device:C C38
+L VBUS-Sense-rescue:C-device C38
 U 1 1 5A30FE1D
 P 5150 3950
@@
 	5150 4200 5150 4100
 $Comp
-L device:R R28
+L VBUS-Sense-rescue:R-device R28
 U 1 1 5A30FF82
 P 4200 3000
@@
 $EndComp
 $Comp
-L device:R R27
+L VBUS-Sense-rescue:R-device R27
 U 1 1 5A30FFC5
 P 3800 3750
@@
 $EndComp
 $Comp
-L device:R R29
+L VBUS-Sense-rescue:R-device R29
 U 1 1 5A30FFF9
 P 4200 3750
@@
 $EndComp
 $Comp
-L device:R R30
+L VBUS-Sense-rescue:R-device R30
 U 1 1 5A310023
 P 4500 3950
@@
 	-1   0    0    1
 $EndComp
-$Comp
-L device:R R31
-U 1 1 5A3100D1
-P 4800 4200
-F 0 "R31" V 5007 4200 50  0000 C CNN
-F 1 "1k" V 4916 4200 50  0000 C CNN
-F 2 "Resistors_SMD:R_0805_HandSoldering" V 4730 4200 50  0001 C CNN
-F 3 "" H 4800 4200 50  0001 C CNN
-	1    4800 4200
-	0    -1   -1   0
-$EndComp
-Wire Wire Line
-	5150 4200 4950 4200
-Wire Wire Line
-	4650 4200 4500 4200
 Wire Wire Line
 	4500 4200 4500 4100
@@
 Connection ~ 5150 3000
 $Comp
-L device:D_Zener D9
+L VBUS-Sense-rescue:D_Zener-device D9
 U 1 1 5A3109F4
 P 4500 3250
@@
 	4500 3450 4500 3400
 $Comp
-L device:C C39
+L VBUS-Sense-rescue:C-device C39
 U 1 1 5A311419
 P 6750 3300
@@
 $EndComp
 $Comp
-L device:C C40
+L VBUS-Sense-rescue:C-device C40
 U 1 1 5A31145B
 P 7200 3300
@@
 	4050 3000 3800 3000
 $Comp
-L device:C C9
+L VBUS-Sense-rescue:C-device C9
 U 1 1 5A4DF1BA
 P 4800 3300
@@
 	1    0    0    -1
 $EndComp
+Wire Wire Line
+	4500 4200 5150 4200
 $EndSCHEMATC

Commit message: Maintenance update
Connections:
- wire segments 48 -> 47
Changed lines of the file:
@@
 $Bitmap
 Pos 1500 2950
-Scale 1.000000
+Scale 1,000000
 Data
 89 50 4E 47 0D 0A 1A 0A 00 00 00 0D 49 48 44 52 00 00 01 E5 00 00 02 56 08 02 00 00 00 E9 E4 08
@@
 $Bitmap
 Pos 2100 6650
-Scale 1.000000
+Scale 1,000000
 Data
 89 50 4E 47 0D 0A 1A 0A 00 00 00 0D 49 48 44 52 00 00 03 7F 00 00 02 77 08 02 00 00 00 AB F1 7F
@@
 $Bitmap
 Pos 9200 6000
-Scale 1.000000
+Scale 1,000000
 Data
 89 50 4E 47 0D 0A 1A 0A 00 00 00 0D 49 48 44 52 00 00 04 A0 00 00 02 55 08 02 00 00 00 66 B4 1A
@@
 Wire Wire Line
 	7200 3050 7700 3050
-$Comp
-L power:+5V #PWR021
-U 1 1 5A31BC2D
-P 7700 3000
-F 0 "#PWR021" H 7700 2850 50  0001 C CNN
-F 1 "+5V" H 7715 3173 50  0000 C CNN
-F 2 "" H 7700 3000 50  0001 C CNN
-F 3 "" H 7700 3000 50  0001 C CNN
-	1    7700 3000
-	1    0    0    -1
-$EndComp
-Wire Wire Line
-	7700 3000 7700 3050
-Connection ~ 7700 3050
 Wire Wire Line
 	7700 3050 7950 3050
@@
 Text HLabel 6650 3850 2    60   Output ~ 0
 Vout-
-$Comp
-L power:GND #PWR035
-U 1 1 5A34B574
-P 7600 3550
-F 0 "#PWR035" H 7600 3300 50  0001 C CNN
-F 1 "GND" H 7605 3377 50  0000 C CNN
-F 2 "" H 7600 3550 50  0001 C CNN
-F 3 "" H 7600 3550 50  0001 C CNN
-	1    7600 3550
-	1    0    0    -1
-$EndComp
 Text HLabel 7700 3550 2    60   Input ~ 0
 GND
 Wire Wire Line
 	7600 3550 7700 3550
-Connection ~ 7600 3550
 Text HLabel 3800 3000 0    60   Input ~ 0
 +VCC
